File: Hardware/USB-C Board.kicad_sch (KiCad schematic)
At the start: 45 parts, among them J1 USB_C_Receptacle_USB2.0, J2 Conn_01x04_Male, J3 Conn_01x02_Male, J4 Conn_01x02_Male, J5 Conn_01x02_Male, J6 Conn_01x02_Male, J9 QWIIC_Stackable, Q1 DMP3013SFV, SW1 SW_Push, U1 AMS1117-3.3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

Commit message: BOMing the place...
Parts:
- C1: Vendor (none) -> LCSC C89246
- C2, C3, C4: Vendor (none) -> LCSC C559769
- C5: Vendor (none) -> LCSC C14663
- D1, D2, D3, D4: Vendor (none) -> LCSC C10677
- D5: Vendor (none) -> LCSC C5355496
- D6: Vendor (none) -> LCSC C434421
- D7, D8: Vendor (none) -> LCSC C434424
- D9: Vendor (none) -> LCSC C434420
- J1: Vendor LCSC -> LCSC C2765186
- J9: Vendor (none) -> LCSC C145956,
- Q1: Vendor (none) -> LCSC C264098
- R1, R2: Vendor (none) -> LCSC C23186
- R10, R11, R12, R13, R14, R15, R3, R8, R9: Vendor (none) -> LCSC C21190
- R16, R17, R4, R6: Vendor (none) -> LCSC C25803
- R5: Vendor (none) -> LCSC C22775
- R7: Vendor (none) -> LCSC C31850
- SW1: Vendor (none) -> LCSC C2858276
- U1: Vendor (none) -> LCSC C6186
- U3: Vendor (none) -> LCSC C2678061
Changed lines of the file:
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@@
+      (effects (font (size 1.27 1.27)) hide)
+    )
+    (property "Vendor" "LCSC C5355496" (id 4) (at 242.57 53.34 90)
       (effects (font (size 1.27 1.27)) hide)
     )
@@
       (effects (font (size 1.27 1.27)) hide)
     )
+    (property "Vendor" "LCSC C145956, " (id 4) (at 133.35 52.07 0)
+      (effects (font (size 1.27 1.27)) hide)
+    )
     (pin "1")
     (pin "2")
@@
       (effects (font (size 1.27 1.27)) hide)
     )
+    (property "Vendor" "LCSC C434420" (id 4) (at 148.59 186.69 0)
+      (effects (font (size 1.27 1.27)) hide)
+    )
     (pin "1")
     (pin "2")
@@
       (effects (font (size 1.27 1.27)) hide)
     )
+    (property "Vendor" "LCSC C434424" (id 4) (at 148.59 166.37 0)
+      (effects (font (size 1.27 1.27)) hide)
+    )
     (pin "1")
     (pin "2")
@@
       (effects (font (size 1.27 1.27)) hide)
     )
+    (property "Vendor" "LCSC C559769" (id 4) (at 157.48 38.1 0)
+      (effects (font (size 1.27 1.27)) hide)
+    )
     (pin "1")
     (pin "2")
@@
     )
     (property "Datasheet" "~" (id 3) (at 242.57 63.5 0)
+      (effects (font (size 1.27 1.27)) hide)
+    )
+    (property "Vendor" "LCSC C559769" (id 4) (at 242.57 63.5 0)
       (effects (font (size 1.27 1.27)) hide)
     )
@@
       (effects (font (size 1.27 1.27)) (justify left bottom) hide)
     )
+    (property "Vendor" "LCSC C10677" (id 15) (at 63.5 44.45 0)
+      (effects (font (size 1.27 1.27)) hide)
+    )
     (pin "1")
     (pin "2")
@@
       (effects (font (size 1.27 1.27)) hide)
     )
+    (property "Vendor" "LCSC C22775" (id 4) (at 229.87 43.18 90)
+      (effects (font (size 1.27 1.27)) hide)
+    )
     (pin "1")
     (pin "2")
@@
     )
     (property "Datasheet" "~" (id 3) (at 213.36 39.37 0)
+      (effects (font (size 1.27 1.27)) hide)
+    )
+    (property "Vendor" "LCSC C25803" (id 4) (at 213.36 39.37 0)
       (effects (font (size 1.27 1.27)) hide)
     )
@@
       (effects (font (size 1.27 1.27)) hide)
     )
+    (property "Vendor" "LCSC C434421" (id 4) (at 148.59 156.21 0)
+      (effects (font (size 1.27 1.27)) hide)
+    )
     (pin "1")
     (pin "2")
@@
     )
     (property "Datasheet" "~" (id 3) (at 231.14 63.5 0)
+      (effects (font (size 1.27 1.27)) hide)
+    )
+    (property "Vendor" "LCSC C559769" (id 4) (at 231.14 63.5 0)
       (effects (font (size 1.27 1.27)) hide)
     )
@@
     (property "Arrow Price/Stock" "https://www.arrow.com/en/products/pgb1010603nr/littelfuse?region=nac" (id 14) (at 76.2 1017.78 0)
       (effects (font (size 1.27 1.27)) (justify left bottom) hide)
+    )
+    (property "Vendor" "LCSC C10677" (id 15) (at 63.5 24.13 0)
+      (effects (font (size 1.27 1.27)) hide)
     )
     (pin "1")
@@
       (effects (font (size 1.27 1.27)) hide)
     )
-    (property "Vendor" "LCSC" (id 4) (at 27.94 49.53 0)
+    (property "Vendor" "LCSC C2765186" (id 4) (at 27.94 49.53 0)
       (effects (font (size 1.27 1.27)) hide)
     )
@@
       (effects (font (size 1.27 1.27)) hide)
     )
+    (property "Vendor" "LCSC C89246" (id 5) (at 44.45 157.48 0)
+      (effects (font (size 1.27 1.27)) hide)
+    )
     (pin "1")
     (pin "2")
@@
       (effects (font (size 1.27 1.27)) hide)
     )
+    (property "Vendor" "LCSC C21190" (id 4) (at 138.43 156.21 90)
+      (effects (font (size 1.27 1.27)) hide)
+    )
     (pin "1")
     (pin "2")
@@
       (effects (font (size 1.27 1.27)) hide)
     )
+    (property "Vendor" "LCSC C25803" (id 4) (at 171.45 116.84 0)
+      (effects (font (size 1.27 1.27)) hide)
+    )
     (pin "1")
     (pin "2")
@@
     )
     (property "Datasheet" "~" (id 3) (at 158.75 83.82 0)
+      (effects (font (size 1.27 1.27)) hide)
+    )
+    (property "Vendor" "LCSC C21190" (id 4) (at 158.75 83.82 0)
       (effects (font (size 1.27 1.27)) hide)
     )
@@
       (effects (font (size 1.27 1.27)) hide)
     )
+    (property "Vendor" "LCSC C21190" (id 4) (at 166.37 38.1 0)
+      (effects (font (size 1.27 1.27)) hide)
+    )
     (pin "1")
     (pin "2")
@@
     )
     (property "Datasheet" "~" (id 3) (at 148.59 83.82 0)
+      (effects (font (size 1.27 1.27)) hide)
+    )
+    (property "Vendor" "LCSC C21190" (id 4) (at 148.59 83.82 0)
       (effects (font (size 1.27 1.27)) hide)
     )
@@
     )
     (property "Datasheet" "~" (id 3) (at 259.08 48.26 0)
+      (effects (font (size 1.27 1.27)) hide)
+    )
+    (property "Vendor" "LCSC C21190" (id 4) (at 259.08 48.26 0)
       (effects (font (size 1.27 1.27)) hide)
     )
@@
       (effects (font (size 1.27 1.27)) hide)
     )
+    (property "Vendor" "LCSC C6186" (id 4) (at 33.02 153.67 0)
+      (effects (font (size 1.27 1.27)) hide)
+    )
     (pin "1")
     (pin "2")
@@
       (effects (font (size 1.27 1.27)) hide)
     )
+    (property "Vendor" "LCSC C434424" (id 4) (at 148.59 176.53 0)
+      (effects (font (size 1.27 1.27)) hide)
+    )
     (pin "1")
     (pin "2")
@@
       (effects (font (size 1.27 1.27)) hide)
     )
+    (property "Vendor" "LCSC C21190" (id 4) (at 138.43 166.37 90)
+      (effects (font (size 1.27 1.27)) hide)
+    )
     (pin "1")
     (pin "2")
@@
       (effects (font (size 1.27 1.27)) hide)
     )
+    (property "Vendor" "LCSC C14663" (id 4) (at 236.22 38.1 0)
+      (effects (font (size 1.27 1.27)) hide)
+    )
     (pin "1")
     (pin "2")
@@
       (effects (font (size 1.27 1.27)) hide)
     )
+    (property "Vendor" "LCSC C23186" (id 4) (at 34.29 118.11 90)
+      (effects (font (size 1.27 1.27)) hide)
+    )
     (pin "1")
     (pin "2")
@@
       (effects (font (size 1.27 1.27)) hide)
     )
+    (property "Vendor" "LCSC C31850" (id 4) (at 215.9 48.26 90)
+      (effects (font (size 1.27 1.27)) hide)
+    )
     (pin "1")
     (pin "2")
@@
     )
     (property "Datasheet" "~" (id 3) (at 138.43 176.53 0)
+      (effects (font (size 1.27 1.27)) hide)
+    )
+    (property "Vendor" "LCSC C21190" (id 4) (at 138.43 176.53 90)
       (effects (font (size 1.27 1.27)) hide)
     )
@@
       (effects (font (size 1.27 1.27)) hide)
     )
+    (property "Vendor" "LCSC C23186" (id 4) (at 34.29 115.57 90)
+      (effects (font (size 1.27 1.27)) hide)
+    )
     (pin "1")
     (pin "2")
@@
       (effects (font (size 1.27 1.27)) hide)
     )
+    (property "Vendor" "LCSC C21190" (id 4) (at 138.43 186.69 90)
+      (effects (font (size 1.27 1.27)) hide)
+    )
     (pin "1")
     (pin "2")
@@
     )
     (property "Datasheet" "~" (id 3) (at 176.53 71.12 0)
+      (effects (font (size 1.27 1.27)) hide)
+    )
+    (property "Vendor" "LCSC C25803" (id 4) (at 176.53 71.12 0)
       (effects (font (size 1.27 1.27)) hide)
     )
@@
     (property "Arrow Price/Stock" "https://www.arrow.com/en/products/pgb1010603nr/littelfuse?region=nac" (id 14) (at 76.2 1027.94 0)
       (effects (font (size 1.27 1.27)) (justify left bottom) hide)
+    )
+    (property "Vendor" "LCSC C10677" (id 15) (at 63.5 34.29 0)
+      (effects (font (size 1.27 1.27)) hide)
     )
     (pin "1")
@@
       (effects (font (size 1.27 1.27)) hide)
     )
+    (property "Vendor" "LCSC C2858276" (id 4) (at 176.53 55.88 90)
+      (effects (font (size 1.27 1.27)) hide)
+    )
     (pin "1")
     (pin "2")
@@
     (property "Arrow Price/Stock" "https://www.arrow.com/en/products/pgb1010603nr/littelfuse?region=nac" (id 14) (at 76.2 1048.26 0)
       (effects (font (size 1.27 1.27)) (justify left bottom) hide)
+    )
+    (property "Vendor" "LCSC C10677" (id 15) (at 63.5 54.61 0)
+      (effects (font (size 1.27 1.27)) hide)
     )
     (pin "1")
@@
     )
     (property "Datasheet" "https://www.st.com/resource/en/datasheet/stusb4500.pdf" (id 3) (at 204.47 82.55 0)
+      (effects (font (size 1.27 1.27)) hide)
+    )
+    (property "Vendor" "LCSC C2678061" (id 4) (at 204.47 82.55 0)
       (effects (font (size 1.27 1.27)) hide)
     )
@@
       (effects (font (size 1.27 1.27)) (justify left) hide)
     )
+    (property "Vendor" "LCSC C264098" (id 4) (at 220.98 34.29 90)
+      (effects (font (size 1.27 1.27)) hide)
+    )
     (pin "1")
     (pin "2")
@@
       (effects (font (size 1.27 1.27)) hide)
     )
+    (property "Vendor" "LCSC C21190" (id 4) (at 138.43 83.82 0)
+      (effects (font (size 1.27 1.27)) hide)
+    )
     (pin "1")
     (pin "2")
@@
       (effects (font (size 1.27 1.27)) hide)
     )
+    (property "Vendor" "LCSC C25803" (id 4) (at 181.61 116.84 0)
+      (effects (font (size 1.27 1.27)) hide)
+    )
