File: Hardware/Controller-Tinker.kicad_pcb (KiCad board)
At the start: 2 copper layers, 34 x 34 mm, 25 parts, among them J2 Conn_01x04_Male, J3 Conn_01x02_Male, J4 Conn_01x02_Male, J5 Conn_01x02_Male, J6 Conn_01x02_Male, J9 Conn_01x04_MountingPin, U1 SST25VF016B-50-4I-S2AF, U2 ESP8266EX, Y1 26.000MHz

Commit message: ......
Parts:
- added C8: 22uf, Capacitor_Tantalum_SMD:CP_EIA-3528-21_Kemet-B_Pad1.50x2.35mm_HandSolder, F.Cu at (95.1, 77.8)
- added J4: Conn_01x07_Male, Connector_PinHeader_2.54mm:PinHeader_1x07_P2.54mm_Vertical, F.Cu at (93.7, 100.9)
- added Q1: UMH3N, Package_TO_SOT_SMD:SOT-363_SC-70-6, F.Cu at (105.1, 97.0)
- added R6: 10K, Resistor_SMD:R_0603_1608Metric, F.Cu at (98.7, 96.6)
- added R7: 10K, Resistor_SMD:R_0603_1608Metric, F.Cu at (107.6, 96.8)
- moved C4 45.5 mm to (103.2, 81.1)
- moved Y1 44.4 mm to (103.2, 83.5)
- moved R3 36.6 mm to (97.5, 79.0), turned to 90 degrees
- moved U2 33.6 mm to (93.1, 92.9), turned to -90 degrees
- moved C7 31.4 mm to (97.0, 96.6), turned to -90 degrees
- moved R1 28.7 mm to (99.0, 79.0), turned to -90 degrees
- moved C3 27.9 mm to (103.2, 85.9), turned to 180 degrees
- moved R5 27.3 mm to (89.3, 94.0), turned to -90 degrees
- moved U1 24.7 mm to (95.1, 83.8), turned to -90 degrees
- moved R2 24.2 mm to (100.4, 84.2), turned to 90 degrees
- moved C6 23.0 mm to (90.2, 85.7), turned to 90 degrees
- moved C5 21.0 mm to (90.5, 82.1), turned to 180 degrees
- moved R4 16.7 mm to (92.7, 79.0), turned to 90 degrees
- renumbered U2 to U1, U1 to U2
Connections:
- J2 pad 1: Vout -> unconnected-(J2-Pad1)
- J2 pad 2: UD+ -> unconnected-(J2-Pad2)
- J2 pad 3: UD- -> unconnected-(J2-Pad3)
- J3 pad 1: Vout -> unconnected-(J3-Pad1)
- J5 pad 1: Vsec -> unconnected-(J5-Pad1)
- J6 pad 1: Vsec -> unconnected-(J6-Pad1)
- J9 pad 2: 2v7 -> +3V3
- R5 pad 1: IO6 -> SCL
Routing:
- net +3V3: track 0.00 -> 77.8 mm, vias 0 -> 3
- net RST: track 0.00 -> 34.1 mm, vias 0 -> 1
- net IO0: track 0.00 -> 22.6 mm, vias 0 -> 2
- net IO3: track 0.00 -> 19.4 mm
- net IO1: track 0.00 -> 18.2 mm
- net IO8: track 0.00 -> 17.1 mm
- net SCL: track 0.00 -> 16.4 mm, vias 0 -> 2
- net IO9: track 0.00 -> 12.3 mm
- net /eXi: track 0.00 -> 9.24 mm
- net IO7: track 0.00 -> 7.85 mm
- net SDA: track 0.00 -> 6.86 mm, vias 0 -> 2
- net /eXo: track 0.00 -> 6.62 mm
- net /RTS: track 0.00 -> 6.59 mm
- net IO10: track 0.00 -> 4.16 mm
- net /DTR: track 0.00 -> 4.07 mm
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Other:
- board text added: "3v3"
- board text added: "DTR"
- board text added: "Freakin' HUGE!"
- board text added: "Needs power from the USB board. Needs a UI. (Needs LEDs! - Austin)"
- board text added: "RST"
- board text added: "RTS"
- board text added: "RxD"
- board text added: "TxD"

Commit message: ...
Parts:
- renumbered J4 to J1
Connections:
- J4 pad 1: Vout -> unconnected-(J4-Pad1)

Commit message: .........
Parts:
- C8: footprint Capacitor_Tantalum_SMD:CP_EIA-3528-21_Kemet-B_Pad1.50x2.35mm_HandSolder -> Tinker:CP_EIA-6032-28-Tantalumm_HandSolder
- J9: value Conn_01x04_MountingPin -> QWIIC_Stackable; footprint Tinker:JST_SH_SM04B-SRSS-TB_1x04-1MP_P1.00mm_Horizontal -> Tinker:QWIIC_Stackable
- moved C8 6.42 mm to (88.8, 78.8), turned to 180 degrees
- moved R4 1.50 mm to (94.2, 79.0)
Routing:
- net SCL: track 16.4 -> 29.3 mm, vias 2 -> 1
- net +3V3: track 77.8 -> 86.1 mm, vias 3 -> 2
- net SDA: track 6.86 -> 7.87 mm, vias 2 -> 1
