File: Hardware/Controller-Tinker.kicad_sch (KiCad schematic)
At the start: 22 parts, among them J1 Conn_Coaxial, J2 Conn_01x04_Male, J3 Conn_01x02_Male, J5 Conn_01x02_Male, J6 Conn_01x02_Male, J9 Conn_01x04_MountingPin, U1 SST25VF016B-50-4I-S2AF, U2 ESP8266EX, Y1 26.000MHz

Commit message: ......
Parts:
- added C8: 22uf, Capacitor_Tantalum_SMD:CP_EIA-3528-21_Kemet-B_Pad1.50x2.35mm_HandSolder, symbol Device:C_Polarized
- added J4: Conn_01x07_Male, Connector_PinHeader_2.54mm:PinHeader_1x07_P2.54mm_Vertical, symbol Connector:Conn_01x07_Male
- added Q1: UMH3N, Package_TO_SOT_SMD:SOT-363_SC-70-6, symbol Transistor_BJT:UMH3N
- added R6, R7: 10K, Resistor_SMD:R_0603_1608Metric, symbol Device:R
- renumbered U2 to U1, U1 to U2
Connections:
- net 2v7 is gone; now on net +3V3: J9.2 (Pin_2)
- net IO6 is gone; now on net SCL: R5.1
- net +3V3: now also C8.1, J4.1 (Pin_1), R6.2, R7.2
- net GND: now also C8.2, J4.4 (Pin_4); no longer J1.2 (Ext)
- net IO0: now also Q1.4 (E2), R7.1
- net IO1: now also J4.3 (Pin_3), R6.1
- net IO3: now also J4.2 (Pin_2)
- net RST: now also J4.7 (Pin_7), Q1.6 (C1)
- net UD+: no longer J2.2 (Pin_2)
- net UD-: no longer J2.3 (Pin_3)
- net Vout: no longer J2.1 (Pin_1), J3.1 (Pin_1)
- net Vsec: no longer J5.1 (Pin_1), J6.1 (Pin_1)
- new net DTR: J4.5 (Pin_5), Q1.2 (B1), Q1.3 (C2)
- new net RTS: J4.6 (Pin_6), Q1.1 (E1), Q1.5 (B2)
- no-connect marks 1 -> 7
Other:
- note added: "ESP8266"
- note added: "I2C"
- note added: "Programming"
- note removed: "(stuff for PD)"
- note removed: "QUESTION! Should J9 pin 2 really be connected to 2v7?"
- note removed: "STUSB4500"
- title: USB-C (PD) Board -> USB-C PD Controller
- moved on the sheet: AE1, C1, C2, C3, C4, C5, C6, C7, J1, J2, J3, J5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

Commit message: ...
Parts:
- added J4: Conn_01x02_Male, Tinker:PinHeader_1x02_P2.54mm_Vertical, symbol Connector:Conn_01x02_Male
- renumbered J4 to J1, J1 to J10
Connections:
- net GND: now also J4.2 (Pin_2)
- no-connect marks 7 -> 8
Changed lines of the file:
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@@
   (no_connect (at 26.67 34.29))
   (no_connect (at 26.67 148.59))
+  (no_connect (at 50.8 102.87))
   (no_connect (at 52.07 148.59))
   (no_connect (at 26.67 36.83))
@@
     (stroke (width 0) (type default) (color 0 0 0 0))
   )
+  (wire (pts (xy 50.8 105.41) (xy 46.99 105.41))
+    (stroke (width 0) (type default) (color 0 0 0 0))
+  )
   (wire (pts (xy 138.43 36.83) (xy 138.43 44.45))
     (stroke (width 0) (type default) (color 0 0 0 0))
@@
     )
   )
+  (global_label "Vout" (shape input) (at 48.26 102.87 180) (fields_autoplaced)
+    (effects (font (size 1.27 1.27)) (justify right))
+    (property "Intersheet References" "${INTERSHEET_REFS}" (id 0) (at 41.7345 102.7906 0)
+      (effects (font (size 1.27 1.27)) (justify right) hide)
+    )
+  )
   (global_label "SCL" (shape input) (at 220.98 127 0) (fields_autoplaced)
     (effects (font (size 1.27 1.27)) (justify left))
@@
   (symbol (lib_id "Connector:Conn_Coaxial") (at 190.5 87.63 0) (unit 1)
     (in_bom no) (on_board no) (fields_autoplaced)
-    (property "Reference" "J1" (id 0) (at 194.31 87.9231 0)
+    (property "Reference" "J10" (id 0) (at 194.31 87.9231 0)
       (effects (font (size 1.27 1.27)) (justify left))
     )
@@
     (pin "1")
   )
+  (symbol (lib_id "power:GND") (at 46.99 105.41 0) (mirror y) (unit 1)
+    (in_bom yes) (on_board yes)
+    (property "Reference" "#PWR0121" (id 0) (at 46.99 111.76 0)
+      (effects (font (size 1.27 1.27)) hide)
+    )
+    (property "Value" "GND" (id 1) (at 46.863 109.8042 0))
+    (property "Footprint" "" (id 2) (at 46.99 105.41 0)
+      (effects (font (size 1.27 1.27)) hide)
+    )
+    (property "Datasheet" "" (id 3) (at 46.99 105.41 0)
+      (effects (font (size 1.27 1.27)) hide)
+    )
+    (pin "1")
+  )
   (symbol (lib_id "power:+3.3V") (at 207.01 39.37 0) (unit 1)
     (in_bom yes) (on_board yes) (fields_autoplaced)
@@
     )
     (pin "1")
+  )
+  (symbol (lib_id "Connector:Conn_01x02_Male") (at 55.88 102.87 0) (mirror y) (unit 1)
+    (in_bom yes) (on_board yes)
+    (property "Reference" "J4" (id 0) (at 55.245 97.79 0))
+    (property "Value" "Conn_01x02_Male" (id 1) (at 55.245 100.33 0))
+    (property "Footprint" "Tinker:PinHeader_1x02_P2.54mm_Vertical" (id 2) (at 55.88 102.87 0)
+      (effects (font (size 1.27 1.27)) hide)
+    )
+    (property "Datasheet" "~" (id 3) (at 55.88 102.87 0)
+      (effects (font (size 1.27 1.27)) hide)
+    )
+    (pin "1")
+    (pin "2")
   )
   (symbol (lib_id "0-TINKER Customs:ABM8-26.000MHz-20-D1X-T") (at 210.82 88.9 0) (unit 1)
@@
   (symbol (lib_id "Connector:Conn_01x07_Male") (at 102.87 50.8 0) (unit 1)
     (in_bom yes) (on_board yes)
-    (property "Reference" "J4" (id 0) (at 103.505 38.1 0))
+    (property "Reference" "J1" (id 0) (at 103.505 38.1 0))
     (property "Value" "Conn_01x07_Male" (id 1) (at 107.95 50.8 90)
       (effects (font (size 1.27 1.27)) hide)
@@
       (reference "#PWR0120") (unit 1) (value "GND") (footprint "")
     )
+    (path "/994694c7-9213-431b-bed4-b4944e05294c"
+      (reference "#PWR0121") (unit 1) (value "GND") (footprint "")
+    )
     (path "/df37fa07-f19e-4b86-8f6a-f7465dd4c78c"
       (reference "#PWR0123") (unit 1) (value "GND") (footprint "")
@@
       (reference "C8") (unit 1) (value "22uf") (footprint "Capacitor_Tantalum_SMD:CP_EIA-3528-21_Kemet-B_Pad1.50x2.35mm_HandSolder")
     )
-    (path "/029b3e5a-c445-46a8-9f4d-5907f95d4882"
-      (reference "J1") (unit 1) (value "Conn_Coaxial") (footprint "Connector_Coaxial:U.FL_Molex_MCRF_73412-0110_Vertical")
+    (path "/ff08f666-d31b-45a5-8777-a0482d9fced1"
+      (reference "J1") (unit 1) (value "Conn_01x07_Male") (footprint "Connector_PinHeader_2.54mm:PinHeader_1x07_P2.54mm_Vertical")
     )
     (path "/ce562b82-4d15-4512-9ef8-80a89b06889d"
@@
       (reference "J3") (unit 1) (value "Conn_01x02_Male") (footprint "Tinker:PinHeader_1x02_P2.54mm_Vertical")
     )
-    (path "/ff08f666-d31b-45a5-8777-a0482d9fced1"
-      (reference "J4") (unit 1) (value "Conn_01x07_Male") (footprint "Connector_PinHeader_2.54mm:PinHeader_1x07_P2.54mm_Vertical")
+    (path "/e516ae01-774d-4d4f-b0c4-6f2304b851fc"
+      (reference "J4") (unit 1) (value "Conn_01x02_Male") (footprint "Tinker:PinHeader_1x02_P2.54mm_Vertical")
     )
     (path "/fb3406f1-7439-4c3c-b07d-423418b2c3c6"
@@
       (reference "J9") (unit 1) (value "Conn_01x04_MountingPin") (footprint "Tinker:JST_SH_SM04B-SRSS-TB_1x04-1MP_P1.00mm_Horizontal")
     )
+    (path "/029b3e5a-c445-46a8-9f4d-5907f95d4882"
+      (reference "J10") (unit 1) (value "Conn_Coaxial") (footprint "Connector_Coaxial:U.FL_Molex_MCRF_73412-0110_Vertical")
+    )
     (path "/19bc14f3-d8ae-4814-b05f-47c0ed846eb8"

Commit message: .........
Parts:
- removed J9: Conn_01x04_MountingPin, Tinker:JST_SH_SM04B-SRSS-TB_1x04-1MP_P1.00mm_Horizontal, symbol Connector_Generic_MountingPin:Conn_01x04_MountingPin
- added J9: QWIIC_Stackable, Tinker:QWIIC_Stackable, symbol Connector_QWIIC_Stackable:QWIIC_Stackable
- C8: footprint Capacitor_Tantalum_SMD:CP_EIA-3528-21_Kemet-B_Pad1.50x2.35mm_HandSolder -> Tinker:CP_EIA-6032-28-Tantalumm_HandSolder
Connections:
- net +3V3: now also J9.2 (Pin_2)
- net GND: now also J9.1 (Pin_1), J9.MP (MountPin)
- net SCL: now also J9.4 (Pin_4)
- net SDA: now also J9.3 (Pin_3)
Changed lines of the file:
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@@
     (company "The Nerd Mage")
   )
+  (junction (at 119.38 88.9) (diameter 0) (color 0 0 0 0)
+  )
   (junction (at 242.57 39.37) (diameter 0) (color 0 0 0 0)
   )
@@
   )
   (junction (at 220.98 88.9) (diameter 0) (color 0 0 0 0)
+  )
+  (junction (at 119.38 86.36) (diameter 0) (color 0 0 0 0)
   )
   (junction (at 212.09 100.33) (diameter 0) (color 0 0 0 0)
@@
     (stroke (width 0) (type default) (color 0 0 0 0))
   )
+  (wire (pts (xy 119.38 88.9) (xy 119.3251 88.9184))
+    (stroke (width 0) (type default) (color 0 0 0 0))
+  )
   (wire (pts (xy 191.77 60.96) (xy 190.5 60.96))
     (stroke (width 0) (type default) (color 0 0 0 0))
@@
     (stroke (width 0) (type default) (color 0 0 0 0))
   )
-  (polyline (pts (xy 133.35 72.39) (xy 133.35 109.22))
+  (polyline (pts (xy 144.78 72.39) (xy 144.78 109.22))
     (stroke (width 0) (type default) (color 0 0 0 0))
   )
@@
     (stroke (width 0) (type default) (color 0 0 0 0))
   )
-  (polyline (pts (xy 99.06 72.39) (xy 133.35 72.39))
+  (polyline (pts (xy 99.06 72.39) (xy 144.78 72.39))
     (stroke (width 0) (type default) (color 0 0 0 0))
   )
@@
     (stroke (width 0) (type default) (color 0 0 0 0))
   )
+  (wire (pts (xy 119.38 86.36) (xy 119.3251 86.3784))
+    (stroke (width 0) (type default) (color 0 0 0 0))
+  )
   (wire (pts (xy 255.27 31.75) (xy 267.97 31.75))
     (stroke (width 0) (type default) (color 0 0 0 0))
@@
     (stroke (width 0) (type default) (color 0 0 0 0))
   )
-  (polyline (pts (xy 133.35 109.22) (xy 99.06 109.22))
+  (polyline (pts (xy 144.78 109.22) (xy 99.06 109.22))
     (stroke (width 0) (type default) (color 0 0 0 0))
   )
@@
       (effects (font (size 1.27 1.27)) (justify left))
     )
-    (property "Footprint" "Capacitor_Tantalum_SMD:CP_EIA-3528-21_Kemet-B_Pad1.50x2.35mm_HandSolder" (id 2) (at 224.4852 46.99 0)
+    (property "Footprint" "Tinker:CP_EIA-6032-28-Tantalumm_HandSolder" (id 2) (at 224.4852 46.99 0)
       (effects (font (size 1.27 1.27)) hide)
     )
@@
     (pin "1")
   )
-  (symbol (lib_id "Connector_Generic_MountingPin:Conn_01x04_MountingPin") (at 124.46 88.9 0) (unit 1)
+  (symbol (lib_id "Device:R") (at 125.73 44.45 180) (unit 1)
+    (in_bom yes) (on_board yes)
+    (property "Reference" "R6" (id 0) (at 123.19 44.45 90))
+    (property "Value" "10K" (id 1) (at 128.27 44.45 90))
+    (property "Footprint" "Resistor_SMD:R_0603_1608Metric" (id 2) (at 127.508 44.45 90)
+      (effects (font (size 1.27 1.27)) hide)
+    )
+    (property "Datasheet" "~" (id 3) (at 125.73 44.45 0)
+      (effects (font (size 1.27 1.27)) hide)
+    )
+    (pin "1")
+    (pin "2")
+  )
+  (symbol (lib_id "power:+3.3V") (at 215.9 115.57 0) (unit 1)
+    (in_bom yes) (on_board yes)
+    (property "Reference" "#PWR0109" (id 0) (at 215.9 119.38 0)
+      (effects (font (size 1.27 1.27)) hide)
+    )
+    (property "Value" "+3.3V" (id 1) (at 215.9 111.76 0))
+    (property "Footprint" "" (id 2) (at 215.9 115.57 0)
+      (effects (font (size 1.27 1.27)) hide)
+    )
+    (property "Datasheet" "" (id 3) (at 215.9 115.57 0)
+      (effects (font (size 1.27 1.27)) hide)
+    )
+    (pin "1")
+  )
+  (symbol (lib_id "Device:R") (at 156.21 54.61 180) (unit 1)
+    (in_bom yes) (on_board yes)
+    (property "Reference" "R7" (id 0) (at 153.67 54.61 90))
+    (property "Value" "10K" (id 1) (at 158.75 54.61 90))
+    (property "Footprint" "Resistor_SMD:R_0603_1608Metric" (id 2) (at 157.988 54.61 90)
+      (effects (font (size 1.27 1.27)) hide)
+    )
+    (property "Datasheet" "~" (id 3) (at 156.21 54.61 0)
+      (effects (font (size 1.27 1.27)) hide)
+    )
+    (pin "1")
+    (pin "2")
+  )
+  (symbol (lib_id "Connector_QWIIC_Stackable:QWIIC_Stackable") (at 124.46 88.9 0) (unit 1)
     (in_bom yes) (on_board yes) (fields_autoplaced)
-    (property "Reference" "J9" (id 0) (at 127 90.5255 0)
+    (property "Reference" "J9" (id 0) (at 127.0549 89.2555 0)
       (effects (font (size 1.27 1.27)) (justify left))
     )
-    (property "Value" "Conn_01x04_MountingPin" (id 1) (at 127 91.7955 0)
-      (effects (font (size 1.27 1.27)) (justify left) hide)
-    )
-    (property "Footprint" "Tinker:JST_SH_SM04B-SRSS-TB_1x04-1MP_P1.00mm_Horizontal" (id 2) (at 124.46 88.9 0)
-      (effects (font (size 1.27 1.27)) hide)
+    (property "Value" "QWIIC_Stackable" (id 1) (at 127.0549 91.7955 0)
+      (effects (font (size 1.27 1.27)) (justify left))
+    )
+    (property "Footprint" "Tinker:QWIIC_Stackable" (id 2) (at 125.73 99.06 0)
+      (effects (font (size 1.27 1.27)) (justify left) hide)
     )
     (property "Datasheet" "~" (id 3) (at 124.46 88.9 0)
@@
     (pin "4")
     (pin "MP")
-  )
-  (symbol (lib_id "Device:R") (at 125.73 44.45 180) (unit 1)
-    (in_bom yes) (on_board yes)
-    (property "Reference" "R6" (id 0) (at 123.19 44.45 90))
-    (property "Value" "10K" (id 1) (at 128.27 44.45 90))
-    (property "Footprint" "Resistor_SMD:R_0603_1608Metric" (id 2) (at 127.508 44.45 90)
-      (effects (font (size 1.27 1.27)) hide)
-    )
-    (property "Datasheet" "~" (id 3) (at 125.73 44.45 0)
-      (effects (font (size 1.27 1.27)) hide)
-    )
-    (pin "1")
-    (pin "2")
-  )
-  (symbol (lib_id "power:+3.3V") (at 215.9 115.57 0) (unit 1)
-    (in_bom yes) (on_board yes)
-    (property "Reference" "#PWR0109" (id 0) (at 215.9 119.38 0)
-      (effects (font (size 1.27 1.27)) hide)
-    )
-    (property "Value" "+3.3V" (id 1) (at 215.9 111.76 0))
-    (property "Footprint" "" (id 2) (at 215.9 115.57 0)
-      (effects (font (size 1.27 1.27)) hide)
-    )
-    (property "Datasheet" "" (id 3) (at 215.9 115.57 0)
-      (effects (font (size 1.27 1.27)) hide)
-    )
-    (pin "1")
-  )
-  (symbol (lib_id "Device:R") (at 156.21 54.61 180) (unit 1)
-    (in_bom yes) (on_board yes)
-    (property "Reference" "R7" (id 0) (at 153.67 54.61 90))
-    (property "Value" "10K" (id 1) (at 158.75 54.61 90))
-    (property "Footprint" "Resistor_SMD:R_0603_1608Metric" (id 2) (at 157.988 54.61 90)
-      (effects (font (size 1.27 1.27)) hide)
-    )
-    (property "Datasheet" "~" (id 3) (at 156.21 54.61 0)
-      (effects (font (size 1.27 1.27)) hide)
-    )
-    (pin "1")
-    (pin "2")
   )
   (symbol (lib_id "Connector:Conn_01x02_Male") (at 57.15 148.59 0) (mirror y) (unit 1)
@@
     )
     (path "/5c104459-36e5-4950-bac8-f51d6ee510aa"
-      (reference "C8") (unit 1) (value "22uf") (footprint "Capacitor_Tantalum_SMD:CP_EIA-3528-21_Kemet-B_Pad1.50x2.35mm_HandSolder")
+      (reference "C8") (unit 1) (value "22uf") (footprint "Tinker:CP_EIA-6032-28-Tantalumm_HandSolder")
     )
     (path "/ff08f666-d31b-45a5-8777-a0482d9fced1"
@@
       (reference "J6") (unit 1) (value "Conn_01x02_Male") (footprint "Tinker:PinHeader_1x02_P2.54mm_Vertical")
     )
-    (path "/ae69f442-7b32-4ab2-972d-28d283e0750f"
-      (reference "J9") (unit 1) (value "Conn_01x04_MountingPin") (footprint "Tinker:JST_SH_SM04B-SRSS-TB_1x04-1MP_P1.00mm_Horizontal")
+    (path "/b8e59293-57c0-410d-9624-31545ded5709"
+      (reference "J9") (unit 1) (value "QWIIC_Stackable") (footprint "Tinker:QWIIC_Stackable")
     )
     (path "/029b3e5a-c445-46a8-9f4d-5907f95d4882"

Commit message: fiddlin' with stuff...
Parts:
- J1: Note (none) -> Footprint only; now left out of the parts list
- J2, J3, J4, J5, J6: now left out of the parts list
Other:
- note added: "Footprint(s) only"
Changed lines of the file:
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@@
     (effects (font (size 2.54 2.54)) (justify left bottom))
+  )
+  (text "Footprint(s) only" (at 27.94 46.99 0)
+    (effects (font (size 1.27 1.27)) (justify left bottom))
+  )
+  (text "Footprint(s) only" (at 27.94 160.02 0)
+    (effects (font (size 1.27 1.27)) (justify left bottom))
   )
   (text "Wake" (at 219.71 67.31 0)
@@
   (text "Programming" (at 121.92 69.85 0)
     (effects (font (size 2.54 2.54)) (justify left bottom))
+  )
+  (text "Footprint(s) only" (at 27.94 114.3 0)
+    (effects (font (size 1.27 1.27)) (justify left bottom))
   )
   (text "Flash" (at 194.31 138.43 0)
@@
   )
   (symbol (lib_id "Connector:Conn_01x02_Male") (at 31.75 102.87 0) (mirror y) (unit 1)
-    (in_bom yes) (on_board yes)
+    (in_bom no) (on_board yes)
     (property "Reference" "J3" (id 0) (at 31.115 97.79 0))
     (property "Value" "Conn_01x02_Male" (id 1) (at 31.115 100.33 0))
@@
   )
   (symbol (lib_id "Connector:Conn_01x02_Male") (at 57.15 148.59 0) (mirror y) (unit 1)
-    (in_bom yes) (on_board yes)
+    (in_bom no) (on_board yes)
     (property "Reference" "J6" (id 0) (at 55.88 143.51 0)
       (effects (font (size 1.27 1.27)) (justify right))
@@
   )
   (symbol (lib_id "Connector:Conn_01x04_Male") (at 31.75 34.29 0) (mirror y) (unit 1)
-    (in_bom yes) (on_board yes)
+    (in_bom no) (on_board yes)
     (property "Reference" "J2" (id 0) (at 27.94 26.67 0)
       (effects (font (size 1.27 1.27)) (justify right))
@@
   )
   (symbol (lib_id "Connector:Conn_01x02_Male") (at 55.88 102.87 0) (mirror y) (unit 1)
-    (in_bom yes) (on_board yes)
+    (in_bom no) (on_board yes)
     (property "Reference" "J4" (id 0) (at 55.245 97.79 0))
     (property "Value" "Conn_01x02_Male" (id 1) (at 55.245 100.33 0))
@@
   )
   (symbol (lib_id "Connector:Conn_01x02_Male") (at 31.75 148.59 0) (mirror y) (unit 1)
-    (in_bom yes) (on_board yes) (fields_autoplaced)
+    (in_bom no) (on_board yes) (fields_autoplaced)
     (property "Reference" "J5" (id 0) (at 31.115 143.51 0))
     (property "Value" "Conn_01x02_Male" (id 1) (at 31.115 146.05 0))
@@
   )
   (symbol (lib_id "Connector:Conn_01x07_Male") (at 102.87 50.8 0) (unit 1)
-    (in_bom yes) (on_board yes)
+    (in_bom no) (on_board yes)
     (property "Reference" "J1" (id 0) (at 103.505 38.1 0))
     (property "Value" "Conn_01x07_Male" (id 1) (at 107.95 50.8 90)
@@
       (effects (font (size 1.27 1.27)) hide)
     )
+    (property "Note" "Footprint only" (id 4) (at 102.87 50.8 0)
+      (effects (font (size 1.27 1.27)) hide)
+    )

Commit message: BOMing the place...
Parts:
- C7: Vendor (none) -> LCSC C14663
- C8: Vendor (none) -> LCSC C89246
- Q1: Vendor (none) -> LCSC C62892
- R1: Vendor (none) -> LCSC C22790
- R2: Vendor (none) -> LCSC C22935
- R3, R4, R6, R7: Vendor (none) -> LCSC C25804
- R5: Vendor (none) -> LCSC C8218
- U1: Vendor (none) -> LCSC C77967
- U2: Arrow Part Number SST25VF016B-50-4I-S2AF -> (none); Arrow Price/Stock https://www.arrow.com/en/products/sst25vf016b-50-4i-s2af/mi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 -> (none); Mouser Part Number 579-25VF016B5IS2AF -> (none); Mouser Price/Stock https://www.mouser.co.uk/ProductDetail/Microchip-Technology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 -> (none); Vendor (none) -> LCSC C68557
Changed lines of the file:
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@@
+      (effects (font (size 1.27 1.27)) hide)
+    )
+    (property "Vendor" "LCSC C62892" (id 4) (at 143.51 49.53 0)
       (effects (font (size 1.27 1.27)) hide)
     )
@@
     )
     (property "Datasheet" "~" (id 3) (at 217.17 127 0)
+      (effects (font (size 1.27 1.27)) hide)
+    )
+    (property "Vendor" "LCSC C8218" (id 4) (at 217.17 127 90)
       (effects (font (size 1.27 1.27)) hide)
     )
@@
       (effects (font (size 1.27 1.27)) hide)
     )
+    (property "Vendor" "LCSC C25804" (id 4) (at 207.01 44.45 90)
+      (effects (font (size 1.27 1.27)) hide)
+    )
     (pin "1")
     (pin "2")
@@
       (effects (font (size 1.27 1.27)) (justify left) hide)
     )
-    (property "Mouser Part Number" "579-25VF016B5IS2AF" (id 8) (at 215.9 134.62 0)
-      (effects (font (size 1.27 1.27)) (justify left) hide)
-    )
-    (property "Mouser Price/Stock" "https://www.mouser.co.uk/ProductDetail/Microchip-Technology/SST25VF016B-50-4I-S2AF?qs=1RUxC5ic%2FMoMGeEXhm8Oww%3D%3D" (id 9) (at 215.9 137.16 0)
-      (effects (font (size 1.27 1.27)) (justify left) hide)
-    )
-    (property "Arrow Part Number" "SST25VF016B-50-4I-S2AF" (id 10) (at 215.9 139.7 0)
-      (effects (font (size 1.27 1.27)) (justify left) hide)
-    )
-    (property "Arrow Price/Stock" "https://www.arrow.com/en/products/sst25vf016b-50-4i-s2af/microchip-technology?region=nac" (id 11) (at 215.9 142.24 0)
-      (effects (font (size 1.27 1.27)) (justify left) hide)
+    (property "Vendor" "LCSC C68557" (id 8) (at 185.42 121.92 0)
+      (effects (font (size 1.27 1.27)) hide)
     )
     (pin "1")
@@
       (effects (font (size 1.27 1.27)) hide)
     )
+    (property "Vendor" "LCSC C89246" (id 5) (at 223.52 43.18 0)
+      (effects (font (size 1.27 1.27)) hide)
+    )
     (pin "1")
     (pin "2")
@@
       (effects (font (size 1.27 1.27)) hide)
     )
+    (property "Vendor" "LCSC C25804" (id 4) (at 214.63 44.45 90)
+      (effects (font (size 1.27 1.27)) hide)
+    )
     (pin "1")
     (pin "2")
@@
     )
     (property "Datasheet" "http://rohmfs.rohm.com/en/products/databook/datasheet/discrete/transistor/digital/emh3t2r-e.pdf" (id 3) (at 148.59 55.88 0)
+      (effects (font (size 1.27 1.27)) hide)
+    )
+    (property "Vendor" "LCSC C62892" (id 4) (at 144.78 55.88 0)
       (effects (font (size 1.27 1.27)) hide)
     )
@@
       (effects (font (size 1.27 1.27)) hide)
     )
+    (property "Vendor" "LCSC C22790" (id 4) (at 195.58 60.96 90)
+      (effects (font (size 1.27 1.27)) hide)
+    )
     (pin "1")
     (pin "2")
@@
       (effects (font (size 1.27 1.27)) hide)
     )
+    (property "Vendor" "LCSC C14663" (id 4) (at 219.71 118.11 0)
+      (effects (font (size 1.27 1.27)) hide)
+    )
     (pin "1")
     (pin "2")
@@
       (effects (font (size 1.27 1.27)) hide)
     )
+    (property "Vendor" "LCSC C22935" (id 4) (at 210.82 78.74 90)
+      (effects (font (size 1.27 1.27)) hide)
+    )
     (pin "1")
     (pin "2")
@@
       (effects (font (size 1.27 1.27)) hide)
     )
+    (property "Vendor" "LCSC C25804" (id 4) (at 125.73 44.45 90)
+      (effects (font (size 1.27 1.27)) hide)
+    )
     (pin "1")
     (pin "2")
@@
     )
     (property "Datasheet" "~" (id 3) (at 156.21 54.61 0)
+      (effects (font (size 1.27 1.27)) hide)
+    )
+    (property "Vendor" "LCSC C25804" (id 4) (at 156.21 54.61 90)
       (effects (font (size 1.27 1.27)) hide)
     )
@@
       (effects (font (size 1.27 1.27)) hide)
     )
+    (property "Vendor" "LCSC C77967" (id 4) (at 250.19 68.58 0)
+      (effects (font (size 1.27 1.27)) hide)
+    )

Commit message: Tryin' a 8285 controller...
Parts:
- C3, C4: Vendor (none) -> LCSC C325468
- C5: value TBD (NC) -> 1uf; Vendor (none) -> LCSC C559769
- C6: Vendor (none) -> LCSC C559769
- J9: Vendor (none) -> LCSC C145956,
Changed lines of the file:
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@@
+      (effects (font (size 1.27 1.27)) hide)
+    )
+    (property "Vendor" "LCSC C325468" (id 4) (at 220.98 96.52 0)
       (effects (font (size 1.27 1.27)) hide)
     )
@@
     )
     (property "Datasheet" "~" (id 3) (at 200.66 96.52 0)
+      (effects (font (size 1.27 1.27)) hide)
+    )
+    (property "Vendor" "LCSC C325468" (id 4) (at 200.66 96.52 0)
       (effects (font (size 1.27 1.27)) hide)
     )
@@
     )
     (property "Datasheet" "~" (id 3) (at 255.27 35.56 0)
+      (effects (font (size 1.27 1.27)) hide)
+    )
+    (property "Vendor" "LCSC C559769" (id 4) (at 255.27 35.56 0)
       (effects (font (size 1.27 1.27)) hide)
     )
@@
       (effects (font (size 1.27 1.27)) hide)
     )
+    (property "Vendor" "LCSC C145956, " (id 4) (at 124.46 88.9 0)
+      (effects (font (size 1.27 1.27)) hide)
+    )
     (pin "1")
     (pin "2")
@@
     (in_bom yes) (on_board yes)
     (property "Reference" "C5" (id 0) (at 240.665 33.655 0))
-    (property "Value" "TBD (NC)" (id 1) (at 247.65 38.1 0))
+    (property "Value" "1uf" (id 1) (at 247.65 38.1 0))
     (property "Footprint" "Capacitor_SMD:C_0603_1608Metric" (id 2) (at 241.6048 31.75 0)
       (effects (font (size 1.27 1.27)) hide)
     )
     (property "Datasheet" "~" (id 3) (at 242.57 35.56 0)
+      (effects (font (size 1.27 1.27)) hide)
+    )
+    (property "Vendor" "LCSC C559769" (id 4) (at 242.57 35.56 0)
       (effects (font (size 1.27 1.27)) hide)
     )
@@
     )
     (path "/dd3aca8e-7f28-4d18-b0e6-f55f5e1454ac"
-      (reference "C5") (unit 1) (value "TBD (NC)") (footprint "Capacitor_SMD:C_0603_1608Metric")
+      (reference "C5") (unit 1) (value "1uf") (footprint "Capacitor_SMD:C_0603_1608Metric")
     )
     (path "/3cf6c72c-3d00-4eb6-af3e-f7072449457f"
