File: Hardware/Proto.kicad_pcb (KiCad board)
At the start: 2 copper layers, 34 x 34 mm, 12 parts, among them J2 Conn_01x04_Male, J3 Conn_01x02_Male, J4 Conn_01x02_Male, J5 Conn_01x02_Male, J6 Conn_01x02_Male, J9 Conn_01x04_MountingPin

Commit message: .........
Parts:
- J9: value Conn_01x04_MountingPin -> QWIIC_Stackable; footprint Tinker:JST_SH_SM04B-SRSS-TB_1x04-1MP_P1.00mm_Horizontal -> Tinker:QWIIC_Stackable
Connections:
- net 2v7 renamed Vcc?
Routing:
- net UD-: track 1.48 -> 0.00 mm
- net UD+: track 1.48 -> 0.00 mm
Other:
- board text added: "I2C"

Commit message: tweakin' not twerkin
Parts:
- removed the REF** at (108.2, 72.9)
- added G***: LOGO, Tinker:NerdMage, F.Cu at (108.0, 72.9)
