File: Hardware/USB-PD Board.kicad_pcb (KiCad board)
At the start: 2 copper layers, 34 x 34 mm, 52 parts, among them J1 USB_C_Receptacle_USB2.0, J2 Conn_01x04_Male, J3 Conn_01x02_Male, J4 Conn_01x02_Male, J5 Conn_01x02_Male, J6 Conn_01x02_Male, J7 Conn_01x08_Male, Q1 DMP3013SFV, Q2 DMP3013SFV, U3 STUSB4500QTR

Commit message: ...
Parts:
- added C1: 22uf, Tinker:CP_EIA-6032-28-Tantalumm_HandSolder, F.Cu at (108.4, 78.0)
- added C6: 1.0uF, Capacitor_SMD:C_0603_1608Metric, F.Cu at (110.2, 92.1)
- added U2: R1501J033B-T1-JE, Tinker:R1501J033BT1JE, F.Cu at (108.4, 85.9)
- renumbered U3 to U1
Routing:
- net Vsec: track 11.3 -> 24.0 mm
- net Vout: track 56.8 -> 63.4 mm

Commit message: Nearly there...
Parts:
- removed R15: 1k, Resistor_SMD:R_0603_1608Metric
- added R18: 1k, Resistor_SMD:R_0603_1608Metric, F.Cu at (90.0, 90.6)
- added SW1: SW_Push, Tinker:SW_Push_TS273014TP, F.Cu at (93.7, 88.1)
- D6: value blue -> yellow
- J7: footprint Connector_PinHeader_1.27mm:PinHeader_2x04_P1.27mm_Vertical -> Tinker:PinHeader_2x04_P1.27mm_Vertical
- Q1, Q2: footprint Package_SON:Diodes_PowerDI3333-8 -> Tinker:Diodes_PowerDI3333-8
- moved D8 9.99 mm to (102.0, 92.1)
- moved R14 6.67 mm to (102.0, 90.6), turned to 0 degrees
- moved D7 5.82 mm to (98.0, 92.1)
- moved C6 4.92 mm to (105.2, 92.1), turned to 180 degrees
- moved R7 3.69 mm to (99.4, 87.2), turned to 180 degrees
- moved D9 3.65 mm to (90.0, 92.1)
- moved R8 3.41 mm to (99.4, 89.0), turned to 180 degrees
- moved R13 2.70 mm to (98.0, 90.6), turned to 0 degrees
- moved R12 2.69 mm to (94.0, 90.6), turned to 0 degrees
- moved D6 2.24 mm to (94.0, 92.1)
- moved JP2 0.80 mm to (84.4, 78.4)
- moved JP3 0.80 mm to (85.9, 78.4)
- moved JP4 0.80 mm to (87.4, 78.4)
- moved R3 0.80 mm to (84.4, 81.3)
- moved R4 0.80 mm to (85.9, 81.3)
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- renumbered R3 to R10, R4 to R11, R7 to R16, R5 to R17, R10 to R3, R9 to R4, R11 to R5, R16 to R7, R17 to R8, R8 to R9
Connections:
- D9 pad 1: Net-(D9-Pad1) -> GND
- D9 pad 2: 2v7 -> Net-(D9-Pad2)
- J7 pad 1: SDA -> RESET
- J7 pad 2: SCL -> ATTACH
- J7 pad 3: ALERT -> SCL
- J7 pad 4: RESET -> POWER_OK2
- J7 pad 5: GPIO -> SDA
- J7 pad 6: ATTACH -> POWER_OK3
- J7 pad 7: POWER_OK3 -> ALERT
- J7 pad 8: POWER_OK2 -> GPIO
- R12 pad 1: GPIO -> ATTACH
- R13 pad 1: POWER_OK3 -> POWER_OK2
- R14 pad 1: POWER_OK2 -> POWER_OK3
Routing:
- net Vbus: track 41.5 -> 53.8 mm, vias 2 -> 4
- net 2v7: track 51.4 -> 40.7 mm, vias 4 -> 2
- net GPIO: track 25.4 -> 15.9 mm
- net RESET: track 8.21 -> 17.1 mm, vias 0 -> 2
- net ALERT: track 16.5 -> 20.3 mm
- net SDA: track 11.8 -> 15.3 mm
- net SCL: track 8.77 -> 11.7 mm
- net ATTACH: track 18.8 -> 15.9 mm
- net Vout: track 63.4 -> 66.1 mm
- net POWER_OK2: track 20.6 -> 23.0 mm, vias 2 -> 3
- net UD-: track 38.7 -> 41.1 mm
- net UD+: track 37.6 -> 39.6 mm
- net Net-(D9-Pad2): track 0.00 -> 1.52 mm
- net Net-(D9-Pad1): track 1.39 -> 0.00 mm
- net POWER_OK3: track 20.5 -> 21.8 mm, vias 2 -> 3
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Other:
- board text added: "PWR"
- board text added: "RESET"
- board text added: "USB PD"
- board text added: "{dblquote}Universal{dblquote}"
- board text removed: "GPIO"
- board text removed: "POK3"
- board text removed: "{dblquote}Universal{dblquote} USB-C Board"

Commit message: buncha tweaks...
Other:
- board text added: "USB-C PD"
- board text removed: "USB PD"

Commit message: just fiddlin' 'round...
Parts:
- J1: value USB_C_Receptacle_USB2.0 -> USB_C_Receptacle
Other:
- board text added: "POK3"

Commit message: Documentation...
Parts:
- renumbered D9 to D6, D6 to D7, D7 to D8, D8 to D9

Commit message: Tinkerin' + RESET & LED on Programmer...
Other:
- board text added: "NerdMage Modules ${TITLE} (v${REVISION})"
- board text removed: "NerdMage Modules (v0.0.1)"
Changed lines of the file:
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@@
   (paper "A4")
   (title_block
-    (title "USB-C (PD) Board")
-    (rev "0.0.1")
+    (title "USB-PD Board")
+    (rev "0.0.9")
     (company "The Nerd Mage")
   )
@@
   (gr_line (start 120 78) (end 80 78) (layer "User.3") (width 0.15))
   (gr_line (start 80 92) (end 120 92) (layer "User.9") (width 0.15))
-  (gr_text "NerdMage Modules (v0.0.1)" (at 100 74.8) (layer "B.SilkS")
+  (gr_text "NerdMage Modules\n${TITLE} (v${REVISION})" (at 100 76) (layer "B.SilkS")
     (effects (font (size 1 1) (thickness 0.15)) (justify mirror))
   )
@@
     (effects (font (size 0.6 0.6) (thickness 0.125)) (justify mirror))
   )
-  (gr_text "S. A. Miller 2023" (at 100 90) (layer "B.SilkS")
+  (gr_text "S. A. Miller 2023" (at 100 79) (layer "B.SilkS")
     (effects (font (size 1 1) (thickness 0.15)) (justify mirror))
   )

Commit message: Expanding on the Controller Board functionality...
Routing:
- net GND: vias 11 -> 2
Changed lines of the file:
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@@
       (effects (font (size 1.27 1.27) (thickness 0.254)))
     )
+    (fp_line (start 3.3 2.025) (end 3.3 1.2) (layer "F.SilkS") (width 0.2))
     (fp_line (start -3.3 1.2) (end -3.3 2.025) (layer "F.SilkS") (width 0.2))
     (fp_line (start -3.3 2.025) (end 3.3 2.025) (layer "F.SilkS") (width 0.2))
-    (fp_line (start 3.3 2.025) (end 3.3 1.2) (layer "F.SilkS") (width 0.2))
-    (fp_line (start 3.4 -5.275) (end 3.4 5.275) (layer "F.CrtYd") (width 0.1))
     (fp_line (start -3.4 -5.275) (end 3.4 -5.275) (layer "F.CrtYd") (width 0.1))
+    (fp_line (start 3.4 -5.275) (end 3.4 5.275) (layer "F.CrtYd") (width 0.1))
     (fp_line (start 3.4 5.275) (end -3.4 5.275) (layer "F.CrtYd") (width 0.1))
     (fp_line (start -3.4 5.275) (end -3.4 -5.275) (layer "F.CrtYd") (width 0.1))
     (fp_line (start 3.3 -4.075) (end 3.3 2.025) (layer "F.Fab") (width 0.1))
     (fp_line (start -3.3 -4.075) (end 3.3 -4.075) (layer "F.Fab") (width 0.1))
-    (fp_line (start -3.3 2.025) (end -3.3 -4.075) (layer "F.Fab") (width 0.1))
     (fp_line (start 3.3 2.025) (end -3.3 2.025) (layer "F.Fab") (width 0.1))
+    (fp_line (start -3.3 2.025) (end -3.3 -4.075) (layer "F.Fab") (width 0.1))
     (pad "1" smd rect (at -2.54 4.075) (size 0.8 2.5) (layers "F.Cu" "F.Paste" "F.Mask")
       (net 20 "Vout") (pinfunction "VDD") (pintype "passive"))
@@
     (pad "5" smd rect (at 2.54 4.075) (size 0.8 2.5) (layers "F.Cu" "F.Paste" "F.Mask")
       (net 23 "Vsec") (pinfunction "VOUT") (pintype "passive"))
+    (pad "6" thru_hole roundrect (at 2 -2.175) (size 1 1) (drill 0.4) (layers *.Cu) (roundrect_rratio 0.25)
+      (net 19 "GND") (pinfunction "GND_3") (pintype "passive"))
+    (pad "6" thru_hole roundrect (at 2 -4.175) (size 1 1) (drill 0.4) (layers *.Cu) (roundrect_rratio 0.25)
+      (net 19 "GND") (pinfunction "GND_3") (pintype "passive"))
+    (pad "6" thru_hole roundrect (at 2 -0.175) (size 1 1) (drill 0.4) (layers *.Cu) (roundrect_rratio 0.25)
+      (net 19 "GND") (pinfunction "GND_3") (pintype "passive"))
     (pad "6" smd rect (at 0 -2.175) (size 6 6) (layers "F.Cu" "F.Paste" "F.Mask")
       (net 19 "GND") (pinfunction "GND_3") (pintype "passive"))
+    (pad "6" thru_hole roundrect (at 0 -2.175) (size 1 1) (drill 0.4) (layers *.Cu) (roundrect_rratio 0.25)
+      (net 19 "GND") (pinfunction "GND_3") (pintype "passive"))
+    (pad "6" thru_hole roundrect (at 0 -0.175) (size 1 1) (drill 0.4) (layers *.Cu) (roundrect_rratio 0.25)
+      (net 19 "GND") (pinfunction "GND_3") (pintype "passive"))
+    (pad "6" thru_hole roundrect (at 0 -4.175) (size 1 1) (drill 0.4) (layers *.Cu) (roundrect_rratio 0.25)
+      (net 19 "GND") (pinfunction "GND_3") (pintype "passive"))
+    (pad "6" thru_hole roundrect (at -2 -2.175) (size 1 1) (drill 0.4) (layers *.Cu) (roundrect_rratio 0.25)
+      (net 19 "GND") (pinfunction "GND_3") (pintype "passive"))
+    (pad "6" thru_hole roundrect (at -2 -4.175) (size 1 1) (drill 0.4) (layers *.Cu) (roundrect_rratio 0.25)
+      (net 19 "GND") (pinfunction "GND_3") (pintype "passive"))
+    (pad "6" thru_hole roundrect (at -2 -0.175) (size 1 1) (drill 0.4) (layers *.Cu) (roundrect_rratio 0.25)
+      (net 19 "GND") (pinfunction "GND_3") (pintype "passive"))
     (model "${KICAD6_3DMODEL_DIR}/Package_TO_SOT_SMD.3dshapes/TO-252-5_TabPin6.step"
       (offset (xyz 0 0 0))
@@
   (segment (start 105.469465 96.509295) (end 105.096965 96.881795) (width 0.25) (layer "F.Cu") (net 19))
   (segment (start 94.143035 101.06) (end 94.153035 101.05) (width 0.25) (layer "F.Cu") (net 19))
-  (via (at 110.4 81.725) (size 0.8) (drill 0.4) (layers "F.Cu" "B.Cu") (net 19))
   (via (at 93.9 81.5) (size 1) (drill 0.5) (layers "F.Cu" "B.Cu") (net 19))
-  (via (at 108.4 83.725) (size 0.8) (drill 0.4) (layers "F.Cu" "B.Cu") (net 19))
-  (via (at 108.4 85.725) (size 0.8) (drill 0.4) (layers "F.Cu" "B.Cu") (net 19))
-  (via (at 110.4 85.725) (size 0.8) (drill 0.4) (layers "F.Cu" "B.Cu") (net 19))
-  (via (at 108.4 81.725) (size 0.8) (drill 0.4) (layers "F.Cu" "B.Cu") (net 19))
-  (via (at 106.4 81.725) (size 0.8) (drill 0.4) (layers "F.Cu" "B.Cu") (net 19))
-  (via (at 106.4 85.725) (size 0.8) (drill 0.4) (layers "F.Cu" "B.Cu") (net 19))
   (via (at 97.475375 85.940367) (size 0.5) (drill 0.3) (layers "F.Cu" "B.Cu") (free) (net 19))
-  (via (at 106.4 83.725) (size 0.8) (drill 0.4) (layers "F.Cu" "B.Cu") (net 19))
-  (via (at 110.4 83.725) (size 0.8) (drill 0.4) (layers "F.Cu" "B.Cu") (net 19))
   (segment (start 108.633618 94.58) (end 108.633618 93.393618) (width 0.8) (layer "F.Cu") (net 20))
   (segment (start 105.86 93.16) (end 106.02 93.32) (width 0.8) (layer "F.Cu") (net 20))
