File: Hardware/USB-PD Proto.kicad_sch (KiCad schematic)
At the start: 7 parts, among them J1 Conn_01x08_Male, J2 Conn_01x04_Male, J3 Conn_01x02_Male, J4 Conn_01x02_Male, J5 Conn_01x02_Male, J6 Conn_01x02_Male, J9 QWIIC_Stackable

Commit message: ... :| ...
Parts:
- J1: now left out of the parts list
Changed lines of the file:
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@@
   )
   (symbol (lib_id "Connector:Conn_01x08_Male") (at 142.24 90.17 0) (mirror y) (unit 1)
-    (in_bom yes) (on_board yes) (fields_autoplaced)
+    (in_bom no) (on_board yes) (fields_autoplaced)
     (property "Reference" "J1" (id 0) (at 143.51 91.4399 0)
       (effects (font (size 1.27 1.27)) (justify right))

Commit message: tweaks...
Parts:
- J1: LCSC (none) -> C2881786 + C2684732
Changed lines of the file:
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@@
+      (effects (font (size 1.27 1.27)) hide)
+    )
+    (property "LCSC" "C2881786 + C2684732" (id 4) (at 142.24 90.17 0)
       (effects (font (size 1.27 1.27)) hide)
     )

Commit message: Documentation
Parts:
- renumbered J1 to J7
Changed lines of the file:
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@@
   (symbol (lib_id "Connector:Conn_01x08_Male") (at 142.24 90.17 0) (mirror y) (unit 1)
     (in_bom no) (on_board yes) (fields_autoplaced)
-    (property "Reference" "J1" (id 0) (at 143.51 91.4399 0)
+    (property "Reference" "J7" (id 0) (at 143.51 91.4399 0)
       (effects (font (size 1.27 1.27)) (justify right))
     )
@@
       (reference "#PWR0124") (unit 1) (value "GND") (footprint "")
     )
-    (path "/df99fb81-9cb2-43d0-b2ba-52fcac23a406"
-      (reference "J1") (unit 1) (value "Conn_01x08_Male") (footprint "Tinker:PinHeader_2x04_P1.27mm_Vertical")
-    )
     (path "/ce562b82-4d15-4512-9ef8-80a89b06889d"
       (reference "J2") (unit 1) (value "Conn_01x04_Male") (footprint "Tinker:PinHeader_1x04_P2.54mm_Vertical")
@@
       (reference "J6") (unit 1) (value "Conn_01x02_Male") (footprint "Tinker:PinHeader_1x02_P2.54mm_Vertical")
     )
+    (path "/df99fb81-9cb2-43d0-b2ba-52fcac23a406"
+      (reference "J7") (unit 1) (value "Conn_01x08_Male") (footprint "Tinker:PinHeader_2x04_P1.27mm_Vertical")
+    )
     (path "/b8a785f2-9322-4569-b066-f0e9fc64eafd"

Commit message: Tinkerin' + RESET & LED on Programmer...
Other:
- note added: "Control"
- note added: "QWIIC"
- moved on the sheet: J3, J4, J5, J6, J7, J9

Commit message: Uber Rework!
Parts:
- added J1: Conn_01x07_Male, Tinker:Board_Stacker_7, symbol Connector:Conn_01x07_Male
- J2: footprint Tinker:PinHeader_1x04_P2.54mm_Vertical -> Tinker:Board_Stacker_4
- J3, J4, J5, J6: footprint Tinker:PinHeader_1x02_P2.54mm_Vertical -> Tinker:Board_Stacker_2
- J9: footprint Tinker:QWIIC_Stackable -> Tinker:QWIIC_Stack_II
Connections:
- net GND: now also J1.4 (Pin_4)
- new net +3V3: J1.1 (Pin_1)
- new net DTR: J1.5 (Pin_5)
- new net IO1: J1.3 (Pin_3)
- new net IO3: J1.2 (Pin_2)
- new net RST: J1.7 (Pin_7)
- new net RTS: J1.6 (Pin_6)
