File: Hardware/Ethernet-S.kicad_sch (KiCad schematic)
At the start: 15 parts, among them J1 Conn_01x07_Male, J10 SPI, J11 Conn_01x10_Male, J12 Conn_01x04_Male, J2 Conn_01x04_Male, J3 Conn_01x02_Male, J4 Conn_01x02_Male, J5 Conn_01x02_Male, J6 Conn_01x02_Male, J7 Conn_01x08_Male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

Commit message: Buncha cosmetic stuff...
Parts:
- removed J10: SPI, bare-footprints:8 pin jst 1.25 vertical, symbol Connector_Generic_MountingPin:Conn_01x08_MountingPin
- removed J11: Conn_01x10_Male, Tinker:PinHeader_1x10_P1.27mm_Vertical, symbol Connector:Conn_01x10_Male
- removed J12: Conn_01x04_Male, Tinker:PinHeader_1x04_P1.27mm_Vertical, symbol Connector:Conn_01x04_Male
- removed J8: SPI, Tinker:PinHeader_1x08_P1.27mm_Vertical, symbol Connector:Conn_01x08_Male
- removed R10, R9: 470R, Resistor_SMD:R_0603_1608Metric, symbol Device:R_US
- removed RJ45-1: ARJM11D7114ABEW2, Tinker:CONN_ARJM11D7-114-AB-EW2_ABR, symbol ARJM11D7-114-AB-EW2_ABR:ARJM11D7114ABEW2
Connections:
- net ATTACH is gone; now on net SCLK: J7.2 (Pin_2)
- net GPIO is gone; now on net ~{SCS}: J7.8 (Pin_8)
- net POWER_OK2 is gone; now on net MISO: J7.4 (Pin_4)
- net POWER_OK3 is gone; now on net MOSI: J7.6 (Pin_6)
- net ALERT: no longer names the net of J7.7 (Pin_7)
- net RESET renamed WIZ_RST
- no-connect marks 2 -> 0
Other:
- note added: "Board-to-Board"
- note added: "SPI"
- note removed: "Control"
- note removed: "Ethernet Connector"
- note removed: "SPI JST"
- note removed: "SPI pin"
- moved on the sheet: J7, J9

Commit message: Starting on POE
Parts:
- added ?: AG9912M, symbol AG9912M:AG9912M
- added ?: AG9912-MTB, symbol AG9912-MTB:AG9912-MTB
- added ?: Ag9912LP, symbol Ag9912LP:Ag9912LP
Changed lines of the file:
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@@
     )
+  )
+  (symbol (lib_id "AG9912M:AG9912M") (at 147.32 86.36 0) (unit 1)
+    (in_bom yes) (on_board yes) (fields_autoplaced)
+    (property "Reference" "?" (id 0) (at 163.83 73.66 0))
+    (property "Value" "AG9912M" (id 1) (at 163.83 76.2 0))
+    (property "Footprint" "" (id 2) (at 147.32 86.36 0)
+      (effects (font (size 1.27 1.27)) hide)
+    )
+    (property "Datasheet" "" (id 3) (at 147.32 86.36 0)
+      (effects (font (size 1.27 1.27)) hide)
+    )
+    (property "Reference_1" "IC" (id 4) (at 163.83 78.74 0))
+    (property "Value_1" "AG9912M" (id 5) (at 163.83 81.28 0))
+    (property "Footprint_1" "AG9912M" (id 6) (at 176.53 181.28 0)
+      (effects (font (size 1.27 1.27)) (justify left top) hide)
+    )
+    (property "Datasheet_1" "https://www.mouser.com/datasheet/2/1048/Ag9900M-datasheet-ultra-miniature-isolated-Power-o-1804309.pdf" (id 7) (at 176.53 281.28 0)
+      (effects (font (size 1.27 1.27)) (justify left top) hide)
+    )
+    (property "Height" "13.85" (id 8) (at 176.53 481.28 0)
+      (effects (font (size 1.27 1.27)) (justify left top) hide)
+    )
+    (property "Manufacturer_Name" "Silvertel" (id 9) (at 176.53 581.28 0)
+      (effects (font (size 1.27 1.27)) (justify left top) hide)
+    )
+    (property "Manufacturer_Part_Number" "AG9912M" (id 10) (at 176.53 681.28 0)
+      (effects (font (size 1.27 1.27)) (justify left top) hide)
+    )
+    (property "Mouser Part Number" "480-AG9912M" (id 11) (at 176.53 781.28 0)
+      (effects (font (size 1.27 1.27)) (justify left top) hide)
+    )
+    (property "Mouser Price/Stock" "https://www.mouser.co.uk/ProductDetail/Silvertel/Ag9912M?qs=OlC7AqGiEDkycJrCl2xLig%3D%3D" (id 12) (at 176.53 881.28 0)
+      (effects (font (size 1.27 1.27)) (justify left top) hide)
+    )
+    (property "Arrow Part Number" "" (id 13) (at 176.53 981.28 0)
+      (effects (font (size 1.27 1.27)) (justify left top) hide)
+    )
+    (property "Arrow Price/Stock" "" (id 14) (at 176.53 1081.28 0)
+      (effects (font (size 1.27 1.27)) (justify left top) hide)
+    )
+    (pin "1")
+    (pin "2")
+    (pin "3")
+    (pin "4")
+    (pin "5")
+    (pin "6")
+    (pin "7")
+    (pin "8")
   )
   (symbol (lib_id "Connector:Conn_01x02_Male") (at 33.02 128.27 0) (mirror y) (unit 1)
@@
     (pin "2")
   )
+  (symbol (lib_id "AG9912-MTB:AG9912-MTB") (at 148.59 43.18 0) (unit 1)
+    (in_bom yes) (on_board yes) (fields_autoplaced)
+    (property "Reference" "?" (id 0) (at 162.56 30.48 0))
+    (property "Value" "AG9912-MTB" (id 1) (at 162.56 33.02 0))
+    (property "Footprint" "" (id 2) (at 148.59 43.18 0)
+      (effects (font (size 1.27 1.27)) hide)
+    )
+    (property "Datasheet" "" (id 3) (at 148.59 43.18 0)
+      (effects (font (size 1.27 1.27)) hide)
+    )
+    (property "Reference_1" "PS" (id 4) (at 162.56 35.56 0))
+    (property "Value_1" "AG9912-MTB" (id 5) (at 162.56 38.1 0))
+    (property "Footprint_1" "AG9912MTB" (id 6) (at 172.72 138.1 0)
+      (effects (font (size 1.27 1.27)) (justify left top) hide)
+    )
+    (property "Datasheet_1" "https://silvertel.com/images/datasheets/Ag9900M-datasheet-ultra-miniature-isolated-Power-over-Ethernet-POE-module.pdf" (id 7) (at 172.72 238.1 0)
+      (effects (font (size 1.27 1.27)) (justify left top) hide)
+    )
+    (property "Height" "13.9" (id 8) (at 172.72 438.1 0)
+      (effects (font (size 1.27 1.27)) (justify left top) hide)
+    )
+    (property "Manufacturer_Name" "Silvertel" (id 9) (at 172.72 538.1 0)
+      (effects (font (size 1.27 1.27)) (justify left top) hide)
+    )
+    (property "Manufacturer_Part_Number" "AG9912-MTB" (id 10) (at 172.72 638.1 0)
+      (effects (font (size 1.27 1.27)) (justify left top) hide)
+    )
+    (property "Mouser Part Number" "480-AG9912-MTB" (id 11) (at 172.72 738.1 0)
+      (effects (font (size 1.27 1.27)) (justify left top) hide)
+    )
+    (property "Mouser Price/Stock" "https://www.mouser.co.uk/ProductDetail/Silvertel/AG9912-MTB?qs=vvQtp7zwQdOqoQu0dV4pzA%3D%3D" (id 12) (at 172.72 838.1 0)
+      (effects (font (size 1.27 1.27)) (justify left top) hide)
+    )
+    (property "Arrow Part Number" "" (id 13) (at 172.72 938.1 0)
+      (effects (font (size 1.27 1.27)) (justify left top) hide)
+    )
+    (property "Arrow Price/Stock" "" (id 14) (at 172.72 1038.1 0)
+      (effects (font (size 1.27 1.27)) (justify left top) hide)
+    )
+    (pin "1")
+    (pin "2")
+    (pin "3")
+    (pin "4")
+    (pin "5")
+  )
   (symbol (lib_id "power:GND") (at 93.98 44.45 0) (unit 1)
     (in_bom yes) (on_board yes)
@@
     )
     (pin "1")
+  )
+  (symbol (lib_id "Ag9912LP:Ag9912LP") (at 147.32 63.5 0) (unit 1)
+    (in_bom yes) (on_board yes) (fields_autoplaced)
+    (property "Reference" "?" (id 0) (at 163.83 50.8 0))
+    (property "Value" "Ag9912LP" (id 1) (at 163.83 53.34 0))
+    (property "Footprint" "" (id 2) (at 147.32 63.5 0)
+      (effects (font (size 1.27 1.27)) hide)
+    )
+    (property "Datasheet" "" (id 3) (at 147.32 63.5 0)
+      (effects (font (size 1.27 1.27)) hide)
+    )
+    (property "Reference_1" "IC" (id 4) (at 163.83 55.88 0))
+    (property "Value_1" "Ag9912LP" (id 5) (at 163.83 58.42 0))
+    (property "Footprint_1" "Ag9912LP" (id 6) (at 176.53 158.42 0)
+      (effects (font (size 1.27 1.27)) (justify left top) hide)
+    )
+    (property "Datasheet_1" "https://au.mouser.com/datasheet/2/1048/Ag9900M-datasheet-ultra-miniature-isolated-Power-o-1804309.pdf" (id 7) (at 176.53 258.42 0)
+      (effects (font (size 1.27 1.27)) (justify left top) hide)
+    )
+    (property "Height" "8" (id 8) (at 176.53 458.42 0)
+      (effects (font (size 1.27 1.27)) (justify left top) hide)
+    )
+    (property "Manufacturer_Name" "Silvertel" (id 9) (at 176.53 558.42 0)
+      (effects (font (size 1.27 1.27)) (justify left top) hide)
+    )
+    (property "Manufacturer_Part_Number" "Ag9912LP" (id 10) (at 176.53 658.42 0)
+      (effects (font (size 1.27 1.27)) (justify left top) hide)
+    )
+    (property "Mouser Part Number" "480-AG9912LP" (id 11) (at 176.53 758.42 0)
+      (effects (font (size 1.27 1.27)) (justify left top) hide)
+    )
+    (property "Mouser Price/Stock" "https://www.mouser.co.uk/ProductDetail/Silvertel/Ag9912LP?qs=OlC7AqGiEDllGSVQiYaPRA%3D%3D" (id 12) (at 176.53 858.42 0)
+      (effects (font (size 1.27 1.27)) (justify left top) hide)
+    )
+    (property "Arrow Part Number" "" (id 13) (at 176.53 958.42 0)
+      (effects (font (size 1.27 1.27)) (justify left top) hide)
+    )
+    (property "Arrow Price/Stock" "" (id 14) (at 176.53 1058.42 0)
+      (effects (font (size 1.27 1.27)) (justify left top) hide)
+    )
+    (pin "1")
+    (pin "2")
+    (pin "3")
+    (pin "4")
+    (pin "5")
+    (pin "6")
+    (pin "7")
+    (pin "8")
   )
   (symbol (lib_id "power:GND") (at 48.26 175.26 0) (mirror y) (unit 1)
@@
       (reference "#PWR0124") (unit 1) (value "GND") (footprint "")
     )
+    (path "/01b16456-6f09-4277-ac34-8974127fabd4"
+      (reference "?") (unit 1) (value "AG9912M") (footprint "")
+    )
+    (path "/4d8f25fe-2f5f-46b8-8a1c-ef90cd7e583d"
+      (reference "?") (unit 1) (value "AG9912-MTB") (footprint "")
+    )
+    (path "/9449d9c7-a361-4341-829c-2ab5d84fb54e"
+      (reference "?") (unit 1) (value "Ag9912LP") (footprint "")
+    )
     (path "/a0724c5c-eedb-4795-8cf2-007c21e2562f"
