File: Hardware/Ethernet-POE-S.kicad_pcb (KiCad board)
At the start: 2 copper layers, 34 x 34 mm, 14 parts, among them J10 Conn_01x02_Male, J11 Conn_01x02_Male, J3 Conn_01x02_Male, J4 Conn_01x02_Male, J5 Conn_01x02_Male, J6 Conn_01x02_Male, J7 Conn_01x08_Male, J9 QWIIC_Stackable

Commit message: Some randomness...
Other:
- board text added: "${TITLE} Board"
Changed lines of the file:
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@@
     (effects (font (size 0.6 0.6) (thickness 0.125)))
+  )
+  (gr_text "${TITLE} Board" (at 100.078744 111.716711) (layer "F.SilkS")
+    (effects (font (size 1 1) (thickness 0.15)))
   )
   (gr_text "GND" (at 86 108.7) (layer "F.SilkS")

Commit message: whole bunche cleanup...
Parts:
- moved REF** 0.23 mm to (109.0, 87.0)
- moved G*** 0.10 mm to (91.0, 86.0)
Other:
- outline, holes or cut-outs redrawn
Changed lines of the file:
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@@
   )
   (footprint "Tinker:DagNabbit" (layer "F.Cu")
-    (at 109.037169 87.226251)
+    (at 109 87)
     (attr smd board_only)
     (fp_text reference "REF**" (at 0 -8.08 unlocked) (layer "F.SilkS") hide
@@
   )
   (footprint "Tinker:NerdMage" (layer "F.Cu")
-    (at 91 85.9)
+    (at 91 86)
     (attr board_only exclude_from_pos_files exclude_from_bom)
     (fp_text reference "G***" (at 0 3.81) (layer "F.SilkS") hide
@@
       ) (layer "F.SilkS") (width 0) (fill solid))
   )
-  (gr_line (start 92 110) (end 92 90) (layer "Edge.Cuts") (width 0.05))
+  (gr_line (start 92 111) (end 92 89) (layer "Edge.Cuts") (width 0.05))
   (gr_line (start 117 86) (end 117 114) (layer "Edge.Cuts") (width 0.1))
-  (gr_line (start 108 90) (end 108 110) (layer "Edge.Cuts") (width 0.05))
+  (gr_line (start 108 89) (end 108 111) (layer "Edge.Cuts") (width 0.05))
   (gr_arc (start 86 117) (mid 83.87868 116.12132) (end 83 114) (layer "Edge.Cuts") (width 0.1))
   (gr_arc (start 83 86) (mid 83.87868 83.87868) (end 86 83) (layer "Edge.Cuts") (width 0.1))
-  (gr_line (start 92 90) (end 108 90) (layer "Edge.Cuts") (width 0.05))
+  (gr_line (start 92 89) (end 108 89) (layer "Edge.Cuts") (width 0.05))
   (gr_line (start 86 83) (end 114 83) (layer "Edge.Cuts") (width 0.1))
   (gr_line (start 114 117) (end 86 117) (layer "Edge.Cuts") (width 0.05))
@@
   (gr_arc (start 114 83) (mid 116.12132 83.87868) (end 117 86) (layer "Edge.Cuts") (width 0.1))
   (gr_arc (start 117 114) (mid 116.12132 116.12132) (end 114 117) (layer "Edge.Cuts") (width 0.1))
-  (gr_line (start 92 110) (end 108 110) (layer "Edge.Cuts") (width 0.05))
+  (gr_line (start 92 111) (end 108 111) (layer "Edge.Cuts") (width 0.05))
   (gr_text "Stacked Rabbit\n${TITLE} (v${REVISION})" (at 100 85) (layer "B.SilkS")
     (effects (font (size 1 1) (thickness 0.15)) (justify mirror))
@@
     (effects (font (size 0.6 0.6) (thickness 0.125)))
   )
-  (gr_text "${TITLE} Board" (at 100.078744 111.716711) (layer "F.SilkS")
+  (gr_text "${TITLE} Board" (at 110 100 90) (layer "F.SilkS")
     (effects (font (size 1 1) (thickness 0.15)))
   )
