File: Hardware/Ethernet-POE-WIP.kicad_pcb (KiCad board)
At the start: 2 copper layers, 34 x 34 mm, 18 parts, among them J3 Conn_01x02_Male, J4 Conn_01x02_Male, J5 Conn_01x02_Male, J6 Conn_01x02_Male, J7 Conn_01x08_Male, J9 QWIIC_Stackable

Commit message: More on POE...
Parts:
- added J10: Conn_01x02_Male, Tinker:Board_Stacker_2, F.Cu at (90.7, 114.0)
- added J11: Conn_01x02_Male, Tinker:Board_Stacker_2, F.Cu at (108.1, 114.0)
Routing:
- net VB2: track 0.00 -> 12.7 mm
- net VA1: track 0.00 -> 12.7 mm
- net VB1: track 0.00 -> 12.2 mm
- net VA2: track 0.00 -> 12.2 mm
Changed lines of the file:
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@@
     )
   )
+  (footprint "Tinker:Board_Stacker_2" (layer "F.Cu")
+    (at 108.055 114 90)
+    (descr "JST SH series connector, SM04B-SRSS-TB (http://www.jst-mfg.com/product/pdf/eng/eSH.pdf), generated with kicad-footprint-generator")
+    (tags "connector JST SH top entry")
+    (property "Sheetfile" "Ethernet-POE-WIP.kicad_sch")
+    (property "Sheetname" "")
+    (property "exclude_from_bom" "")
+    (attr smd exclude_from_bom)
+    (fp_text reference "J11" (at 1.6 0.635) (layer "F.SilkS")
+      (effects (font (size 0.6 0.6) (thickness 0.15)))
+    )
+    (fp_text value "Conn_01x02_Male" (at 0 4.084197 90) (layer "F.Fab")
+      (effects (font (size 1 1) (thickness 0.15)))
+    )
+    (fp_line (start -2 1.915) (end 2 1.915) (layer "F.CrtYd") (width 0.05))
+    (fp_line (start -2 -0.645) (end -2 1.915) (layer "F.CrtYd") (width 0.05))
+    (fp_line (start 2 -0.645) (end -2 -0.645) (layer "F.CrtYd") (width 0.05))
+    (fp_line (start 2 1.915) (end 2 -0.645) (layer "F.CrtYd") (width 0.05))
+    (fp_line (start 1.079472 -0.635) (end 1.079472 1.905) (layer "F.Fab") (width 0.1))
+    (fp_line (start -1.020528 -0.11) (end -0.495528 -0.635) (layer "F.Fab") (width 0.1))
+    (fp_line (start 1.079472 1.905) (end -1.020528 1.905) (layer "F.Fab") (width 0.1))
+    (fp_line (start -0.495528 -0.635) (end 1.079472 -0.635) (layer "F.Fab") (width 0.1))
+    (fp_line (start -1.020528 1.905) (end -1.020528 -0.11) (layer "F.Fab") (width 0.1))
+    (pad "1" thru_hole rect (at 0 0 90) (size 1 1) (drill 0.65) (layers *.Cu *.Mask)
+      (net 15 "VA1") (pinfunction "Pin_1") (pintype "passive"))
+    (pad "1" smd rect (at 1.35 0 90) (size 1.8 0.65) (layers "B.Cu" "B.Paste" "B.Mask")
+      (net 15 "VA1") (pinfunction "Pin_1") (pintype "passive"))
+    (pad "2" thru_hole oval (at 0 1.27 90) (size 1 1) (drill 0.65) (layers *.Cu *.Mask)
+      (net 14 "VA2") (pinfunction "Pin_2") (pintype "passive"))
+    (pad "2" smd rect (at -1.35 1.27 90) (size 1.8 0.65) (layers "B.Cu" "B.Paste" "B.Mask")
+      (net 14 "VA2") (pinfunction "Pin_2") (pintype "passive"))
+    (model "${KICAD6_3DMODEL_DIR}/Connector_PinHeader_1.27mm.3dshapes/PinHeader_1x02_P1.27mm_Vertical.step"
+      (offset (xyz 0 0 0))
+      (scale (xyz 1 1 1))
+      (rotate (xyz 0 0 0))
+    )
+    (model "${KICAD6_3DMODEL_DIR}/Connector_PinSocket_1.27mm.3dshapes/PinSocket_1x02_P1.27mm_Vertical_SMD_Pin1Left.step" hide
+      (offset (xyz 0 -0.635 -1.72))
+      (scale (xyz 1 1 1))
+      (rotate (xyz 0 -180 0))
+    )
+    (model "${KICAD6_3DMODEL_DIR}/Connector_PinSocket_1.27mm.3dshapes/PinSocket_1x02_P1.27mm_Vertical.step" hide
+      (offset (xyz 0 0 -1.72))
+      (scale (xyz 1 1 1))
+      (rotate (xyz 0 180 0))
+    )
+  )
   (footprint "Tinker:PinHeader_2x04_P1.27mm_Vertical" (layer "F.Cu")
     (at 86 98.095)
@@
   )
   (footprint "Tinker:Board_Stacker_2" (layer "F.Cu")
+    (at 90.675 114 90)
+    (descr "JST SH series connector, SM04B-SRSS-TB (http://www.jst-mfg.com/product/pdf/eng/eSH.pdf), generated with kicad-footprint-generator")
+    (tags "connector JST SH top entry")
+    (property "Sheetfile" "Ethernet-POE-WIP.kicad_sch")
+    (property "Sheetname" "")
+    (property "exclude_from_bom" "")
+    (attr smd exclude_from_bom)
+    (fp_text reference "J10" (at 1.6 0.635) (layer "F.SilkS")
+      (effects (font (size 0.6 0.6) (thickness 0.15)))
+    )
+    (fp_text value "Conn_01x02_Male" (at 0 4.084197 90) (layer "F.Fab")
+      (effects (font (size 1 1) (thickness 0.15)))
+    )
+    (fp_line (start -2 1.915) (end 2 1.915) (layer "F.CrtYd") (width 0.05))
+    (fp_line (start 2 -0.645) (end -2 -0.645) (layer "F.CrtYd") (width 0.05))
+    (fp_line (start 2 1.915) (end 2 -0.645) (layer "F.CrtYd") (width 0.05))
+    (fp_line (start -2 -0.645) (end -2 1.915) (layer "F.CrtYd") (width 0.05))
+    (fp_line (start 1.079472 -0.635) (end 1.079472 1.905) (layer "F.Fab") (width 0.1))
+    (fp_line (start 1.079472 1.905) (end -1.020528 1.905) (layer "F.Fab") (width 0.1))
+    (fp_line (start -1.020528 -0.11) (end -0.495528 -0.635) (layer "F.Fab") (width 0.1))
+    (fp_line (start -1.020528 1.905) (end -1.020528 -0.11) (layer "F.Fab") (width 0.1))
+    (fp_line (start -0.495528 -0.635) (end 1.079472 -0.635) (layer "F.Fab") (width 0.1))
+    (pad "1" smd rect (at 1.35 0 90) (size 1.8 0.65) (layers "B.Cu" "B.Paste" "B.Mask")
+      (net 11 "VB1") (pinfunction "Pin_1") (pintype "passive"))
+    (pad "1" thru_hole rect (at 0 0 90) (size 1 1) (drill 0.65) (layers *.Cu *.Mask)
+      (net 11 "VB1") (pinfunction "Pin_1") (pintype "passive"))
+    (pad "2" thru_hole oval (at 0 1.27 90) (size 1 1) (drill 0.65) (layers *.Cu *.Mask)
+      (net 10 "VB2") (pinfunction "Pin_2") (pintype "passive"))
+    (pad "2" smd rect (at -1.35 1.27 90) (size 1.8 0.65) (layers "B.Cu" "B.Paste" "B.Mask")
+      (net 10 "VB2") (pinfunction "Pin_2") (pintype "passive"))
+    (model "${KICAD6_3DMODEL_DIR}/Connector_PinHeader_1.27mm.3dshapes/PinHeader_1x02_P1.27mm_Vertical.step"
+      (offset (xyz 0 0 0))
+      (scale (xyz 1 1 1))
+      (rotate (xyz 0 0 0))
+    )
+    (model "${KICAD6_3DMODEL_DIR}/Connector_PinSocket_1.27mm.3dshapes/PinSocket_1x02_P1.27mm_Vertical_SMD_Pin1Left.step" hide
+      (offset (xyz 0 -0.635 -1.72))
+      (scale (xyz 1 1 1))
+      (rotate (xyz 0 -180 0))
+    )
+    (model "${KICAD6_3DMODEL_DIR}/Connector_PinSocket_1.27mm.3dshapes/PinSocket_1x02_P1.27mm_Vertical.step" hide
+      (offset (xyz 0 0 -1.72))
+      (scale (xyz 1 1 1))
+      (rotate (xyz 0 180 0))
+    )
+  )
+  (footprint "Tinker:Board_Stacker_2" (layer "F.Cu")
     (at 114 106.32)
     (descr "JST SH series connector, SM04B-SRSS-TB (http://www.jst-mfg.com/product/pdf/eng/eSH.pdf), generated with kicad-footprint-generator")
@@
   (segment (start 113.953367 106.366633) (end 114 106.32) (width 0.6) (layer "B.Cu") (net 7))
   (segment (start 105.69 106.785) (end 105.69 109.325) (width 0.6) (layer "B.Cu") (net 7))
+  (segment (start 96.27 109.675) (end 96.27 103.075) (width 0.6) (layer "B.Cu") (net 10))
+  (segment (start 91.945 114) (end 96.27 109.675) (width 0.6) (layer "B.Cu") (net 10))
+  (segment (start 90.675 113.926497) (end 92.658672 111.942825) (width 0.6) (layer "B.Cu") (net 11))
+  (segment (start 92.658672 104.146328) (end 93.73 103.075) (width 0.6) (layer "B.Cu") (net 11))
+  (segment (start 92.658672 111.942825) (end 92.658672 104.146328) (width 0.6) (layer "B.Cu") (net 11))
+  (segment (start 90.675 114) (end 90.675 113.926497) (width 0.6) (layer "B.Cu") (net 11))
   (segment (start 94.31 93.215) (end 94.31 90.675) (width 0.6) (layer "B.Cu") (net 12))
   (segment (start 94.970757 95.37084) (end 93.73 96.611597) (width 0.6) (layer "B.Cu") (net 12))
@@
   (segment (start 94.31 106.785) (end 95 106.095) (width 0.6) (layer "B.Cu") (net 13))
   (segment (start 104.31533 98.87967) (end 106.27 96.925) (width 0.6) (layer "B.Cu") (net 13))
+  (segment (start 107.277119 104.082119) (end 107.277119 109.144237) (width 0.6) (layer "B.Cu") (net 14))
+  (segment (start 109.325 111.192118) (end 109.325 114) (width 0.6) (layer "B.Cu") (net 14))
+  (segment (start 106.27 103.075) (end 107.277119 104.082119) (width 0.6) (layer "B.Cu") (net 14))
+  (segment (start 107.277119 109.144237) (end 109.325 111.192118) (width 0.6) (layer "B.Cu") (net 14))
+  (segment (start 103.73 109.675) (end 103.73 103.075) (width 0.6) (layer "B.Cu") (net 15))
+  (segment (start 108.055 114) (end 103.73 109.675) (width 0.6) (layer "B.Cu") (net 15))
   (zone (net 8) (net_name "GND") (layer "F.Cu") (hatch edge 0.508)
     (connect_pads (clearance 0.254))

Commit message: Some randomness...
Other:
- board text added: "${TITLE} Board"
Changed lines of the file:
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@@
     (effects (font (size 0.6 0.6) (thickness 0.125)))
+  )
+  (gr_text "${TITLE} Board" (at 99.934711 113.90372) (layer "F.SilkS")
+    (effects (font (size 1 1) (thickness 0.15)))
   )
   (gr_text "GND" (at 114 101) (layer "F.SilkS")

Commit message: whole bunche cleanup...
Parts:
- moved REF** 2.06 mm to (109.0, 87.0)
- moved G*** 2.00 mm to (91.0, 86.0)
Changed lines of the file:
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@@
   )
   (footprint "Tinker:DagNabbit" (layer "F.Cu")
-    (at 107 86.5)
+    (at 109 87)
     (attr smd board_only)
     (fp_text reference "REF**" (at 0 -8.08 unlocked) (layer "F.SilkS") hide
@@
   )
   (footprint "Tinker:NerdMage" (layer "F.Cu")
-    (at 93 85.9)
+    (at 91 86)
     (attr board_only exclude_from_pos_files exclude_from_bom)
     (fp_text reference "G***" (at 0 3.81) (layer "F.SilkS") hide
@@
     (effects (font (size 0.6 0.6) (thickness 0.125)))
   )
-  (gr_text "${TITLE} Board" (at 99.934711 113.90372) (layer "F.SilkS")
+  (gr_text "${TITLE} Board" (at 110 100 90) (layer "F.SilkS")
     (effects (font (size 1 1) (thickness 0.15)))
   )
