File: Hardware/Ethernet-S.kicad_pcb (KiCad board)
At the start: 2 copper layers, 34 x 34 mm, 14 parts, among them J11 Conn_01x10_Male, J12 Conn_01x04_Male, J3 Conn_01x02_Male, J4 Conn_01x02_Male, J5 Conn_01x02_Male, J6 Conn_01x02_Male, J7 Conn_01x08_Male, J9 QWIIC_Stackable

Commit message: Buncha cosmetic stuff...
Parts:
- removed J11: Conn_01x10_Male, Tinker:PinHeader_1x10_P1.27mm_Vertical
- removed J12: Conn_01x04_Male, Tinker:PinHeader_1x04_P1.27mm_Vertical
Connections:
- net ATTACH renamed SCLK
- net GPIO renamed ~{SCS}
- net POWER_OK2 renamed MISO
- net POWER_OK3 renamed MOSI
- net RESET renamed WIZ_RST
- J7 pad 7: ALERT -> unconnected-(J7-Pad7)
Routing:
- net Vsec: track 28.1 -> 8.26 mm
Other:
- board text added: "Stacked Rabbit ${TITLE} (v${REVISION})"
- board text removed: "NerdMage Modules ${TITLE} (v${REVISION})"

Commit message: Some randomness...
Other:
- board text added: "${TITLE} Board"
Changed lines of the file:
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@@
     (effects (font (size 0.6 0.6) (thickness 0.125)))
+  )
+  (gr_text "${TITLE} Board" (at 109.747392 104.749597 90) (layer "F.SilkS")
+    (effects (font (size 1 1) (thickness 0.15)))
   )
   (gr_text "I2C" (at 86 100) (layer "User.9")

Commit message: whole bunche cleanup...
Parts:
- moved REF** 0.23 mm to (109.0, 87.0)
- moved G*** 0.10 mm to (91.0, 86.0)
Changed lines of the file:
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@@
   )
   (footprint "Tinker:DagNabbit" (layer "F.Cu")
-    (at 109.037169 87.226251)
+    (at 109 87)
     (attr smd board_only)
     (fp_text reference "REF**" (at 0 -8.08 unlocked) (layer "F.SilkS") hide
@@
   )
   (footprint "Tinker:NerdMage" (layer "F.Cu")
-    (at 91 85.9)
+    (at 91 86)
     (attr board_only exclude_from_pos_files exclude_from_bom)
     (fp_text reference "G***" (at 0 3.81) (layer "F.SilkS") hide
@@
     (effects (font (size 0.6 0.6) (thickness 0.125)))
   )
-  (gr_text "${TITLE} Board" (at 109.747392 104.749597 90) (layer "F.SilkS")
+  (gr_text "${TITLE} Board" (at 110 100 90) (layer "F.SilkS")
     (effects (font (size 1 1) (thickness 0.15)))
   )
