File: Hardware/RP2040.kicad_sch (KiCad schematic)
At the start: 42 parts, among them J2 Conn_01x04_Male, J3 Conn_01x02_Male, J4 Conn_01x02_Male, J5 Conn_01x02_Male, J6 Conn_01x02_Male, J7 Conn_01x08_Male, J8 QWIIC_Vertical, J9 QWIIC_Stackable, Q1 DMG1012T, U1 RP2040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

Commit message: Tarduino!!!!!!!!!!!!!!!!!!!!!
Parts:
- added J1: Conn_01x07_Male, Tinker:Board_Stacker_7, symbol Connector:Conn_01x07_Male
- LED1: LCSC (none) -> C5349953
- Y1: footprint Crystal:Crystal_SMD_2016-4Pin_2.0x1.6mm -> Tinker:Crystal_SMD_2016-4Pin_2.0x1.6mm; LCSC https://www.lcsc.com/product-detail/Crystals_JWT-CN4020M000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 -> C2932954
Connections:
- net +3V3: now also J1.1 (Pin_1)
- net GND: now also J1.4 (Pin_4)
- new net DTR: J1.5 (Pin_5)
- new net IO1: J1.3 (Pin_3)
- new net IO3: J1.2 (Pin_2)
- new net RST: J1.7 (Pin_7)
- new net RTS: J1.6 (Pin_6)
Other:
- note added: "RP2040"
- note removed: "ESP8285"
- title: USB-C PD Controller -> RP2040
Changed lines of the file:
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@@
   (paper "A4")
   (title_block
-    (title "USB-C PD Controller")
-    (rev "0.1.3")
+    (title "RP2040")
+    (rev "0.0.0")
     (company "The Nerd Mage")
     (comment 2 "Massively a WIP!")
@@
     (stroke (width 0) (type default) (color 0 0 0 0))
   )
+  (wire (pts (xy 68.58 66.04) (xy 69.85 66.04))
+    (stroke (width 0) (type default) (color 0 0 0 0))
+  )
   (polyline (pts (xy 95.25 144.78) (xy 173.99 144.78))
     (stroke (width 0) (type default) (color 0 0 0 0))
@@
     (stroke (width 0) (type default) (color 0 0 0 0))
   )
+  (wire (pts (xy 85.09 63.5) (xy 68.58 63.5))
+    (stroke (width 0) (type default) (color 0 0 0 0))
+  )
   (wire (pts (xy 482.6 106.68) (xy 482.6 110.49))
     (stroke (width 0) (type default) (color 0 0 0 0))
@@
     (stroke (width 0) (type default) (color 0 0 0 0))
   )
+  (wire (pts (xy 85.09 72.39) (xy 85.09 63.5))
+    (stroke (width 0) (type default) (color 0 0 0 0))
+  )
   (polyline (pts (xy 13.97 194.31) (xy 92.71 194.31))
     (stroke (width 0) (type default) (color 0 0 0 0))
@@
   )
   (wire (pts (xy 447.04 77.47) (xy 447.04 74.93))
+    (stroke (width 0) (type default) (color 0 0 0 0))
+  )
+  (wire (pts (xy 68.58 71.12) (xy 74.93 71.12))
     (stroke (width 0) (type default) (color 0 0 0 0))
   )
@@
     (stroke (width 0) (type default) (color 0 0 0 0))
   )
+  (wire (pts (xy 68.58 58.42) (xy 74.93 58.42))
+    (stroke (width 0) (type default) (color 0 0 0 0))
+  )
   (wire (pts (xy 314.96 120.65) (xy 314.96 130.81))
     (stroke (width 0) (type default) (color 0 0 0 0))
@@
     (stroke (width 0) (type default) (color 0 0 0 0))
   )
+  (wire (pts (xy 68.58 55.88) (xy 74.93 55.88))
+    (stroke (width 0) (type default) (color 0 0 0 0))
+  )
   (wire (pts (xy 339.09 60.96) (xy 358.14 60.96))
+    (stroke (width 0) (type default) (color 0 0 0 0))
+  )
+  (wire (pts (xy 68.58 68.58) (xy 69.85 68.58))
+    (stroke (width 0) (type default) (color 0 0 0 0))
+  )
+  (wire (pts (xy 68.58 60.96) (xy 74.93 60.96))
     (stroke (width 0) (type default) (color 0 0 0 0))
   )
@@
     (effects (font (size 1.27 1.27)) (justify left bottom))
   )
-  (text "ESP8285" (at 106.68 27.94 180)
+  (text "RP2040" (at 106.68 27.94 180)
     (effects (font (size 2.54 2.54) (thickness 0.508) bold) (justify left bottom))
   )
@@
     (effects (font (size 2.54 2.54) (thickness 0.508) bold) (justify left bottom))
   )
+  (label "RxD" (at 69.85 58.42 0)
+    (effects (font (size 1.27 1.27)) (justify left bottom))
+  )
   (label "USB_DP" (at 350.52 60.96 0)
     (effects (font (size 1.27 1.27)) (justify left bottom))
@@
   )
   (label "USB_DM" (at 350.52 63.5 0)
+    (effects (font (size 1.27 1.27)) (justify left bottom))
+  )
+  (label "RTS" (at 69.85 68.58 0)
+    (effects (font (size 1.27 1.27)) (justify left bottom))
+  )
+  (label "TxD" (at 69.85 60.96 0)
+    (effects (font (size 1.27 1.27)) (justify left bottom))
+  )
+  (label "DTR" (at 69.85 66.04 0)
     (effects (font (size 1.27 1.27)) (justify left bottom))
   )
@@
     )
   )
+  (global_label "+3V3" (shape input) (at 74.93 55.88 0) (fields_autoplaced)
+    (effects (font (size 1.27 1.27)) (justify left))
+    (property "Intersheet References" "${INTERSHEET_REFS}" (id 0) (at 82.4231 55.8006 0)
+      (effects (font (size 1.27 1.27)) (justify left) hide)
+    )
+  )
   (global_label "io4" (shape input) (at 408.94 63.5 0) (fields_autoplaced)
     (effects (font (size 1.27 1.27)) (justify left))
@@
     )
   )
+  (global_label "IO3" (shape input) (at 74.93 58.42 0) (fields_autoplaced)
+    (effects (font (size 1.27 1.27)) (justify left))
+    (property "Intersheet References" "${INTERSHEET_REFS}" (id 0) (at 80.4879 58.3406 0)
+      (effects (font (size 1.27 1.27)) (justify left) hide)
+    )
+  )
   (global_label "SCL" (shape input) (at 161.29 82.55 180) (fields_autoplaced)
     (effects (font (size 1.27 1.27) (thickness 0.254) bold) (justify right))
@@
     )
   )
+  (global_label "RST" (shape input) (at 74.93 71.12 0) (fields_autoplaced)
+    (effects (font (size 1.27 1.27)) (justify left))
+    (property "Intersheet References" "${INTERSHEET_REFS}" (id 0) (at 80.7902 71.0406 0)
+      (effects (font (size 1.27 1.27)) (justify left) hide)
+    )
+  )
+  (global_label "IO1" (shape input) (at 74.93 60.96 0) (fields_autoplaced)
+    (effects (font (size 1.27 1.27)) (justify left))
+    (property "Intersheet References" "${INTERSHEET_REFS}" (id 0) (at 80.4879 60.8806 0)
+      (effects (font (size 1.27 1.27)) (justify left) hide)
+    )
+  )
   (global_label "POWER_OK2" (shape output) (at 161.29 85.09 180) (fields_autoplaced)
     (effects (font (size 1.27 1.27) (thickness 0.254) bold) (justify right))
@@
     )
     (pin "1")
+  )
+  (symbol (lib_id "Connector:Conn_01x07_Male") (at 63.5 63.5 0) (unit 1)
+    (in_bom no) (on_board no)
+    (property "Reference" "J1" (id 0) (at 64.77 53.34 0))
+    (property "Value" "Conn_01x07_Male" (id 1) (at 68.58 63.5 90)
+      (effects (font (size 1.27 1.27)) hide)
+    )
+    (property "Footprint" "Tinker:Board_Stacker_7" (id 2) (at 63.5 63.5 0)
+      (effects (font (size 1.27 1.27)) hide)
+    )
+    (property "Datasheet" "~" (id 3) (at 63.5 63.5 0)
+      (effects (font (size 1.27 1.27)) hide)
+    )
+    (property "Note" "Footprint only" (id 4) (at 63.5 63.5 0)
+      (effects (font (size 1.27 1.27)) hide)
+    )
+    (pin "1")
+    (pin "2")
+    (pin "3")
+    (pin "4")
+    (pin "5")
+    (pin "6")
+    (pin "7")
   )
   (symbol (lib_id "Device:R") (at 542.29 15.24 90) (unit 1)
@@
     (pin "1")
   )
+  (symbol (lib_id "power:GND") (at 85.09 72.39 0) (unit 1)
+    (in_bom yes) (on_board yes)
+    (property "Reference" "#PWR0139" (id 0) (at 85.09 78.74 0)
+      (effects (font (size 1.27 1.27)) hide)
+    )
+    (property "Value" "GND" (id 1) (at 85.09 76.2 0))
+    (property "Footprint" "" (id 2) (at 85.09 72.39 0)
+      (effects (font (size 1.27 1.27)) hide)
+    )
+    (property "Datasheet" "" (id 3) (at 85.09 72.39 0)
+      (effects (font (size 1.27 1.27)) hide)
+    )
+    (pin "1")
+  )
   (symbol (lib_id "Device:R") (at 471.17 55.88 90) (unit 1)
     (in_bom yes) (on_board yes)
@@
     (property "Reference" "Y1" (id 0) (at 332.74 123.19 0))
     (property "Value" "12MHz" (id 1) (at 334.01 128.27 0))
-    (property "Footprint" "Crystal:Crystal_SMD_2016-4Pin_2.0x1.6mm" (id 2) (at 327.66 125.73 0)
+    (property "Footprint" "Tinker:Crystal_SMD_2016-4Pin_2.0x1.6mm" (id 2) (at 327.66 125.73 0)
       (effects (font (size 1.27 1.27)) hide)
     )
@@
       (effects (font (size 1.27 1.27)) hide)
     )
-    (property "LCSC" "https://www.lcsc.com/product-detail/Crystals_JWT-CN4020M00015T8188108_C2932954.html" (id 4) (at 327.66 125.73 0)
+    (property "LCSC" "C2932954" (id 4) (at 327.66 125.73 0)
       (effects (font (size 1.27 1.27)) hide)
     )
@@
       (effects (font (size 1.27 1.27)) (justify left top) hide)
     )
-    (property "Mouser Part Number" "" (id 11) (at 549.91 727.94 0)
-      (effects (font (size 1.27 1.27)) (justify left top) hide)
-    )
-    (property "Mouser Price/Stock" "" (id 12) (at 549.91 827.94 0)
-      (effects (font (size 1.27 1.27)) (justify left top) hide)
-    )
-    (property "Arrow Part Number" "" (id 13) (at 549.91 927.94 0)
-      (effects (font (size 1.27 1.27)) (justify left top) hide)
-    )
-    (property "Arrow Price/Stock" "" (id 14) (at 549.91 1027.94 0)
+    (property "LCSC" "C5349953" (id 14) (at 549.91 1027.94 0)
       (effects (font (size 1.27 1.27)) (justify left top) hide)
     )
@@
       (reference "#PWR0138") (unit 1) (value "GND") (footprint "")
     )
+    (path "/6353fa02-1a9b-4560-bae0-c27892d6f64e"
+      (reference "#PWR0139") (unit 1) (value "GND") (footprint "")
+    )
     (path "/a7015c69-c3ab-4d4d-9a0c-d2b8a89c3066"
       (reference "C1") (unit 1) (value "20p") (footprint "Capacitor_SMD:C_0402_1005Metric")
@@
       (reference "D2") (unit 1) (value "LED") (footprint "LED_SMD:LED_0402_1005Metric")
     )
+    (path "/0edc2c7a-7d2e-478d-a97b-c3d26d3a9e6a"
+      (reference "J1") (unit 1) (value "Conn_01x07_Male") (footprint "Tinker:Board_Stacker_7")
+    )
     (path "/ce562b82-4d15-4512-9ef8-80a89b06889d"
       (reference "J2") (unit 1) (value "Conn_01x04_Male") (footprint "Tinker:Board_Stacker_4")
@@
     )
     (path "/970339ae-2250-4e02-93ba-cdc5493eac4d"
-      (reference "Y1") (unit 1) (value "12MHz") (footprint "Crystal:Crystal_SMD_2016-4Pin_2.0x1.6mm")
-    )
-  )
+      (reference "Y1") (unit 1) (value "12MHz") (footprint "Tinker:Crystal_SMD_2016-4Pin_2.0x1.6mm")
+    )
+  )

Commit message: Still cleaning up J7
Connections:
- net ALERT renamed DEV_GPIO
- net ATTACH renamed SCLK
- net IO12 renamed MISO
- net IO13 renamed MOSI
- net IO15 renamed ~{SCS}
- net IO16 renamed DEV_RST
Other:
- note added: "SPI"
- note removed: "MCU"
- moved on the sheet: C1, C10, C11, C12, C13, C14, C15, C16, C2, C3, C4, C5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
