File: Hardware/Tarduino Clone.kicad_pcb (KiCad board)
At the start: 2 copper layers, 34 x 34 mm, 25 parts, among them J1 Conn_01x07_Male, J2 Conn_01x04_Male, J3 Conn_01x02_Male, J4 Conn_01x02_Male, J5 Conn_01x02_Male, J6 Conn_01x02_Male, J7 Conn_01x08_Male, J9 QWIIC_Stackable, SW1 SW_Push, U1 ATmega328PB-A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

Commit message: whole bunche cleanup...
Parts:
- moved REF** 2.06 mm to (109.0, 87.0)
- moved G*** 2.00 mm to (91.0, 86.0)
Changed lines of the file:
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@@
   )
   (footprint "Tinker:DagNabbit" (layer "F.Cu")
-    (at 107 86.5)
+    (at 109 87)
     (attr smd board_only)
     (fp_text reference "REF**" (at 0 -8.08 unlocked) (layer "F.SilkS") hide
@@
   )
   (footprint "Tinker:NerdMage" (layer "F.Cu")
-    (at 93 85.9)
+    (at 91 86)
     (attr board_only exclude_from_pos_files exclude_from_bom)
     (fp_text reference "G***" (at 5.08 0) (layer "F.SilkS") hide

Commit message: Still cleaning up J7
Connections:
- net WIZ_RST renamed DEV_RST
- J7 pad 7: unconnected-(J7-Pad7) -> DEV_GPIO
Other:
- board text added: "DEV-IO"
- board text added: "DEV-RST"
- board text removed: "????"
- board text removed: "RST->"
Changed lines of the file:
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@@
   (net 13 "UD+")
   (net 14 "UD-")
-  (net 15 "Net-(U1-Pad8)")
-  (net 16 "Net-(U1-Pad7)")
+  (net 15 "Net-(C3-Pad2)")
+  (net 16 "Net-(C4-Pad2)")
   (net 17 "D3")
   (net 18 "D4")
@@
   (net 35 "/AREF")
   (net 36 "DTR")
-  (net 37 "WIZ_RST")
+  (net 37 "DEV_RST")
   (net 38 "SCLK")
-  (net 39 "unconnected-(J7-Pad7)")
+  (net 39 "DEV_GPIO")
   (net 40 "~{SCS}")
   (footprint "Tinker:Mount" (layer "F.Cu")
@@
       (net 3 "GND") (pintype "passive"))
     (pad "2" smd roundrect (at 0.775 0 180) (size 0.9 0.95) (layers "F.Cu" "F.Paste" "F.Mask") (roundrect_rratio 0.25)
-      (net 16 "Net-(U1-Pad7)") (pintype "passive"))
+      (net 16 "Net-(C4-Pad2)") (pintype "passive"))
     (model "${KICAD6_3DMODEL_DIR}/Capacitor_SMD.3dshapes/C_0603_1608Metric.wrl"
       (offset (xyz 0 0 0))
@@
       (net 3 "GND") (pintype "passive"))
     (pad "2" smd roundrect (at 0.775 0) (size 0.9 0.95) (layers "F.Cu" "F.Paste" "F.Mask") (roundrect_rratio 0.25)
-      (net 15 "Net-(U1-Pad8)") (pintype "passive"))
+      (net 15 "Net-(C3-Pad2)") (pintype "passive"))
     (model "${KICAD6_3DMODEL_DIR}/Capacitor_SMD.3dshapes/C_0603_1608Metric.wrl"
       (offset (xyz 0 0 0))
@@
       (net 4 "+3V3") (pinfunction "PE1") (pintype "bidirectional"))
     (pad "7" smd rect (at -4.25 2) (size 1.6 0.55) (layers "F.Cu" "F.Paste" "F.Mask")
-      (net 16 "Net-(U1-Pad7)") (pinfunction "XTAL1/PB6") (pintype "bidirectional"))
+      (net 16 "Net-(C4-Pad2)") (pinfunction "XTAL1/PB6") (pintype "bidirectional"))
     (pad "8" smd rect (at -4.25 2.8) (size 1.6 0.55) (layers "F.Cu" "F.Paste" "F.Mask")
-      (net 15 "Net-(U1-Pad8)") (pinfunction "XTAL2/PB7") (pintype "bidirectional"))
+      (net 15 "Net-(C3-Pad2)") (pinfunction "XTAL2/PB7") (pintype "bidirectional"))
     (pad "9" smd rect (at -2.8 4.25 90) (size 1.6 0.55) (layers "F.Cu" "F.Paste" "F.Mask")
       (net 19 "D5") (pinfunction "PD5") (pintype "bidirectional"))
@@
     (fp_line (start 1.6 1.25) (end -1.6 1.25) (layer "F.Fab") (width 0.2))
     (pad "1" smd rect (at -1.15 0.875 180) (size 1.05 1.3) (layers "F.Cu" "F.Paste" "F.Mask")
-      (net 15 "Net-(U1-Pad8)") (pinfunction "Xt_1") (pintype "passive"))
+      (net 15 "Net-(C3-Pad2)") (pinfunction "Xt_1") (pintype "passive"))
     (pad "2" smd rect (at 1.15 0.875 180) (size 1.05 1.3) (layers "F.Cu" "F.Paste" "F.Mask")
       (net 3 "GND") (pinfunction "G_1") (pintype "passive"))
     (pad "3" smd rect (at 1.15 -0.875 180) (size 1.05 1.3) (layers "F.Cu" "F.Paste" "F.Mask")
-      (net 16 "Net-(U1-Pad7)") (pinfunction "Xt_2") (pintype "passive"))
+      (net 16 "Net-(C4-Pad2)") (pinfunction "Xt_2") (pintype "passive"))
     (pad "4" smd rect (at -1.15 -0.875 180) (size 1.05 1.3) (layers "F.Cu" "F.Paste" "F.Mask")
       (net 3 "GND") (pinfunction "G_2") (pintype "passive"))
@@
     (fp_line (start -0.2175 -0.635) (end 2.34 -0.635) (layer "F.Fab") (width 0.1))
     (pad "1" thru_hole rect (at 0 0) (size 1 1) (drill 0.65) (layers *.Cu *.Mask)
-      (net 37 "WIZ_RST") (pinfunction "Pin_1") (pintype "passive"))
+      (net 37 "DEV_RST") (pinfunction "Pin_1") (pintype "passive"))
     (pad "1" smd rect (at -1.195 0) (size 2.1 0.75) (layers "B.Cu" "B.Paste" "B.Mask")
-      (net 37 "WIZ_RST") (pinfunction "Pin_1") (pintype "passive"))
+      (net 37 "DEV_RST") (pinfunction "Pin_1") (pintype "passive"))
     (pad "2" thru_hole oval (at 1.27 0) (size 1 1) (drill 0.65) (layers *.Cu *.Mask)
       (net 38 "SCLK") (pinfunction "Pin_2") (pintype "passive"))
@@
       (net 25 "MOSI") (pinfunction "Pin_6") (pintype "passive"))
     (pad "7" smd rect (at -1.195 3.81) (size 2.1 0.75) (layers "B.Cu" "B.Paste" "B.Mask")
-      (net 39 "unconnected-(J7-Pad7)") (pinfunction "Pin_7") (pintype "passive"))
+      (net 39 "DEV_GPIO") (pinfunction "Pin_7") (pintype "passive"))
     (pad "7" thru_hole oval (at 0 3.81) (size 1 1) (drill 0.65) (layers *.Cu *.Mask)
-      (net 39 "unconnected-(J7-Pad7)") (pinfunction "Pin_7") (pintype "passive"))
+      (net 39 "DEV_GPIO") (pinfunction "Pin_7") (pintype "passive"))
     (pad "8" thru_hole oval (at 1.27 3.81) (size 1 1) (drill 0.65) (layers *.Cu *.Mask)
       (net 40 "~{SCS}") (pinfunction "Pin_8") (pintype "passive"))
@@
     (effects (font (size 2 2) (thickness 0.3)))
   )
-  (gr_text "????" (at 87.5 103.175) (layer "F.SilkS")
+  (gr_text "DEV-IO" (at 87.5 103.175) (layer "F.SilkS")
     (effects (font (size 0.5 0.5) (thickness 0.125)) (justify left))
   )
@@
     (effects (font (size 0.6 0.6) (thickness 0.125)))
   )
-  (gr_text "RST->" (at 87.5 96.825) (layer "F.SilkS")
+  (gr_text "DEV-RST" (at 87.5 96.825) (layer "F.SilkS")
     (effects (font (size 0.5 0.5) (thickness 0.125)) (justify left))
   )
