File: Hardware/USB-PD Proto.kicad_pcb (KiCad board)
At the start: 2 copper layers, 34 x 34 mm, 12 parts, among them J1 Conn_01x08_Male, J2 Conn_01x04_Male, J3 Conn_01x02_Male, J4 Conn_01x02_Male, J5 Conn_01x02_Male, J6 Conn_01x02_Male

Commit message: Documentation
Parts:
- renumbered J1 to J7
Changed lines of the file:
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@@
     (descr "Through hole straight pin header, 2x04, 1.27mm pitch, double rows")
     (tags "Through hole pin header THT 2x04 1.27mm double row")
+    (property "LCSC" "C2881786 + C2684732")
     (property "Sheetfile" "USB-PD Proto.kicad_sch")
     (property "Sheetname" "")
     (property "exclude_from_bom" "")
     (attr through_hole exclude_from_bom)
-    (fp_text reference "J1" (at 0.635 -1.27) (layer "F.SilkS")
+    (fp_text reference "J7" (at 0.635 -1.27) (layer "F.SilkS")
       (effects (font (size 0.75 0.75) (thickness 0.15)))
     )

Commit message: Tinkerin' + RESET & LED on Programmer...
Parts:
- moved G*** 17.6 mm to (90.4, 72.9)
- moved REF** 16.6 mm to (108.0, 73.5)
Other:
- board text added: "${TITLE}"
- board text added: "NerdMage Modules ${TITLE} (v${REVISION})"
- board text removed: "NerdMage Modules (v0.0.1)"
- board text removed: "Prototype Board"
Changed lines of the file:
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@@
   (title_block
     (title "Prototype Board")
-    (rev "0.0.1")
+    (rev "0.0.2")
     (company "The Nerd Mage")
   )
@@
   )
   (footprint "Tinker:DagNabbit" (layer "F.Cu")
-    (at 91.4 73.5)
+    (at 108 73.5)
     (attr smd board_only)
     (fp_text reference "REF**" (at 0 -8.08 unlocked) (layer "F.SilkS") hide
@@
   )
   (footprint "Tinker:NerdMage" (layer "F.Cu")
-    (at 108 72.9)
+    (at 90.4 72.9)
     (attr board_only exclude_from_pos_files exclude_from_bom)
     (fp_text reference "G***" (at 0 3.81) (layer "F.SilkS") hide
@@
   (gr_line (start 86 104) (end 114 104) (layer "Edge.Cuts") (width 0.1))
   (gr_arc (start 117 101) (mid 116.12132 103.12132) (end 114 104) (layer "Edge.Cuts") (width 0.1))
-  (gr_text "NerdMage Modules (v0.0.1)" (at 100 74.8) (layer "B.SilkS")
+  (gr_text "NerdMage Modules\n${TITLE} (v${REVISION})" (at 100 76) (layer "B.SilkS")
     (effects (font (size 1 1) (thickness 0.15)) (justify mirror))
   )
@@
     (effects (font (size 0.6 0.6) (thickness 0.125)) (justify mirror))
   )
-  (gr_text "S. A. Miller 2023" (at 100 103) (layer "B.SilkS")
+  (gr_text "S. A. Miller 2023" (at 100 79) (layer "B.SilkS")
     (effects (font (size 1 1) (thickness 0.15)) (justify mirror))
   )
@@
     (effects (font (size 0.6 0.6) (thickness 0.125)))
   )
-  (gr_text "Prototype Board" (at 99.20714 103) (layer "F.SilkS")
+  (gr_text "${TITLE}" (at 99.20714 103) (layer "F.SilkS")
     (effects (font (size 0.75 0.75) (thickness 0.15)))
   )

Commit message: Uber Rework!
Parts:
- added J1: Conn_01x07_Male, Tinker:Board_Stacker_7, F.Cu at (96.2, 114.0)
- added J9: QWIIC_Stackable, Tinker:QWIIC_Stack_II, F.Cu at (87.3, 93.0)
- J2: footprint Tinker:PinHeader_1x04_P2.54mm_Vertical -> Tinker:Board_Stacker_4
- J3, J4, J5, J6: footprint Tinker:PinHeader_1x02_P2.54mm_Vertical -> Tinker:Board_Stacker_2
- moved G*** 13.3 mm to (93.0, 85.9)
- moved J2 13.1 mm to (101.9, 86.0)
- moved REF** 13.0 mm to (107.0, 86.5)
- moved J6 13.0 mm to (114.0, 91.1)
- moved J3 13.0 mm to (86.0, 106.3)
- moved J4 13.0 mm to (114.0, 106.3)
- moved J5 13.0 mm to (114.0, 98.7)
- moved J7 13.0 mm to (86.0, 98.1)
- moved REF** 13.0 mm to (114.0, 114.0)
- moved REF** 13.0 mm to (86.0, 114.0)
- moved REF** 13.0 mm to (114.0, 86.0)
- moved REF** 13.0 mm to (86.0, 86.0)
Routing:
- net SDA: track 0.00 -> 10.6 mm
- net SCL: track 0.00 -> 6.15 mm
Other:
- board text added: "3v3"
- board text added: "DTR"
- board text added: "RST"
- board text added: "RTS"
- board text added: "RxD"
- board text added: "TxD"

Commit message: Buncha cosmetic stuff...
Other:
- board text added: "Stacked Rabbit ${TITLE} (v${REVISION})"
- board text removed: "NerdMage Modules ${TITLE} (v${REVISION})"
Changed lines of the file:
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@@
   (gr_line (start 86 117) (end 114 117) (layer "Edge.Cuts") (width 0.1))
   (gr_arc (start 117 114) (mid 116.12132 116.12132) (end 114 117) (layer "Edge.Cuts") (width 0.1))
-  (gr_text "NerdMage Modules\n${TITLE} (v${REVISION})" (at 100 90) (layer "B.SilkS")
+  (gr_text "Stacked Rabbit\n${TITLE} (v${REVISION})" (at 100 90) (layer "B.SilkS")
     (effects (font (size 1 1) (thickness 0.15)) (justify mirror))
   )

Commit message: whole bunche cleanup...
Parts:
- moved REF** 2.06 mm to (109.0, 87.0)
- moved G*** 2.00 mm to (91.0, 86.0)
Changed lines of the file:
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@@
   )
   (footprint "Tinker:DagNabbit" (layer "F.Cu")
-    (at 107 86.5)
+    (at 109 87)
     (attr smd board_only)
     (fp_text reference "REF**" (at 0 -8.08 unlocked) (layer "F.SilkS") hide
@@
   )
   (footprint "Tinker:NerdMage" (layer "F.Cu")
-    (at 93 85.9)
+    (at 91 86)
     (attr board_only exclude_from_pos_files exclude_from_bom)
     (fp_text reference "G***" (at 0 3.81) (layer "F.SilkS") hide

Commit message: still messing about with SPI stuff...
Other:
- board text added: "DEV-IO"
- board text added: "DEV-RST"
- board text added: "MISO"
- board text added: "MOSI"
- board text added: "QWIIC"
- board text added: "SCL"
- board text added: "SCLK"
- board text added: "SDA"
- board text added: "~{SCS}"
Changed lines of the file:
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@@
     (property "exclude_from_bom" "")
     (attr smd exclude_from_bom)
-    (fp_text reference "J9" (at 3.158643 -2.390416 90) (layer "F.SilkS")
+    (fp_text reference "J9" (at 2.61321 -2.390416 180) (layer "F.SilkS")
       (effects (font (size 0.6 0.6) (thickness 0.15)))
     )
@@
     (property "exclude_from_bom" "")
     (attr through_hole exclude_from_bom)
-    (fp_text reference "J7" (at 3 1.905 90) (layer "F.SilkS")
+    (fp_text reference "J7" (at 0.635 5.345 180) (layer "F.SilkS")
       (effects (font (size 0.6 0.6) (thickness 0.15)))
     )
@@
     (effects (font (size 0.6 0.6) (thickness 0.125)) (justify mirror))
   )
+  (gr_text "SDA" (at 90.9 94.905) (layer "F.SilkS")
+    (effects (font (size 0.5 0.5) (thickness 0.125)) (justify left))
+  )
+  (gr_text "SCLK" (at 88.5 98.095) (layer "F.SilkS")
+    (effects (font (size 0.5 0.5) (thickness 0.125)) (justify left))
+  )
   (gr_text "TxD" (at 97.46 115.9 270) (layer "F.SilkS")
     (effects (font (size 0.6 0.6) (thickness 0.125)))
   )
+  (gr_text "3v3" (at 90.9 92.365) (layer "F.SilkS")
+    (effects (font (size 0.5 0.5) (thickness 0.125)) (justify left))
+  )
   (gr_text "RTS" (at 102.54 115.9 270) (layer "F.SilkS")
     (effects (font (size 0.6 0.6) (thickness 0.125)))
@@
     (effects (font (size 0.6 0.6) (thickness 0.125)))
   )
+  (gr_text "~{SCS}" (at 88.5 101.905) (layer "F.SilkS")
+    (effects (font (size 0.5 0.5) (thickness 0.125)) (justify left))
+  )
   (gr_text "RST" (at 103.81 115.9 270) (layer "F.SilkS")
     (effects (font (size 0.6 0.6) (thickness 0.125)))
   )
+  (gr_text "DEV-RST" (at 87.5 96.825) (layer "F.SilkS")
+    (effects (font (size 0.5 0.5) (thickness 0.125)) (justify left))
+  )
   (gr_text "GND" (at 114 93.4) (layer "F.SilkS")
     (effects (font (size 0.6 0.6) (thickness 0.125)))
   )
+  (gr_text "GND" (at 90.9 91.095) (layer "F.SilkS")
+    (effects (font (size 0.5 0.5) (thickness 0.125)) (justify left))
+  )
   (gr_text "GND" (at 100 115.9 270) (layer "F.SilkS")
     (effects (font (size 0.6 0.6) (thickness 0.125)))
@@
     (effects (font (size 0.6 0.6) (thickness 0.15)))
   )
+  (gr_text "DEV-IO" (at 87.5 103.175) (layer "F.SilkS")
+    (effects (font (size 0.5 0.5) (thickness 0.125)) (justify left))
+  )
   (gr_text "GND" (at 114 101) (layer "F.SilkS")
     (effects (font (size 0.6 0.6) (thickness 0.125)))
@@
     (effects (font (size 0.6 0.6) (thickness 0.125)))
   )
+  (gr_text "SCL" (at 90.9 93.635) (layer "F.SilkS")
+    (effects (font (size 0.5 0.5) (thickness 0.125)) (justify left))
+  )
   (gr_text "GND" (at 114 108.7) (layer "F.SilkS")
     (effects (font (size 0.6 0.6) (thickness 0.125)))
   )
+  (gr_text "QWIIC" (at 83.695923 93 270) (layer "F.SilkS")
+    (effects (font (size 0.6 0.6) (thickness 0.15)))
+  )
+  (gr_text "MOSI" (at 88.5 100.635) (layer "F.SilkS")
+    (effects (font (size 0.5 0.5) (thickness 0.125)) (justify left))
+  )
   (gr_text "DTR" (at 101.27 115.9 270) (layer "F.SilkS")
     (effects (font (size 0.6 0.6) (thickness 0.125)))
@@
     (effects (font (size 0.6 0.6) (thickness 0.125)))
   )
+  (gr_text "SDA" (at 84.8 100.7275) (layer "F.SilkS")
+    (effects (font (size 0.5 0.5) (thickness 0.125)) (justify right))
+  )
   (gr_text "Vsec" (at 114 97.6) (layer "F.SilkS")
     (effects (font (size 0.6 0.6) (thickness 0.125)))
   )
+  (gr_text "MISO" (at 88.5 99.365) (layer "F.SilkS")
+    (effects (font (size 0.5 0.5) (thickness 0.125)) (justify left))
+  )
   (gr_text "Vout" (at 86 105.2) (layer "F.SilkS")
     (effects (font (size 0.6 0.6) (thickness 0.125)))
@@
     (effects (font (size 0.6 0.6) (thickness 0.125)))
   )
+  (gr_text "SCL" (at 84.8 99.4575) (layer "F.SilkS")
+    (effects (font (size 0.5 0.5) (thickness 0.125)) (justify right))
+  )
   (gr_text "3v3" (at 96.19 115.9 270) (layer "F.SilkS")
