File: Hardware/USB-PD Board 2.kicad_pcb (KiCad board)
At the start: 2 copper layers, 34 x 34 mm, 54 parts, among them J1 USB_C_Receptacle, J2 Conn_01x04_Male, J3 Conn_01x02_Male, J4 Conn_01x02_Male, J5 Conn_01x02_Male, J6 Conn_01x02_Male, J7 Conn_01x08_Male, J9 QWIIC_Stackable, Q1 DMP3013SFV, Q2 DMP3013SFV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

Commit message: ...
Routing:
- net Vbus: track 52.6 -> 40.3 mm
- net POWER_OK3: track 9.77 -> 11.4 mm
- net ATTACH: track 6.08 -> 6.81 mm
- net GND: vias 3 -> 11

Commit message: Working on changes to J7/J9
Parts:
- moved J6 1.28 mm to (114.0, 92.4)
- moved J5 0.66 mm to (114.0, 99.4)
Routing:
- net Vsec: track 24.0 -> 26.2 mm
Other:
- board text added: "USB"
- board text added: "Vusb"
- board text removed: "D+"
- board text removed: "D-"
Changed lines of the file:
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@@
   )
   (footprint "Tinker:Board_Stacker_2" (layer "F.Cu")
-    (at 114 106.32)
+    (at 114 106.365)
     (descr "JST SH series connector, SM04B-SRSS-TB (http://www.jst-mfg.com/product/pdf/eng/eSH.pdf), generated with kicad-footprint-generator")
     (tags "connector JST SH top entry")
@@
   )
   (footprint "Tinker:Board_Stacker_2" (layer "F.Cu")
-    (at 86 106.32)
+    (at 86 106.365)
     (descr "JST SH series connector, SM04B-SRSS-TB (http://www.jst-mfg.com/product/pdf/eng/eSH.pdf), generated with kicad-footprint-generator")
     (tags "connector JST SH top entry")
@@
   )
   (footprint "Tinker:Board_Stacker_2" (layer "F.Cu")
-    (at 114 91.08)
+    (at 114 92.365)
     (descr "JST SH series connector, SM04B-SRSS-TB (http://www.jst-mfg.com/product/pdf/eng/eSH.pdf), generated with kicad-footprint-generator")
     (tags "connector JST SH top entry")
@@
   )
   (footprint "Tinker:Board_Stacker_2" (layer "F.Cu")
-    (at 114 98.7)
+    (at 114 99.365)
     (descr "JST SH series connector, SM04B-SRSS-TB (http://www.jst-mfg.com/product/pdf/eng/eSH.pdf), generated with kicad-footprint-generator")
     (tags "connector JST SH top entry")
@@
     (effects (font (size 0.6 0.6) (thickness 0.125)) (justify mirror))
   )
-  (gr_text "GND" (at 114.007828 93.440254) (layer "B.SilkS")
+  (gr_text "GND" (at 114.007828 94.725254) (layer "B.SilkS")
     (effects (font (size 0.6 0.6) (thickness 0.125)) (justify mirror))
   )
-  (gr_text "Vsec" (at 113.891319 90.061488) (layer "B.SilkS")
+  (gr_text "Vsec" (at 113.891319 91.346488) (layer "B.SilkS")
     (effects (font (size 0.6 0.6) (thickness 0.125)) (justify mirror))
   )
-  (gr_text "Vsec" (at 113.913793 97.690477) (layer "B.SilkS")
+  (gr_text "Vsec" (at 113.913793 98.294169) (layer "B.SilkS")
     (effects (font (size 0.6 0.6) (thickness 0.125)) (justify mirror))
   )
@@
     (effects (font (size 1 1) (thickness 0.15)) (justify mirror))
   )
-  (gr_text "GND" (at 114.030302 101.069243) (layer "B.SilkS")
+  (gr_text "GND" (at 114.030302 101.694169) (layer "B.SilkS")
     (effects (font (size 0.6 0.6) (thickness 0.125)) (justify mirror))
   )
@@
     (effects (font (size 0.75 0.75) (thickness 0.15)))
   )
-  (gr_text "Vsec" (at 114.083614 97.629169) (layer "F.SilkS")
+  (gr_text "Vsec" (at 114.083614 98.294169) (layer "F.SilkS")
     (effects (font (size 0.6 0.6) (thickness 0.125)))
   )
-  (gr_text "Vout" (at 86.068727 105.243053) (layer "F.SilkS")
+  (gr_text "Vout" (at 86.068727 105.288053) (layer "F.SilkS")
     (effects (font (size 0.6 0.6) (thickness 0.125)))
   )
@@
     (effects (font (size 0.75 0.6) (thickness 0.15)))
   )
-  (gr_text "Vout" (at 101.95585 84.3 90) (layer "F.SilkS")
-    (effects (font (size 0.6 0.6) (thickness 0.125)))
-  )
   (gr_text "RESET" (at 95.659571 98.9) (layer "F.SilkS")
     (effects (font (size 1 1) (thickness 0.15)))
   )
-  (gr_text "GND" (at 86.068727 108.743053) (layer "F.SilkS")
-    (effects (font (size 0.6 0.6) (thickness 0.125)))
+  (gr_text "Vsec" (at 116.2 100 90) (layer "F.SilkS")
+    (effects (font (size 1 1) (thickness 0.15)))
+  )
+  (gr_text "Vusb" (at 116.2 107 90) (layer "F.SilkS")
+    (effects (font (size 1 1) (thickness 0.15)))
   )
-  (gr_text "GND" (at 98.14585 84.3 90) (layer "F.SilkS")
+  (gr_text "Vsec" (at 116.2 93 90) (layer "F.SilkS")
+    (effects (font (size 1 1) (thickness 0.15)))
+  )
+  (gr_text "GND" (at 86.068727 108.788053) (layer "F.SilkS")
     (effects (font (size 0.6 0.6) (thickness 0.125)))
   )
@@
     (effects (font (size 1 1) (thickness 0.15)))
   )
-  (gr_text "GND" (at 114.070757 108.73712) (layer "F.SilkS")
+  (gr_text "USB" (at 100 83.8 180) (layer "F.SilkS")
+    (effects (font (size 1 1) (thickness 0.15)))
+  )
+  (gr_text "GND" (at 114.070757 108.78212) (layer "F.SilkS")
     (effects (font (size 0.6 0.6) (thickness 0.125)))
   )
-  (gr_text "GND" (at 114.083614 101.029169) (layer "F.SilkS")
+  (gr_text "GND" (at 114.083614 101.694169) (layer "F.SilkS")
     (effects (font (size 0.6 0.6) (thickness 0.125)))
   )
-  (gr_text "Vsec" (at 114.06114 90.00018) (layer "F.SilkS")
+  (gr_text "Vsec" (at 114.06114 91.28518) (layer "F.SilkS")
     (effects (font (size 0.6 0.6) (thickness 0.125)))
   )
-  (gr_text "GND" (at 114.06114 93.40018) (layer "F.SilkS")
+  (gr_text "GND" (at 114.06114 94.68518) (layer "F.SilkS")
     (effects (font (size 0.6 0.6) (thickness 0.125)))
   )
@@
     (effects (font (size 0.75 0.75) (thickness 0.15) italic))
   )
-  (gr_text "D+" (at 100.68585 84.3 90) (layer "F.SilkS")
-    (effects (font (size 0.6 0.6) (thickness 0.15)))
+  (gr_text "Vusb" (at 83.8 107 -90) (layer "F.SilkS")
+    (effects (font (size 1 1) (thickness 0.15)))
   )
   (gr_text "PWR" (at 90 106.5) (layer "F.SilkS")
     (effects (font (size 0.75 0.6) (thickness 0.15)))
   )
-  (gr_text "Vout" (at 114.070757 105.23712) (layer "F.SilkS")
+  (gr_text "Vout" (at 114.070757 105.28212) (layer "F.SilkS")
     (effects (font (size 0.6 0.6) (thickness 0.125)))
   )
@@
     (effects (font (size 0.75 0.6) (thickness 0.15)))
   )
-  (gr_text "D-" (at 99.41585 84.3 90) (layer "F.SilkS")
-    (effects (font (size 0.6 0.6) (thickness 0.15)))
-  )
   (gr_text "back side obstruction(s)" (at 120 75.5) (layer "User.2")
     (effects (font (size 0.5 0.5) (thickness 0.125)) (justify left))
@@
   (segment (start 95.85 93.121335) (end 96.945399 94.216734) (width 0.25) (layer "B.Cu") (net 22))
   (segment (start 96.945399 94.216734) (end 96.945399 102.845399) (width 0.25) (layer "B.Cu") (net 22))
+  (segment (start 114 92.365) (end 115.857511 92.365) (width 1) (layer "F.Cu") (net 23))
   (segment (start 113.902854 91.08) (end 110.95 91.08) (width 1) (layer "F.Cu") (net 23))
+  (segment (start 114 99.365) (end 115.794416 99.365) (width 1) (layer "F.Cu") (net 23))
+  (segment (start 116.067165 99.092251) (end 116.067165 102.731217) (width 1) (layer "F.Cu") (net 23))
   (segment (start 113.902854 91.08) (end 115.468859 91.08) (width 1) (layer "F.Cu") (net 23))
+  (segment (start 115.857511 92.365) (end 116.069587 92.152924) (width 1) (layer "F.Cu") (net 23))
+  (segment (start 116.069587 91.680728) (end 116.069587 92.152924) (width 1) (layer "F.Cu") (net 23))
+  (segment (start 116.069587 92.152924) (end 116.069587 98.236772) (width 1) (layer "F.Cu") (net 23))
   (segment (start 115.323382 103.475) (end 110.94 103.475) (width 1) (layer "F.Cu") (net 23))
-  (segment (start 116.069587 91.680728) (end 116.069587 98.236772) (width 1) (layer "F.Cu") (net 23))
+  (segment (start 115.794416 99.365) (end 116.067165 99.092251) (width 1) (layer "F.Cu") (net 23))
   (segment (start 116.067165 98.239194) (end 116.067165 98.587165) (width 1) (layer "F.Cu") (net 23))
+  (segment (start 116.067165 98.587165) (end 116.067165 99.092251) (width 1) (layer "F.Cu") (net 23))
   (segment (start 115.468859 91.08) (end 116.069587 91.680728) (width 1) (layer "F.Cu") (net 23))
   (segment (start 116.067165 102.731217) (end 115.323382 103.475) (width 1) (layer "F.Cu") (net 23))
   (segment (start 116.069587 98.236772) (end 116.067165 98.239194) (width 1) (layer "F.Cu") (net 23))
-  (segment (start 115.95433 98.7) (end 116.067165 98.587165) (width 1) (layer "F.Cu") (net 23))
-  (segment (start 113.97 98.7) (end 115.95433 98.7) (width 1) (layer "F.Cu") (net 23))
-  (segment (start 116.067165 98.587165) (end 116.067165 102.731217) (width 1) (layer "F.Cu") (net 23))
   (segment (start 89.175 105.0625) (end 89.2125 105.1) (width 0.25) (layer "F.Cu") (net 24))
   (segment (start 89.175 103.6) (end 89.175 105.0625) (width 0.25) (layer "F.Cu") (net 24))
