File: Hardware/Programmer.kicad_sch (KiCad schematic)
At the start: 31 parts, among them J1 Conn_01x07_Male, J2 Conn_01x04_Male, J3 Conn_01x02_Male, J4 Conn_01x02_Male, J5 Conn_01x02_Male, J6 Conn_01x02_Male, J7 Conn_01x08_Male, J9 QWIIC_Stackable, SW1 SW_Push, U1 R1501J033B-T1-JE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

Commit message: Still working on changes to J7/J9
Parts:
- J9: footprint Tinker:QWIIC_Stackable -> Tinker:QWIIC_Stack_II
Connections:
- net ATTACH is gone; now on net RESET: J7.2 (Pin_2)
- net RESET: no longer J7.1 (Pin_1)
- net SCL: no longer J7.3 (Pin_3)
- net SDA: no longer J7.5 (Pin_5)
- net ALERT renamed ~{SCS}0
- net GPIO renamed MOSI
- net POWER_OK2 renamed SCLK
- net POWER_OK3 renamed MISO
- new net ~{SCS}1: J7.5 (Pin_5)
- new net ~{SCS}2: J7.3 (Pin_3)
- new net ~{SCS}3: J7.1 (Pin_1)
Other:
- note added: "I2C"
- note added: "SPI"
- note removed: "Control"
- note removed: "QWIIC"
- title: USB-PD Programmer -> Programmer
Changed lines of the file:
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@@
   (paper "A4")
   (title_block
-    (title "USB-PD Programmer")
-    (rev "0.1.4")
+    (title "Programmer")
+    (rev "0.2.4")
     (company "The Nerd Mage")
   )
@@
     (effects (font (size 1.27 1.27)) (justify left bottom))
   )
-  (text "QWIIC" (at 68.58 95.25 0)
+  (text "I2C" (at 68.58 95.25 0)
     (effects (font (size 2.54 2.54)) (justify left bottom))
   )
@@
     (effects (font (size 5 5) (thickness 1) bold) (justify left bottom))
   )
-  (text "Control" (at 33.02 95.25 0)
+  (text "SPI" (at 33.02 95.25 0)
     (effects (font (size 2.54 2.54)) (justify left bottom))
   )
@@
   (label "XO" (at 143.51 76.2 0)
     (effects (font (size 1.27 1.27)) (justify left bottom))
+  )
+  (global_label "MOSI" (shape bidirectional) (at 40.64 87.63 180) (fields_autoplaced)
+    (effects (font (size 1.27 1.27)) (justify right))
+    (property "Intersheet References" "${INTERSHEET_REFS}" (id 0) (at 33.6307 87.5506 0)
+      (effects (font (size 1.27 1.27)) (justify right) hide)
+    )
   )
   (global_label "DTR" (shape input) (at 132.08 172.72 180) (fields_autoplaced)
@@
     )
   )
-  (global_label "SDA" (shape input) (at 40.64 80.01 180) (fields_autoplaced)
-    (effects (font (size 1.27 1.27) bold) (justify right))
-    (property "Intersheet References" "${INTERSHEET_REFS}" (id 0) (at 34.4684 79.883 0)
-      (effects (font (size 1.27 1.27) bold) (justify right) hide)
+  (global_label "~{SCS}0" (shape bidirectional) (at 40.64 85.09 180) (fields_autoplaced)
+    (effects (font (size 1.27 1.27)) (justify right))
+    (property "Intersheet References" "${INTERSHEET_REFS}" (id 0) (at 33.3283 85.0106 0)
+      (effects (font (size 1.27 1.27)) (justify right) hide)
     )
   )
@@
     (property "Intersheet References" "${INTERSHEET_REFS}" (id 0) (at 130.574 65.9606 0)
       (effects (font (size 1.27 1.27)) (justify right) hide)
-    )
-  )
-  (global_label "POWER_OK3" (shape input) (at 40.64 82.55 180) (fields_autoplaced)
-    (effects (font (size 1.27 1.27) (thickness 0.254) bold) (justify right))
-    (property "Intersheet References" "${INTERSHEET_REFS}" (id 0) (at 26.7879 82.423 0)
-      (effects (font (size 1.27 1.27) (thickness 0.254) bold) (justify right) hide)
-    )
-  )
-  (global_label "GPIO" (shape input) (at 40.64 87.63 180) (fields_autoplaced)
-    (effects (font (size 1.27 1.27) (thickness 0.254) bold) (justify right))
-    (property "Intersheet References" "${INTERSHEET_REFS}" (id 0) (at 33.5613 87.503 0)
-      (effects (font (size 1.27 1.27) (thickness 0.254) bold) (justify right) hide)
     )
   )
@@
     )
   )
+  (global_label "~{SCS}3" (shape bidirectional) (at 40.64 69.85 180) (fields_autoplaced)
+    (effects (font (size 1.27 1.27) (thickness 0.254) bold) (justify right))
+    (property "Intersheet References" "${INTERSHEET_REFS}" (id 0) (at 33.1379 69.723 0)
+      (effects (font (size 1.27 1.27) (thickness 0.254) bold) (justify right) hide)
+    )
+  )
   (global_label "Vout" (shape input) (at 25.4 119.38 180) (fields_autoplaced)
     (effects (font (size 1.27 1.27)) (justify right))
@@
     )
   )
+  (global_label "MISO" (shape bidirectional) (at 40.64 82.55 180) (fields_autoplaced)
+    (effects (font (size 1.27 1.27)) (justify right))
+    (property "Intersheet References" "${INTERSHEET_REFS}" (id 0) (at 33.6307 82.4706 0)
+      (effects (font (size 1.27 1.27)) (justify right) hide)
+    )
+  )
   (global_label "DCD" (shape input) (at 167.64 71.12 0) (fields_autoplaced)
     (effects (font (size 1.27 1.27)) (justify left))
@@
     )
   )
-  (global_label "ALERT" (shape input) (at 40.64 85.09 180) (fields_autoplaced)
-    (effects (font (size 1.27 1.27) bold) (justify right))
-    (property "Intersheet References" "${INTERSHEET_REFS}" (id 0) (at 32.5332 84.963 0)
-      (effects (font (size 1.27 1.27) bold) (justify right) hide)
-    )
-  )
   (global_label "RTS" (shape input) (at 132.08 181.61 180) (fields_autoplaced)
     (effects (font (size 1.27 1.27) (thickness 0.254) bold) (justify right))
@@
     )
   )
-  (global_label "ATTACH" (shape input) (at 40.64 72.39 180) (fields_autoplaced)
-    (effects (font (size 1.27 1.27) (thickness 0.254) bold) (justify right))
-    (property "Intersheet References" "${INTERSHEET_REFS}" (id 0) (at 31.3236 72.263 0)
-      (effects (font (size 1.27 1.27) (thickness 0.254) bold) (justify right) hide)
-    )
-  )
   (global_label "Vsec" (shape input) (at 87.63 167.64 180) (fields_autoplaced)
     (effects (font (size 1.27 1.27)) (justify right))
     (property "Intersheet References" "${INTERSHEET_REFS}" (id 0) (at 80.9231 167.5606 0)
       (effects (font (size 1.27 1.27)) (justify right) hide)
-    )
-  )
-  (global_label "POWER_OK2" (shape input) (at 40.64 77.47 180) (fields_autoplaced)
-    (effects (font (size 1.27 1.27) (thickness 0.254) bold) (justify right))
-    (property "Intersheet References" "${INTERSHEET_REFS}" (id 0) (at 26.7879 77.343 0)
-      (effects (font (size 1.27 1.27) (thickness 0.254) bold) (justify right) hide)
     )
   )
@@
     )
   )
+  (global_label "RESET" (shape input) (at 40.64 72.39 180) (fields_autoplaced)
+    (effects (font (size 1.27 1.27) (thickness 0.254) bold) (justify right))
+    (property "Intersheet References" "${INTERSHEET_REFS}" (id 0) (at 32.2913 72.263 0)
+      (effects (font (size 1.27 1.27) (thickness 0.254) bold) (justify right) hide)
+    )
+  )
   (global_label "+3V3" (shape input) (at 203.2 68.58 0) (fields_autoplaced)
     (effects (font (size 1.27 1.27)) (justify left))
@@
     )
   )
-  (global_label "RESET" (shape input) (at 40.64 69.85 180) (fields_autoplaced)
-    (effects (font (size 1.27 1.27) (thickness 0.254) bold) (justify right))
-    (property "Intersheet References" "${INTERSHEET_REFS}" (id 0) (at 32.2913 69.723 0)
-      (effects (font (size 1.27 1.27) (thickness 0.254) bold) (justify right) hide)
+  (global_label "SCLK" (shape bidirectional) (at 40.64 77.47 180) (fields_autoplaced)
+    (effects (font (size 1.27 1.27)) (justify right))
+    (property "Intersheet References" "${INTERSHEET_REFS}" (id 0) (at 33.4493 77.3906 0)
+      (effects (font (size 1.27 1.27)) (justify right) hide)
     )
   )
@@
     )
   )
-  (global_label "SCL" (shape input) (at 40.64 74.93 180) (fields_autoplaced)
+  (global_label "~{SCS}2" (shape bidirectional) (at 40.64 74.93 180) (fields_autoplaced)
     (effects (font (size 1.27 1.27) (thickness 0.254) bold) (justify right))
-    (property "Intersheet References" "${INTERSHEET_REFS}" (id 0) (at 34.5289 74.803 0)
+    (property "Intersheet References" "${INTERSHEET_REFS}" (id 0) (at 33.1379 74.803 0)
+      (effects (font (size 1.27 1.27) (thickness 0.254) bold) (justify right) hide)
+    )
+  )
+  (global_label "~{SCS}1" (shape bidirectional) (at 40.64 80.01 180) (fields_autoplaced)
+    (effects (font (size 1.27 1.27) (thickness 0.254) bold) (justify right))
+    (property "Intersheet References" "${INTERSHEET_REFS}" (id 0) (at 33.1379 79.883 0)
       (effects (font (size 1.27 1.27) (thickness 0.254) bold) (justify right) hide)
     )
@@
   )
   (symbol (lib_id "Connector_QWIIC_Stackable:QWIIC_Stackable") (at 80.01 72.39 0) (unit 1)
-    (in_bom no) (on_board no) (fields_autoplaced)
+    (in_bom no) (on_board yes) (fields_autoplaced)
     (property "Reference" "J9" (id 0) (at 82.55 72.7455 0)
       (effects (font (size 1.27 1.27)) (justify left))
@@
       (effects (font (size 1.27 1.27)) (justify left))
     )
-    (property "Footprint" "Tinker:QWIIC_Stackable" (id 2) (at 81.28 82.55 0)
+    (property "Footprint" "Tinker:QWIIC_Stack_II" (id 2) (at 81.28 82.55 0)
       (effects (font (size 1.27 1.27)) (justify left) hide)
     )
@@
     )
     (path "/b8a785f2-9322-4569-b066-f0e9fc64eafd"
-      (reference "J9") (unit 1) (value "QWIIC_Stackable") (footprint "Tinker:QWIIC_Stackable")
+      (reference "J9") (unit 1) (value "QWIIC_Stackable") (footprint "Tinker:QWIIC_Stack_II")
     )
     (path "/c9a27b82-cdac-46ce-ab09-549b2bdc6694"

Commit message: Still migrating to 0.2.x
Connections:
- net ~{SCS}3 renamed ~{RESET}
Changed lines of the file:
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@@
-    )
-  )
-  (global_label "~{SCS}3" (shape bidirectional) (at 40.64 69.85 180) (fields_autoplaced)
-    (effects (font (size 1.27 1.27) (thickness 0.254) bold) (justify right))
-    (property "Intersheet References" "${INTERSHEET_REFS}" (id 0) (at 33.1379 69.723 0)
-      (effects (font (size 1.27 1.27) (thickness 0.254) bold) (justify right) hide)
     )
   )
@@
     )
   )
+  (global_label "~{RESET}" (shape input) (at 40.64 69.85 180) (fields_autoplaced)
+    (effects (font (size 1.27 1.27) (thickness 0.254) bold) (justify right))
+    (property "Intersheet References" "${INTERSHEET_REFS}" (id 0) (at 32.2913 69.723 0)
+      (effects (font (size 1.27 1.27) (thickness 0.254) bold) (justify right) hide)
+    )
+  )
