File: Hardware/Controller-8285.kicad_pcb (KiCad board)
At the start: 2 copper layers, 34 x 34 mm, 34 parts, among them J1 Conn_01x07_Male, J10 Conn_Coaxial, J2 Conn_01x04_Male, J3 Conn_01x02_Male, J4 Conn_01x02_Male, J5 Conn_01x02_Male, J6 Conn_01x02_Male, J7 Conn_01x08_Male, J9 QWIIC_Stackable, Q1 UMH3N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

Commit message: Working on changes to J7/J9
Parts:
- moved J6 1.28 mm to (114.0, 92.4)
- moved J5 0.66 mm to (114.0, 99.4)
- moved JP1 0.20 mm to (108.1, 89.9)
- moved C1 0.08 mm to (100.0, 90.6)
Connections:
- J7 pad 1: IO16 -> ~{SCS}3
- J7 pad 2: ATTACH -> DEV_RESET
- J7 pad 3: SCL -> ~{SCS}2
- J7 pad 4: IO12 -> IO14
- J7 pad 5: SDA -> ~{SCS}1
- J7 pad 6: IO13 -> IO12
- J7 pad 7: ALERT -> IO15
- J7 pad 8: IO15 -> IO13
- U1 pad 14: ALERT -> IO2
- U1 pad 8: IO16 -> DEV_RESET
- U1 pad 9: ATTACH -> IO14
Routing:
- net IO16: track 16.0 -> 0.00 mm, vias 1 -> 0
- net DEV_RESET: track 0.00 -> 14.8 mm
- net ALERT: track 14.3 -> 0.00 mm, vias 1 -> 0
- net IO14: track 0.00 -> 13.9 mm
- net ATTACH: track 13.4 -> 0.00 mm
- net SDA: track 25.0 -> 14.9 mm
- net SCL: track 25.4 -> 18.5 mm
- net IO15: track 12.6 -> 15.0 mm
- net Vsec: track 15.9 -> 16.9 mm
- net IO12: track 13.4 -> 13.9 mm
- net IO13: track 12.6 -> 13.1 mm
Other:
- board text added: ">RST"
- board text added: "I2C"
- board text added: "SPI"
- board text added: "USB"
- board text added: "Vusb"
- board text removed: "BIG Empty Waste Man..."
- board text removed: "DEV-IO"
- board text removed: "DEV-RST"
- board text removed: "QWIIC"

Commit message: Still migrating to 0.2.x
Connections:
- J7 pad 1: ~{SCS}3 -> IO2
Routing:
- net IO2: track 0.00 -> 13.4 mm, vias 0 -> 1
- net SDA: track 14.9 -> 14.1 mm
- net SCL: track 18.5 -> 17.9 mm

Commit message: Bit more of the RP2040...
Changed lines of the file:
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@@
     (property "Sheetname" "")
     (attr smd)
-    (fp_text reference "R3" (at -2.053028 0.041061 90) (layer "F.SilkS")
+    (fp_text reference "R3" (at -1.811315 0.041061 180) (layer "F.SilkS")
       (effects (font (size 0.6 0.6) (thickness 0.15)))
     )
@@
     (property "Sheetname" "")
     (attr smd)
-    (fp_text reference "R6" (at -2.162523 0.247452 90) (layer "F.SilkS")
+    (fp_text reference "R6" (at -1.811315 0 180) (layer "F.SilkS")
       (effects (font (size 0.6 0.6) (thickness 0.15)))
     )

Commit message: Some tweaks
Other:
- board text added: "${TITLE}"
- board text removed: "${TITLE} (etc...etc...etc...)"
- board text removed: "{dblquote}Universal{dblquote}"
Changed lines of the file:
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@@
   )
   (footprint "Tinker:SW_Push_TS273014TP" (layer "F.Cu")
-    (at 108.482364 110.588685 180)
+    (at 108.5 110.6 180)
     (descr "CK components KMR2 tactile switch http://www.ckswitches.com/media/1479/kmr2.pdf")
     (tags "tactile switch kmr2")
@@
     (effects (font (size 0.6 0.6) (thickness 0.15)) (justify right))
   )
-  (gr_text "{dblquote}Universal{dblquote}" (at 90.471181 110.337609 90) (layer "F.SilkS")
-    (effects (font (size 0.75 0.75) (thickness 0.15) italic))
-  )
   (gr_text "TxD" (at 97.429475 115.901362 270) (layer "F.SilkS")
     (effects (font (size 0.6 0.6) (thickness 0.125)))
@@
     (effects (font (size 0.6 0.6) (thickness 0.125)))
   )
-  (gr_text "RESET" (at 108.384923 113.183331) (layer "F.SilkS")
+  (gr_text "RESET" (at 108.5 113) (layer "F.SilkS")
     (effects (font (size 1 1) (thickness 0.15)))
   )
-  (gr_text "${TITLE}\n(etc...etc...etc...)" (at 92.333688 110.4263 90) (layer "F.SilkS")
+  (gr_text "${TITLE}" (at 91.591459 107.527079 45) (layer "F.SilkS")
     (effects (font (size 0.75 0.75) (thickness 0.15)))
   )
@@
   (segment (start 102.117608 98.582074) (end 102.298097 98.762563) (width 0.3) (layer "F.Cu") (net 6))
   (segment (start 103.655521 96.0367) (end 103.655521 95.9367) (width 0.3) (layer "F.Cu") (net 6))
+  (segment (start 104.916762 109.763685) (end 106.636315 109.763685) (width 0.6) (layer "F.Cu") (net 6))
   (segment (start 101.944544 101.59099) (end 102.257898 101.59099) (width 0.25) (layer "F.Cu") (net 6))
-  (segment (start 104.916762 109.763685) (end 103.417474 109.763685) (width 0.25) (layer "F.Cu") (net 6))
   (segment (start 96.604841 100.212956) (end 96.677422 100.212956) (width 0.25) (layer "F.Cu") (net 6))
   (segment (start 103.306561 97.945626) (end 103.448197 98.087263) (width 0.3) (layer "F.Cu") (net 6))
   (segment (start 102.155521 94.4367) (end 97.8633 94.4367) (width 0.3) (layer "F.Cu") (net 6))
   (segment (start 103.987597 89.926721) (end 107.49 89.926721) (width 0.6) (layer "F.Cu") (net 6))
+  (segment (start 106.65 109.75) (end 110.35 109.75) (width 0.6) (layer "F.Cu") (net 6))
   (segment (start 103.671821 96.053) (end 103.671821 97.863639) (width 0.3) (layer "F.Cu") (net 6))
   (segment (start 102.754056 97.945626) (end 103.306561 97.945626) (width 0.3) (layer "F.Cu") (net 6))
   (segment (start 97.8633 94.4367) (end 97.8 94.5) (width 0.3) (layer "F.Cu") (net 6))
+  (segment (start 106.636315 109.763685) (end 106.65 109.75) (width 0.6) (layer "F.Cu") (net 6))
   (segment (start 104.773029 102.051971) (end 105.225 101.6) (width 0.25) (layer "F.Cu") (net 6))
+  (segment (start 103.417474 109.763685) (end 104.916762 109.763685) (width 0.6) (layer "F.Cu") (net 6))
   (segment (start 103.671821 97.863639) (end 103.448197 98.087263) (width 0.3) (layer "F.Cu") (net 6))
   (segment (start 102.117608 98.582074) (end 102.754056 97.945626) (width 0.3) (layer "F.Cu") (net 6))
-  (segment (start 106.632364 109.738685) (end 104.941762 109.738685) (width 0.25) (layer "F.Cu") (net 6))
   (segment (start 96.636903 111.231967) (end 96.19 111.67887) (width 0.25) (layer "F.Cu") (net 6))
   (segment (start 103.655521 96.0367) (end 103.671821 96.053) (width 0.3) (layer "F.Cu") (net 6))
@@
   (segment (start 103.428343 109.752816) (end 103.417474 109.763685) (width 0.6) (layer "F.Cu") (net 6))
   (segment (start 103.68114 98.320205) (end 103.68114 98.797793) (width 0.3) (layer "F.Cu") (net 6))
-  (segment (start 110.332364 109.828458) (end 106.632364 109.828458) (width 0.25) (layer "F.Cu") (net 6))
   (segment (start 96.677422 100.212956) (end 96.994796 100.53033) (width 0.25) (layer "F.Cu") (net 6))
   (segment (start 102.718879 102.051971) (end 104.773029 102.051971) (width 0.25) (layer "F.Cu") (net 6))
@@
   (segment (start 103.340755 89.726721) (end 102.55 90.517476) (width 0.6) (layer "F.Cu") (net 6))
   (segment (start 103.68114 98.797793) (end 103.009263 99.46967) (width 0.3) (layer "F.Cu") (net 6))
-  (segment (start 104.941762 109.738685) (end 104.916762 109.763685) (width 0.25) (layer "F.Cu") (net 6))
   (segment (start 102.616576 101.949668) (end 102.718879 102.051971) (width 0.25) (layer "F.Cu") (net 6))
   (segment (start 96.19 111.67887) (end 96.19 114) (width 0.25) (layer "F.Cu") (net 6))
@@
   (segment (start 104.941762 111.438685) (end 104.916762 111.413685) (width 0.25) (layer "F.Cu") (net 7))
   (segment (start 103.132905 110.625867) (end 104.128944 110.625867) (width 0.25) (layer "F.Cu") (net 7))
-  (segment (start 110.332364 111.528458) (end 106.632364 111.528458) (width 0.25) (layer "F.Cu") (net 7))
   (segment (start 102.557038 110.05) (end 103.132905 110.625867) (width 0.25) (layer "F.Cu") (net 7))
   (segment (start 101.89 110.05) (end 102.557038 110.05) (width 0.25) (layer "F.Cu") (net 7))
   (segment (start 103.656387 101.126971) (end 103.601845 101.126971) (width 0.25) (layer "F.Cu") (net 7))
+  (segment (start 106.65 111.45) (end 110.35 111.45) (width 0.25) (layer "F.Cu") (net 7))
   (via (at 105.634625 111.464139) (size 0.5) (drill 0.3) (layers "F.Cu" "B.Cu") (net 7))
   (via (at 103.656387 101.126971) (size 0.4) (drill 0.3) (layers "F.Cu" "B.Cu") (net 7))

Commit message: Working on the RP2040 & cleaning up stuff...
Other:
- board text added: "Stacked Rabbit"
Changed lines of the file:
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@@
     (effects (font (size 0.6 0.6) (thickness 0.125)))
+  )
+  (gr_text "Stacked Rabbit" (at 90.876215 106.573419 45) (layer "F.SilkS")
+    (effects (font (size 0.75 0.75) (thickness 0.15) italic))
   )
   (gr_text "GND" (at 99.969475 115.901362 270) (layer "F.SilkS")

Commit message: Whole bunch of cleanup & 3D rework
Parts:
- J9: value QWIIC_Stackable -> QWIIC_Stack_II
Changed lines of the file:
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@@
     )
     (pad_to_mask_clearance 0)
+    (grid_origin 100 100)
     (pcbplotparams
       (layerselection 0x0000030_7ffffffe)
@@
       (effects (font (size 0.6 0.6) (thickness 0.15)))
     )
-    (fp_text value "QWIIC_Stackable" (at 0 4.084197 -90) (layer "F.Fab")
+    (fp_text value "QWIIC_Stack_II" (at 0 4.084197 -90) (layer "F.Fab")
       (effects (font (size 1 1) (thickness 0.15)))
     )
@@
     (fp_line (start -1.35 -0.73) (end 1.35 -0.73) (layer "F.CrtYd") (width 0.05))
     (pad "1" smd custom (at -0.65 0 180) (size 1 0.2) (layers "F.Cu" "F.Mask")
-      (net 29 "Vsec") (pinfunction "A") (pintype "passive") (zone_connect 2)
+      (net 29 "Vsec") (pinfunction "A") (pintype "passive+no_connect") (zone_connect 2)
       (options (clearance outline) (anchor rect))
       (primitives
@@
     (fp_line (start 1.079472 -0.635) (end 1.079472 1.905) (layer "F.Fab") (width 0.1))
     (pad "1" smd rect (at 1.35 0) (size 1.8 0.65) (layers "B.Cu" "B.Paste" "B.Mask")
-      (net 29 "Vsec") (pinfunction "Pin_1") (pintype "passive"))
+      (net 29 "Vsec") (pinfunction "Pin_1") (pintype "passive+no_connect"))
     (pad "1" thru_hole rect (at 0 0) (size 1 1) (drill 0.65) (layers *.Cu *.Mask)
-      (net 29 "Vsec") (pinfunction "Pin_1") (pintype "passive"))
+      (net 29 "Vsec") (pinfunction "Pin_1") (pintype "passive+no_connect"))
     (pad "2" smd rect (at -1.35 1.27) (size 1.8 0.65) (layers "B.Cu" "B.Paste" "B.Mask")
       (net 3 "GND") (pinfunction "Pin_2") (pintype "passive"))
@@
     (fp_line (start -1.020528 1.905) (end -1.020528 -0.11) (layer "F.Fab") (width 0.1))
     (pad "1" smd rect (at 1.35 0) (size 1.8 0.65) (layers "B.Cu" "B.Paste" "B.Mask")
-      (net 29 "Vsec") (pinfunction "Pin_1") (pintype "passive"))
+      (net 29 "Vsec") (pinfunction "Pin_1") (pintype "passive+no_connect"))
     (pad "1" thru_hole rect (at 0 0) (size 1 1) (drill 0.65) (layers *.Cu *.Mask)
-      (net 29 "Vsec") (pinfunction "Pin_1") (pintype "passive"))
+      (net 29 "Vsec") (pinfunction "Pin_1") (pintype "passive+no_connect"))
     (pad "2" smd rect (at -1.35 1.27) (size 1.8 0.65) (layers "B.Cu" "B.Paste" "B.Mask")
       (net 3 "GND") (pinfunction "Pin_2") (pintype "passive"))
