File: Hardware/Controller-8285.kicad_sch (KiCad schematic)
At the start: 31 parts, among them J1 Conn_01x07_Male, J10 Conn_Coaxial, J2 Conn_01x04_Male, J3 Conn_01x02_Male, J4 Conn_01x02_Male, J5 Conn_01x02_Male, J6 Conn_01x02_Male, J7 Conn_01x08_Male, J8 QWIIC_Vertical, J9 QWIIC_Stackable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

Commit message: Working on changes to J7/J9
Connections:
- net IO12: now also J7.6 (Pin_6); no longer J7.4 (Pin_4)
- net IO13: now also J7.8 (Pin_8); no longer J7.6 (Pin_6)
- net IO14: now also J7.4 (Pin_4); no longer J7.2 (Pin_2)
- net SCL: no longer J7.3 (Pin_3)
- net SDA: no longer J7.5 (Pin_5)
- net ~{SCS}: no longer J7.8 (Pin_8)
- net IO16 renamed DEV_RESET
- net DEV_RESET: now also J7.2 (Pin_2); no longer J7.1 (Pin_1)
- new net ~{SCS}1: J7.5 (Pin_5)
- new net ~{SCS}2: J7.3 (Pin_3)
- new net ~{SCS}3: J7.1 (Pin_1)
Other:
- title: USB-C PD Controller -> Controller-8285

Commit message: Still migrating to 0.2.x
Connections:
- net ~{SCS}3 is gone; now on net IO2: J7.1 (Pin_1)
Changed lines of the file:
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@@
-    )
-  )
-  (global_label "~{SCS}3" (shape bidirectional) (at 161.29 77.47 180) (fields_autoplaced)
-    (effects (font (size 1.27 1.27) (thickness 0.254) bold) (justify right))
-    (property "Intersheet References" "${INTERSHEET_REFS}" (id 0) (at 153.7879 77.343 0)
-      (effects (font (size 1.27 1.27) (thickness 0.254) bold) (justify right) hide)
     )
   )
@@
     (property "Intersheet References" "${INTERSHEET_REFS}" (id 0) (at 133.8279 48.1806 0)
       (effects (font (size 1.27 1.27)) (justify left) hide)
+    )
+  )
+  (global_label "~{DEV_RESET}" (shape input) (at 161.29 77.47 180) (fields_autoplaced)
+    (effects (font (size 1.27 1.27) (thickness 0.254) bold) (justify right))
+    (property "Intersheet References" "${INTERSHEET_REFS}" (id 0) (at 148.466 77.343 0)
+      (effects (font (size 1.27 1.27) (thickness 0.254) bold) (justify right) hide)
     )
   )
@@
     )
   )
+  (global_label "~{DEV_RESET}" (shape output) (at 157.48 100.33 0) (fields_autoplaced)
+    (effects (font (size 1.27 1.27) (thickness 0.254) bold) (justify left))
+    (property "Intersheet References" "${INTERSHEET_REFS}" (id 0) (at 170.304 100.203 0)
+      (effects (font (size 1.27 1.27) (thickness 0.254) bold) (justify left) hide)
+    )
+  )

Commit message: Working on the RP2040 & cleaning up stuff...
Parts:
- J9: value QWIIC_Stackable -> QWIIC_Stack_II
Other:
- note added: "I2C"
- note removed: "Footprint(s) only"
- moved on the sheet: J2, J3, J4, J5, J6, J7, J8, J9, JP1

Commit message: Whole bunch of cleanup & 3D rework
Other:
- moved on the sheet: C1
