File: Hardware/Controller-RP2040.kicad_pcb (KiCad board)
At the start: 2 copper layers, 34 x 34 mm, 43 parts, among them J2 Conn_01x04_Male, J3 Conn_01x02_Male, J4 Conn_01x02_Male, J5 Conn_01x02_Male, J6 Conn_01x02_Male, J7 Conn_01x08_Male, J9 QWIIC_Stackable, U1 RP2040, U2 W25Q32JVXGIQ, Y1 12MHz

Commit message: Bit more of the RP2040...
Parts:
- moved J6 1.28 mm to (114.0, 92.4)
- moved J5 0.66 mm to (114.0, 99.4)
Connections:
- net DEV_RST renamed ~{RESET}
- J7 pad 2: SCLK -> RESET
- J7 pad 3: SCL -> ~{SCS}2
- J7 pad 4: MISO -> SCLK
- J7 pad 5: SDA -> ~{SCS}1
- J7 pad 6: MOSI -> MISO
- J7 pad 7: DEV_GPIO -> ~{SCS}0
- J7 pad 8: ~{SCS} -> MOSI
- U1 pad 14: io11 -> MOSI
- U1 pad 15: io12 -> MISO
- U1 pad 16: io13 -> SCLK
- U1 pad 17: io14 -> ~{SCS}0
Routing:
- net ~{SCS}0: track 0.00 -> 14.4 mm, vias 0 -> 1
- net SCLK: track 0.00 -> 13.1 mm, vias 0 -> 1
- net MISO: track 0.00 -> 11.8 mm, vias 0 -> 1
- net SDA: track 9.73 -> 0.00 mm
- net MOSI: track 0.00 -> 9.59 mm, vias 0 -> 1
- net SCL: track 6.91 -> 0.00 mm
Other:
- board text added: "2,1,0"
- board text added: ">RST"
- board text added: ">~{RST}"
- board text added: "I2C"
- board text added: "SPI"
- board text added: "USB"
- board text removed: "DEV-IO"
- board text removed: "DEV-RST"
- board text removed: "QWIIC"

Commit message: I2C on the RP2040
Parts:
- moved C6 2.09 mm to (93.6, 96.4)
Connections:
- net ~{SCS}0 renamed io14
- U1 pad 6: io4 -> SDA
- U1 pad 7: io5 -> SCL
Routing:
- net SDA: track 0.00 -> 11.7 mm
- net SCL: track 0.00 -> 11.1 mm
- net +3V3: track 86.2 -> 85.3 mm
- net GND: vias 11 -> 12

Commit message: Working on the RP2040 & cleaning up stuff...
Parts:
- added SW1: SW_Push, Tinker:SW_Push_TS273014TP, F.Cu at (108.5, 110.6)
- added SW2: SW_Push, Tinker:SW_Push_TS273014TP, F.Cu at (91.5, 110.6)
- J9: value QWIIC_Stackable -> QWIIC_Stack_II
- moved C9 18.4 mm to (106.0, 96.5), turned to 0 degrees
- moved C10 17.8 mm to (94.8, 93.2)
- moved R7 1.98 mm to (96.7, 94.7), turned to 180 degrees
- moved C11 1.30 mm to (94.9, 97.4)
- moved C6 1.30 mm to (94.9, 96.4)
- moved C5 0.40 mm to (106.0, 95.5)
- moved C7 0.26 mm to (106.0, 97.5)
- moved D2 0.19 mm to (109.0, 94.0), turned to 0 degrees
- moved R8 0.19 mm to (109.0, 93.0), turned to 0 degrees
Connections:
- net /Xin renamed Net-(C1-Pad1)
- net RESET renamed DEV_RESET
- net ~{RESET} renamed ~{DEV_RESET}
- U2 pad 9: unconnected-(U2-Pad9) -> GND
- Y1 pad 2: GND -> unconnected-(Y1-Pad2)
Routing:
- net BootMode: track 0.00 -> 21.9 mm, vias 0 -> 2
- net Reset: track 0.00 -> 14.5 mm, vias 0 -> 2
- net +3V3: track 85.3 -> 71.6 mm
- net +1V1: track 22.3 -> 20.5 mm
- net QSPI SS: track 4.97 -> 3.26 mm
- net SCL: track 11.1 -> 11.6 mm
Other:
- board text added: "MODE"
- board text added: "RESET"
