File: Hardware/Programmer.kicad_pcb (KiCad board)
At the start: 2 copper layers, 34 x 34 mm, 36 parts, among them J1 Conn_01x07_Male, J2 Conn_01x04_Male, J3 Conn_01x02_Male, J4 Conn_01x02_Male, J5 Conn_01x02_Male, J6 Conn_01x02_Male, J7 Conn_01x08_Male, SW1 SW_Push, U1 R1501J033B-T1-JE, U2 CH340G/C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

Commit message: Still working on changes to J7/J9
Parts:
- added J9: QWIIC_Stackable, Tinker:QWIIC_Stack_II, F.Cu at (87.3, 93.0)
- moved J6 1.28 mm to (114.0, 92.4)
- moved C6 1.00 mm to (103.0, 89.7)
- moved J5 0.66 mm to (114.0, 99.4)
- moved J4 0.05 mm to (114.0, 106.4)
Connections:
- net ALERT renamed ~{SCS}0
- net GPIO renamed MOSI
- net POWER_OK2 renamed SCLK
- net POWER_OK3 renamed MISO
- net SCL renamed ~{SCS}2
- net SDA renamed ~{SCS}1
- J7 pad 1: RESET -> ~{SCS}3
- J7 pad 2: ATTACH -> RESET
Other:
- board text added: "100 , 80"
- board text added: ">RST"
- board text added: "MISO"
- board text added: "MOSI"
- board text added: "SCL"
- board text added: "SCLK"
- board text added: "SDA"
- board text added: "SPI"
- board text added: "USB"
- board text added: "Vusb"
- board text added: "~{SCS}"

Commit message: Still working on changes to J7/J9...
Other:
- board text removed: "100 , 80"
Changed lines of the file:
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@@
     (effects (font (size 0.6 0.6) (thickness 0.125)))
-  )
-  (gr_text "100 , 80" (at 100 80) (layer "F.SilkS")
-    (effects (font (size 1 1) (thickness 0.15)))
   )
   (gr_text "3v3" (at 96.191516 115.802425 270) (layer "F.SilkS")

Commit message: Still migrating to 0.2.x
Connections:
- net ~{SCS}3 renamed ~{RESET}
Changed lines of the file:
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@@
   (net 32 "Net-(R7-Pad1)")
   (net 33 "Vcc?")
-  (net 34 "~{SCS}3")
+  (net 34 "~{RESET}")
   (net 35 "~{SCS}2")
   (net 36 "SCLK")
@@
     (tags "resistor")
     (property "LCSC" "C21190")
-    (property "Sheetfile" "USB-PD Programmer.kicad_sch")
+    (property "Sheetfile" "Programmer.kicad_sch")
     (property "Sheetname" "")
     (attr smd)
@@
     (tags "resistor")
     (property "LCSC" "C21190")
-    (property "Sheetfile" "USB-PD Programmer.kicad_sch")
+    (property "Sheetfile" "Programmer.kicad_sch")
     (property "Sheetname" "")
     (attr smd)
@@
     (tags "Through hole pin header THT 2x04 1.27mm double row")
     (property "LCSC" "C2881786 + C2684732")
-    (property "Sheetfile" "USB-PD Programmer.kicad_sch")
+    (property "Sheetfile" "Programmer.kicad_sch")
     (property "Sheetname" "")
     (property "exclude_from_bom" "")
@@
     (fp_line (start -1.07 0.2175) (end -0.2175 -0.635) (layer "F.Fab") (width 0.1))
     (pad "1" thru_hole rect (at 0 0) (size 1 1) (drill 0.65) (layers *.Cu *.Mask)
-      (net 34 "~{SCS}3") (pinfunction "Pin_1") (pintype "passive"))
+      (net 34 "~{RESET}") (pinfunction "Pin_1") (pintype "passive"))
     (pad "1" smd rect (at -1.195 0) (size 2.1 0.75) (layers "B.Cu" "B.Paste" "B.Mask")
-      (net 34 "~{SCS}3") (pinfunction "Pin_1") (pintype "passive"))
+      (net 34 "~{RESET}") (pinfunction "Pin_1") (pintype "passive"))
     (pad "2" thru_hole oval (at 1.27 0) (size 1 1) (drill 0.65) (layers *.Cu *.Mask)
       (net 9 "RESET") (pinfunction "Pin_2") (pintype "passive"))
@@
     (tags "capacitor handsolder")
     (property "LCSC" "C325469")
-    (property "Sheetfile" "USB-PD Programmer.kicad_sch")
+    (property "Sheetfile" "Programmer.kicad_sch")
     (property "Sheetname" "")
     (attr smd)
@@
     (tags "resistor handsolder")
     (property "LCSC" "C25804")
-    (property "Sheetfile" "USB-PD Programmer.kicad_sch")
+    (property "Sheetfile" "Programmer.kicad_sch")
     (property "Sheetname" "")
     (attr smd)
@@
     (tags "capacitor handsolder")
     (property "LCSC" "C325469")
-    (property "Sheetfile" "USB-PD Programmer.kicad_sch")
+    (property "Sheetfile" "Programmer.kicad_sch")
     (property "Sheetname" "")
     (attr smd)
@@
     (tags "SOIC SO")
     (property "LCSC" "C14267/C84681")
-    (property "Sheetfile" "USB-PD Programmer.kicad_sch")
+    (property "Sheetfile" "Programmer.kicad_sch")
     (property "Sheetname" "")
     (attr smd)
@@
     (descr "JST SH series connector, SM04B-SRSS-TB (http://www.jst-mfg.com/product/pdf/eng/eSH.pdf), generated with kicad-footprint-generator")
     (tags "connector JST SH top entry")
-    (property "Sheetfile" "USB-PD Programmer.kicad_sch")
+    (property "Sheetfile" "Programmer.kicad_sch")
     (property "Sheetname" "")
     (property "exclude_from_bom" "")
@@
     (property "LCSC" "C89246")
     (property "P/N" "TAJB226M010RNJ")
-    (property "Sheetfile" "USB-PD Programmer.kicad_sch")
+    (property "Sheetfile" "Programmer.kicad_sch")
     (property "Sheetname" "")
     (attr smd)
@@
     (tags "capacitor handsolder")
     (property "LCSC" "C235731")
-    (property "Sheetfile" "USB-PD Programmer.kicad_sch")
+    (property "Sheetfile" "Programmer.kicad_sch")
     (property "Sheetname" "")
     (attr smd)
@@
     (tags "SMD SMT crystal")
     (property "LCSC" "C2842275")
-    (property "Sheetfile" "USB-PD Programmer.kicad_sch")
+    (property "Sheetfile" "Programmer.kicad_sch")
     (property "Sheetname" "")
     (attr smd)
@@
     (tags "resistor")
     (property "LCSC" "C21190")
-    (property "Sheetfile" "USB-PD Programmer.kicad_sch")
+    (property "Sheetfile" "Programmer.kicad_sch")
     (property "Sheetname" "")
     (attr smd)
@@
     (tags "tactile switch kmr2")
     (property "LCSC" "C2858276")
-    (property "Sheetfile" "USB-PD Programmer.kicad_sch")
+    (property "Sheetfile" "Programmer.kicad_sch")
     (property "Sheetname" "")
     (attr smd)
@@
     (descr "JST SH series connector, SM04B-SRSS-TB (http://www.jst-mfg.com/product/pdf/eng/eSH.pdf), generated with kicad-footprint-generator")
     (tags "connector JST SH top entry")
-    (property "Sheetfile" "USB-PD Programmer.kicad_sch")
+    (property "Sheetfile" "Programmer.kicad_sch")
     (property "Sheetname" "")
     (property "exclude_from_bom" "")
@@
     (tags "resistor")
     (property "LCSC" "C21190")
-    (property "Sheetfile" "USB-PD Programmer.kicad_sch")
+    (property "Sheetfile" "Programmer.kicad_sch")
     (property "Sheetname" "")
     (attr smd)
@@
     (tags "LED")
     (property "LCSC" "C434421")
-    (property "Sheetfile" "USB-PD Programmer.kicad_sch")
+    (property "Sheetfile" "Programmer.kicad_sch")
     (property "Sheetname" "")
     (attr smd)
@@
     (tags "LED")
     (property "LCSC" "C434420")
-    (property "Sheetfile" "USB-PD Programmer.kicad_sch")
+    (property "Sheetfile" "Programmer.kicad_sch")
     (property "Sheetname" "")
     (attr smd)
@@
     (tags "resistor handsolder")
     (property "LCSC" "C25804")
-    (property "Sheetfile" "USB-PD Programmer.kicad_sch")
+    (property "Sheetfile" "Programmer.kicad_sch")
     (property "Sheetname" "")
     (attr smd)
@@
     (descr "JST SH series connector, SM04B-SRSS-TB (http://www.jst-mfg.com/product/pdf/eng/eSH.pdf), generated with kicad-footprint-generator")
     (tags "connector JST SH top entry")
-    (property "Sheetfile" "USB-PD Programmer.kicad_sch")
+    (property "Sheetfile" "Programmer.kicad_sch")
     (property "Sheetname" "")
     (property "exclude_from_bom" "")
@@
     (tags "resistor")
     (property "LCSC" "C21190")
-    (property "Sheetfile" "USB-PD Programmer.kicad_sch")
+    (property "Sheetfile" "Programmer.kicad_sch")
     (property "Sheetname" "")
     (attr smd)
@@
     (property "Manufacturer_Part_Number" "R1501J033B-T1-JE")
     (property "Reference_1" "IC")
-    (property "Sheetfile" "USB-PD Programmer.kicad_sch")
+    (property "Sheetfile" "Programmer.kicad_sch")
     (property "Sheetname" "")
     (property "Value_1" "R1501J033B-T1-JE")
@@
     (tags "LED")
     (property "LCSC" "C434420")
-    (property "Sheetfile" "USB-PD Programmer.kicad_sch")
+    (property "Sheetfile" "Programmer.kicad_sch")
     (property "Sheetname" "")
     (attr smd)
@@
     (tags "capacitor handsolder")
     (property "LCSC" "C161232")
-    (property "Sheetfile" "USB-PD Programmer.kicad_sch")
+    (property "Sheetfile" "Programmer.kicad_sch")
     (property "Sheetname" "")
     (attr smd)
@@
     (tags "LED")
     (property "LCSC" "C434424")
-    (property "Sheetfile" "USB-PD Programmer.kicad_sch")
+    (property "Sheetfile" "Programmer.kicad_sch")
     (property "Sheetname" "")
     (attr smd)
@@
     (tags "connector JST SH top entry")
     (property "Note" "Footprint only")
-    (property "Sheetfile" "USB-PD Programmer.kicad_sch")
+    (property "Sheetfile" "Programmer.kicad_sch")
     (property "Sheetname" "")
     (property "exclude_from_bom" "")
@@
     (tags "LED")
     (property "LCSC" "C434420")
-    (property "Sheetfile" "USB-PD Programmer.kicad_sch")
+    (property "Sheetfile" "Programmer.kicad_sch")
     (property "Sheetname" "")
     (attr smd)
@@
     (descr "JST SH series connector, SM04B-SRSS-TB (http://www.jst-mfg.com/product/pdf/eng/eSH.pdf), generated with kicad-footprint-generator")
     (tags "connector JST SH top entry")
-    (property "Sheetfile" "USB-PD Programmer.kicad_sch")
+    (property "Sheetfile" "Programmer.kicad_sch")
     (property "Sheetname" "")
     (property "exclude_from_bom" "")
@@
     (descr "JST SH series connector, SM04B-SRSS-TB (http://www.jst-mfg.com/product/pdf/eng/eSH.pdf), generated with kicad-footprint-generator")
     (tags "connector JST SH top entry")
-    (property "Sheetfile" "USB-PD Programmer.kicad_sch")
+    (property "Sheetfile" "Programmer.kicad_sch")
     (property "Sheetname" "")
     (property "exclude_from_bom" "")
@@
     (descr "JST SH series connector, SM04B-SRSS-TB (http://www.jst-mfg.com/product/pdf/eng/eSH.pdf), generated with kicad-footprint-generator")
     (tags "connector JST SH top entry")
-    (property "Sheetfile" "USB-PD Programmer.kicad_sch")
+    (property "Sheetfile" "Programmer.kicad_sch")
     (property "Sheetname" "")
     (property "exclude_from_bom" "")
@@
     (tags "capacitor")
     (property "LCSC" "C559769")
-    (property "Sheetfile" "USB-PD Programmer.kicad_sch")
+    (property "Sheetfile" "Programmer.kicad_sch")
     (property "Sheetname" "")
     (attr smd)
@@
     (descr "SMD Solder Jumper, 1x1.5mm, rounded Pads, 0.3mm gap, bridged with 1 copper strip")
     (tags "net tie solder jumper bridged")
-    (property "Sheetfile" "USB-PD Programmer.kicad_sch")
+    (property "Sheetfile" "Programmer.kicad_sch")
     (property "Sheetname" "")
     (property "exclude_from_bom" "")

Commit message: Some tweaks
Parts:
- moved SW1 1.48 mm to (108.5, 110.6)
Routing:
- net Vsec: track 44.6 -> 47.3 mm
- net RST: track 8.44 -> 7.60 mm
Other:
- board text added: "Stacked Rabbit"
Changed lines of the file:
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@@
   )
   (footprint "Tinker:SW_Push_TS273014TP" (layer "F.Cu")
-    (at 107.8 109.3 180)
+    (at 108.5 110.6 180)
     (descr "CK components KMR2 tactile switch http://www.ckswitches.com/media/1479/kmr2.pdf")
     (tags "tactile switch kmr2")
@@
     (effects (font (size 0.6 0.6) (thickness 0.125)))
   )
-  (gr_text "RESET" (at 107.8 112) (layer "F.SilkS")
+  (gr_text "RESET" (at 108.5 113) (layer "F.SilkS")
     (effects (font (size 1 1) (thickness 0.15)))
   )
@@
     (effects (font (size 0.5 0.5) (thickness 0.125)) (justify left))
   )
-  (gr_text "${TITLE}" (at 90.714825 108.589626 45) (layer "F.SilkS")
+  (gr_text "Stacked Rabbit" (at 90.194422 107.868088 45) (layer "F.SilkS")
+    (effects (font (size 0.75 0.75) (thickness 0.15) italic))
+  )
+  (gr_text "${TITLE}" (at 91.09507 108.749574 45) (layer "F.SilkS")
     (effects (font (size 0.75 0.75) (thickness 0.15)))
   )
@@
   (segment (start 110.598834 95.604578) (end 110.086331 95.092075) (width 0.6) (layer "F.Cu") (net 4))
   (segment (start 104.14 106.575) (end 104.14 106.653055) (width 0.6) (layer "F.Cu") (net 10))
+  (segment (start 104.14 105.81279) (end 104.14 106.240317) (width 0.6) (layer "F.Cu") (net 10))
   (segment (start 97.052801 95.975076) (end 94.9625 95.975076) (width 0.6) (layer "F.Cu") (net 10))
   (segment (start 105.518834 97.009151) (end 105.518834 91.317711) (width 0.6) (layer "F.Cu") (net 10))
   (segment (start 102.002801 90.5625) (end 102.002801 92.165076) (width 0.6) (layer "F.Cu") (net 10))
-  (segment (start 104.14 98.387985) (end 104.14 106.240317) (width 0.6) (layer "F.Cu") (net 10))
   (segment (start 95.89473 90.5625) (end 94.9625 91.49473) (width 0.6) (layer "F.Cu") (net 10))
   (segment (start 105.518834 97.009151) (end 104.14 98.387985) (width 0.6) (layer "F.Cu") (net 10))
   (segment (start 102.002801 90.5625) (end 95.89473 90.5625) (width 0.6) (layer "F.Cu") (net 10))
-  (segment (start 104.153055 106.653055) (end 105.95 108.45) (width 0.6) (layer "F.Cu") (net 10))
+  (segment (start 106.65 109.75) (end 106.147408 109.75) (width 0.6) (layer "F.Cu") (net 10))
   (segment (start 101.27 106.575) (end 102.94 106.575) (width 0.6) (layer "F.Cu") (net 10))
   (segment (start 104.919045 90.5625) (end 105.596545 91.24) (width 0.6) (layer "F.Cu") (net 10))
+  (segment (start 104.14 98.387985) (end 104.14 105.81279) (width 0.6) (layer "F.Cu") (net 10))
   (segment (start 102.002801 90.5625) (end 104.919045 90.5625) (width 0.6) (layer "F.Cu") (net 10))
   (segment (start 104.14 106.653055) (end 104.153055 106.653055) (width 0.6) (layer "F.Cu") (net 10))
+  (segment (start 104.14 107.742592) (end 104.14 105.81279) (width 0.6) (layer "F.Cu") (net 10))
+  (segment (start 106.147408 109.75) (end 104.14 107.742592) (width 0.6) (layer "F.Cu") (net 10))
   (segment (start 104.153055 106.253372) (end 104.153055 106.653055) (width 0.6) (layer "F.Cu") (net 10))
   (segment (start 94.9625 95.975076) (end 94.9625 91.49473) (width 0.6) (layer "F.Cu") (net 10))
   (segment (start 102.94 106.575) (end 104.14 106.575) (width 0.6) (layer "F.Cu") (net 10))
-  (segment (start 105.95 108.45) (end 109.65 108.45) (width 0.6) (layer "F.Cu") (net 10))
+  (segment (start 106.65 109.75) (end 110.35 109.75) (width 0.6) (layer "F.Cu") (net 10))
   (segment (start 104.14 106.240317) (end 104.153055 106.253372) (width 0.6) (layer "F.Cu") (net 10))
   (segment (start 97.052801 99.785076) (end 95.045689 99.785076) (width 0.25) (layer "F.Cu") (net 11))
@@
   (segment (start 102.54 96.229747) (end 101.015329 94.705076) (width 0.25) (layer "B.Cu") (net 20))
   (segment (start 102.54 114) (end 102.54 96.229747) (width 0.25) (layer "B.Cu") (net 20))
-  (segment (start 109.65 110.15) (end 105.95 110.15) (width 0.25) (layer "F.Cu") (net 22))
-  (segment (start 105.95 111.86) (end 103.81 114) (width 0.25) (layer "F.Cu") (net 22))
-  (segment (start 105.95 110.15) (end 105.95 111.86) (width 0.25) (layer "F.Cu") (net 22))
+  (segment (start 106.36 111.45) (end 106.65 111.45) (width 0.25) (layer "F.Cu") (net 22))
+  (segment (start 103.81 114) (end 106.36 111.45) (width 0.25) (layer "F.Cu") (net 22))
+  (segment (start 106.65 111.45) (end 110.35 111.45) (width 0.25) (layer "F.Cu") (net 22))
   (segment (start 94.92 112.73) (end 96.19 114) (width 0.6) (layer "F.Cu") (net 25))
   (segment (start 94.92 111.1875) (end 94.92 112.73) (width 0.6) (layer "F.Cu") (net 25))
