File: Hardware/Prototype.kicad_pcb (KiCad board)
At the start: 2 copper layers, 34 x 34 mm, 14 parts, among them J1 Conn_01x07_Male, J2 Conn_01x04_Male, J3 Conn_01x02_Male, J4 Conn_01x02_Male, J5 Conn_01x02_Male, J6 Conn_01x02_Male, J7 Conn_01x08_Male, J9 QWIIC_Stackable

Commit message: Cleanup & working on J7/J9 rework
Parts:
- removed J1: Conn_01x07_Male, Tinker:Board_Stacker_7
Connections:
- net ALERT renamed ~{SCS}0
- net GPIO renamed MOSI
- net POWER_OK2 renamed SCLK
- net POWER_OK3 renamed MISO
- J7 pad 1: RESET -> ~{SCS}3
- J7 pad 2: ATTACH -> RESET
- J7 pad 3: SCL -> ~{SCS}2
- J7 pad 5: SDA -> ~{SCS}1
Routing:
- net SDA: track 10.6 -> 0.00 mm
- net SCL: track 6.15 -> 0.00 mm
Other:
- board text added: "SCL"
- board text added: "SDA"
- board text added: "SPI"
- board text removed: "DTR"
- board text removed: "RST"
- board text removed: "RTS"
- board text removed: "RxD"
- board text removed: "TxD"

Commit message: Working on changes to J7/J9
Parts:
- moved J6 1.28 mm to (114.0, 92.4)
- moved J5 0.66 mm to (114.0, 99.4)
Other:
- board text added: ">RST"
- board text added: "MISO"
- board text added: "MOSI"
- board text added: "SCLK"
- board text added: "USB"
- board text added: "Vusb"
- board text added: "~{SCS}"
Changed lines of the file:
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@@
   )
   (footprint "Tinker:Board_Stacker_2" (layer "F.Cu")
-    (at 114 106.32)
+    (at 114 106.365)
     (descr "JST SH series connector, SM04B-SRSS-TB (http://www.jst-mfg.com/product/pdf/eng/eSH.pdf), generated with kicad-footprint-generator")
     (tags "connector JST SH top entry")
@@
     (property "Sheetname" "")
     (attr smd)
-    (fp_text reference "J2" (at 1.6 1.905) (layer "F.SilkS")
+    (fp_text reference "J2" (at 0 5.305) (layer "F.SilkS")
       (effects (font (size 0.6 0.6) (thickness 0.15)))
     )
@@
   )
   (footprint "Tinker:Board_Stacker_2" (layer "F.Cu")
-    (at 86 106.32)
+    (at 86 106.365)
     (descr "JST SH series connector, SM04B-SRSS-TB (http://www.jst-mfg.com/product/pdf/eng/eSH.pdf), generated with kicad-footprint-generator")
     (tags "connector JST SH top entry")
@@
   )
   (footprint "Tinker:Board_Stacker_2" (layer "F.Cu")
-    (at 114 91.08)
+    (at 114 92.365)
     (descr "JST SH series connector, SM04B-SRSS-TB (http://www.jst-mfg.com/product/pdf/eng/eSH.pdf), generated with kicad-footprint-generator")
     (tags "connector JST SH top entry")
@@
   )
   (footprint "Tinker:Board_Stacker_2" (layer "F.Cu")
-    (at 114 98.7)
+    (at 114 99.365)
     (descr "JST SH series connector, SM04B-SRSS-TB (http://www.jst-mfg.com/product/pdf/eng/eSH.pdf), generated with kicad-footprint-generator")
     (tags "connector JST SH top entry")
@@
     (effects (font (size 1 1) (thickness 0.15)) (justify mirror))
   )
-  (gr_text "GND" (at 113.911636 101.079492) (layer "B.SilkS")
+  (gr_text "GND" (at 113.911636 101.744492) (layer "B.SilkS")
     (effects (font (size 0.6 0.6) (thickness 0.125)) (justify mirror))
   )
-  (gr_text "GND" (at 85.995908 108.702728) (layer "B.SilkS")
+  (gr_text "GND" (at 85.995908 108.747728) (layer "B.SilkS")
     (effects (font (size 0.6 0.6) (thickness 0.125)) (justify mirror))
   )
-  (gr_text "Vout" (at 113.950572 105.258488) (layer "B.SilkS")
+  (gr_text "Vout" (at 113.950572 105.303488) (layer "B.SilkS")
     (effects (font (size 0.6 0.6) (thickness 0.125)) (justify mirror))
   )
-  (gr_text "GND" (at 113.946688 93.440074) (layer "B.SilkS")
+  (gr_text "GND" (at 113.946688 94.725074) (layer "B.SilkS")
     (effects (font (size 0.6 0.6) (thickness 0.125)) (justify mirror))
   )
-  (gr_text "Vsec" (at 113.872799 97.603635) (layer "B.SilkS")
+  (gr_text "Vsec" (at 113.872799 98.268635) (layer "B.SilkS")
     (effects (font (size 0.6 0.6) (thickness 0.125)) (justify mirror))
   )
-  (gr_text "Vsec" (at 113.830179 90.061308) (layer "B.SilkS")
+  (gr_text "Vsec" (at 113.830179 91.346308) (layer "B.SilkS")
     (effects (font (size 0.6 0.6) (thickness 0.125)) (justify mirror))
   )
-  (gr_text "GND" (at 113.997176 108.84697) (layer "B.SilkS")
+  (gr_text "GND" (at 113.997176 108.89197) (layer "B.SilkS")
     (effects (font (size 0.6 0.6) (thickness 0.125)) (justify mirror))
   )
@@
     (effects (font (size 1 1) (thickness 0.15)) (justify mirror))
   )
-  (gr_text "Vout" (at 86.009393 105.223635) (layer "B.SilkS")
+  (gr_text "Vout" (at 86.009393 105.268635) (layer "B.SilkS")
     (effects (font (size 0.6 0.6) (thickness 0.125)) (justify mirror))
   )
-  (gr_text "SDA" (at 90.9 94.905) (layer "F.SilkS")
+  (gr_text "SDA" (at 90.5 94.905) (layer "F.SilkS")
     (effects (font (size 0.5 0.5) (thickness 0.125)) (justify left))
   )
-  (gr_text "3v3" (at 90.9 92.365) (layer "F.SilkS")
+  (gr_text "Vsec" (at 116.2 100 90) (layer "F.SilkS")
+    (effects (font (size 1 1) (thickness 0.15)))
+  )
+  (gr_text "3v3" (at 90.5 92.365) (layer "F.SilkS")
     (effects (font (size 0.5 0.5) (thickness 0.125)) (justify left))
   )
-  (gr_text "Vout" (at 114 105.2) (layer "F.SilkS")
+  (gr_text "Vout" (at 114 105.245) (layer "F.SilkS")
     (effects (font (size 0.6 0.6) (thickness 0.125)))
   )
-  (gr_text "GND" (at 114 93.4) (layer "F.SilkS")
+  (gr_text "~{SCS}" (at 83.347793 103.30044) (layer "F.SilkS")
+    (effects (font (size 0.5 0.5) (thickness 0.125)) (justify left))
+  )
+  (gr_text "GND" (at 114 94.685) (layer "F.SilkS")
     (effects (font (size 0.6 0.6) (thickness 0.125)))
   )
-  (gr_text "GND" (at 90.9 91.095) (layer "F.SilkS")
+  (gr_text "GND" (at 90.5 91.095) (layer "F.SilkS")
     (effects (font (size 0.5 0.5) (thickness 0.125)) (justify left))
   )
-  (gr_text "D-" (at 99.365 84.3 90) (layer "F.SilkS")
-    (effects (font (size 0.6 0.6) (thickness 0.15)))
-  )
-  (gr_text "D+" (at 100.635 84.3 90) (layer "F.SilkS")
-    (effects (font (size 0.6 0.6) (thickness 0.15)))
-  )
-  (gr_text "GND" (at 114 101) (layer "F.SilkS")
+  (gr_text "D-" (at 99.365 86.8 90) (layer "F.SilkS")
+    (effects (font (size 0.6 0.6) (thickness 0.15)) (justify right))
+  )
+  (gr_text "D+" (at 100.635 86.8 90) (layer "F.SilkS")
+    (effects (font (size 0.6 0.6) (thickness 0.15)) (justify right))
+  )
+  (gr_text "GND" (at 114 101.665) (layer "F.SilkS")
     (effects (font (size 0.6 0.6) (thickness 0.125)))
+  )
+  (gr_text "Vsec" (at 116.2 93 90) (layer "F.SilkS")
+    (effects (font (size 1 1) (thickness 0.15)))
+  )
+  (gr_text "USB" (at 100 83.8 180) (layer "F.SilkS")
+    (effects (font (size 1 1) (thickness 0.15)))
+  )
+  (gr_text "SCLK" (at 88.5 99.365) (layer "F.SilkS")
+    (effects (font (size 0.5 0.5) (thickness 0.125)) (justify left))
+  )
+  (gr_text ">RST" (at 88.5 98.095) (layer "F.SilkS")
+    (effects (font (size 0.5 0.5) (thickness 0.125)) (justify left))
   )
   (gr_text "SPI" (at 83.8 100 -90) (layer "F.SilkS")
     (effects (font (size 1 1) (thickness 0.15)))
   )
-  (gr_text "GND" (at 98.095 84.3 90) (layer "F.SilkS")
-    (effects (font (size 0.6 0.6) (thickness 0.125)))
-  )
-  (gr_text "SCL" (at 90.9 93.635) (layer "F.SilkS")
+  (gr_text "Vusb" (at 116.2 107 90) (layer "F.SilkS")
+    (effects (font (size 1 1) (thickness 0.15)))
+  )
+  (gr_text "GND" (at 98.095 86.8 90) (layer "F.SilkS")
+    (effects (font (size 0.6 0.6) (thickness 0.125)) (justify right))
+  )
+  (gr_text "SCL" (at 90.5 93.635) (layer "F.SilkS")
     (effects (font (size 0.5 0.5) (thickness 0.125)) (justify left))
   )
-  (gr_text "GND" (at 114 108.7) (layer "F.SilkS")
+  (gr_text "GND" (at 114 108.745) (layer "F.SilkS")
     (effects (font (size 0.6 0.6) (thickness 0.125)))
   )
@@
     (effects (font (size 1 1) (thickness 0.15)))
   )
-  (gr_text "GND" (at 86 108.7) (layer "F.SilkS")
+  (gr_text "MISO" (at 88.5 100.635) (layer "F.SilkS")
+    (effects (font (size 0.5 0.5) (thickness 0.125)) (justify left))
+  )
+  (gr_text "MOSI" (at 88.5 101.905) (layer "F.SilkS")
+    (effects (font (size 0.5 0.5) (thickness 0.125)) (justify left))
+  )
+  (gr_text "GND" (at 86 108.745) (layer "F.SilkS")
     (effects (font (size 0.6 0.6) (thickness 0.125)))
   )
@@
     (effects (font (size 0.75 0.75) (thickness 0.15)))
   )
-  (gr_text "Vout" (at 101.905 84.3 90) (layer "F.SilkS")
+  (gr_text "Vout" (at 101.905 86.8 90) (layer "F.SilkS")
+    (effects (font (size 0.6 0.6) (thickness 0.125)) (justify right))
+  )
+  (gr_text "Vusb" (at 83.8 107 -90) (layer "F.SilkS")
+    (effects (font (size 1 1) (thickness 0.15)))
+  )
+  (gr_text "Vsec" (at 114 98.265) (layer "F.SilkS")
     (effects (font (size 0.6 0.6) (thickness 0.125)))
   )
-  (gr_text "Vsec" (at 114 97.6) (layer "F.SilkS")
+  (gr_text "Vout" (at 86 105.245) (layer "F.SilkS")
     (effects (font (size 0.6 0.6) (thickness 0.125)))
   )
-  (gr_text "Vout" (at 86 105.2) (layer "F.SilkS")
+  (gr_text "Vsec" (at 114 91.285) (layer "F.SilkS")
     (effects (font (size 0.6 0.6) (thickness 0.125)))
   )
-  (gr_text "Vsec" (at 114 90) (layer "F.SilkS")
-    (effects (font (size 0.6 0.6) (thickness 0.125)))
-  )

Commit message: Still migrating to 0.2.x
Connections:
- net ~{SCS}3 renamed ~{RESET}
Other:
- board text added: "2,1,0"
- board text added: ">~{RST}"
Changed lines of the file:
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@@
   (net 10 "SCL")
   (net 11 "RESET")
-  (net 12 "~{SCS}3")
+  (net 12 "~{RESET}")
   (net 13 "~{SCS}2")
   (net 14 "SCLK")
@@
     (descr "JST SH series connector, SM04B-SRSS-TB (http://www.jst-mfg.com/product/pdf/eng/eSH.pdf), generated with kicad-footprint-generator")
     (tags "connector JST SH top entry")
+    (property "LCSC" "C145956 + C2938401 + C2881513")
     (property "Sheetfile" "Prototype.kicad_sch")
     (property "Sheetname" "")
@@
     (fp_line (start -1.07 4.445) (end -1.07 0.2175) (layer "F.Fab") (width 0.1))
     (pad "1" smd rect (at -1.195 0) (size 2.1 0.75) (layers "B.Cu" "B.Paste" "B.Mask")
-      (net 12 "~{SCS}3") (pinfunction "Pin_1") (pintype "passive"))
+      (net 12 "~{RESET}") (pinfunction "Pin_1") (pintype "passive"))
     (pad "1" thru_hole rect (at 0 0) (size 1 1) (drill 0.65) (layers *.Cu *.Mask)
-      (net 12 "~{SCS}3") (pinfunction "Pin_1") (pintype "passive"))
+      (net 12 "~{RESET}") (pinfunction "Pin_1") (pintype "passive"))
     (pad "2" smd rect (at 2.405 0) (size 2.1 0.75) (layers "B.Cu" "B.Paste" "B.Mask")
       (net 11 "RESET") (pinfunction "Pin_2") (pintype "passive"))
@@
     (descr "JST SH series connector, SM04B-SRSS-TB (http://www.jst-mfg.com/product/pdf/eng/eSH.pdf), generated with kicad-footprint-generator")
     (tags "connector JST SH top entry")
+    (property "LCSC" "C2938400 + C2881511")
     (property "Sheetfile" "Prototype.kicad_sch")
     (property "Sheetname" "")
@@
     (descr "JST SH series connector, SM04B-SRSS-TB (http://www.jst-mfg.com/product/pdf/eng/eSH.pdf), generated with kicad-footprint-generator")
     (tags "connector JST SH top entry")
+    (property "LCSC" "C2938401 + C2881513")
     (property "Sheetfile" "Prototype.kicad_sch")
     (property "Sheetname" "")
@@
     (descr "JST SH series connector, SM04B-SRSS-TB (http://www.jst-mfg.com/product/pdf/eng/eSH.pdf), generated with kicad-footprint-generator")
     (tags "connector JST SH top entry")
+    (property "LCSC" "C2938400 + C2881511")
     (property "Sheetfile" "Prototype.kicad_sch")
     (property "Sheetname" "")
@@
     (descr "JST SH series connector, SM04B-SRSS-TB (http://www.jst-mfg.com/product/pdf/eng/eSH.pdf), generated with kicad-footprint-generator")
     (tags "connector JST SH top entry")
+    (property "LCSC" "C2938400 + C2881511")
     (property "Sheetfile" "Prototype.kicad_sch")
     (property "Sheetname" "")
@@
     (descr "JST SH series connector, SM04B-SRSS-TB (http://www.jst-mfg.com/product/pdf/eng/eSH.pdf), generated with kicad-footprint-generator")
     (tags "connector JST SH top entry")
+    (property "LCSC" "C2938400 + C2881511")
     (property "Sheetfile" "Prototype.kicad_sch")
     (property "Sheetname" "")
@@
     (effects (font (size 0.6 0.6) (thickness 0.125)) (justify mirror))
   )
-  (gr_text "GND" (at 113.946688 94.725074) (layer "B.SilkS")
+  (gr_text "GND" (at 114 94.7) (layer "B.SilkS")
     (effects (font (size 0.6 0.6) (thickness 0.125)) (justify mirror))
   )
@@
     (effects (font (size 0.6 0.6) (thickness 0.125)) (justify mirror))
   )
-  (gr_text "Vsec" (at 113.830179 91.346308) (layer "B.SilkS")
+  (gr_text "Vsec" (at 114 91.3) (layer "B.SilkS")
     (effects (font (size 0.6 0.6) (thickness 0.125)) (justify mirror))
   )
@@
     (effects (font (size 0.6 0.6) (thickness 0.125)) (justify mirror))
   )
-  (gr_text "SDA" (at 90.5 94.905) (layer "F.SilkS")
+  (gr_text "SDA" (at 90.2 94.905) (layer "F.SilkS")
     (effects (font (size 0.5 0.5) (thickness 0.125)) (justify left))
   )
@@
     (effects (font (size 1 1) (thickness 0.15)))
   )
-  (gr_text "3v3" (at 90.5 92.365) (layer "F.SilkS")
+  (gr_text "2,1,0" (at 83.6 103.94) (layer "F.SilkS")
+    (effects (font (size 0.5 0.5) (thickness 0.125)) (justify left))
+  )
+  (gr_text "3v3" (at 90.2 92.365) (layer "F.SilkS")
     (effects (font (size 0.5 0.5) (thickness 0.125)) (justify left))
   )
@@
     (effects (font (size 0.6 0.6) (thickness 0.125)))
   )
-  (gr_text "~{SCS}" (at 83.347793 103.30044) (layer "F.SilkS")
+  (gr_text "~{SCS}" (at 83.3 103.3) (layer "F.SilkS")
     (effects (font (size 0.5 0.5) (thickness 0.125)) (justify left))
   )
-  (gr_text "GND" (at 114 94.685) (layer "F.SilkS")
+  (gr_text "GND" (at 114 94.7) (layer "F.SilkS")
     (effects (font (size 0.6 0.6) (thickness 0.125)))
   )
-  (gr_text "GND" (at 90.5 91.095) (layer "F.SilkS")
+  (gr_text "GND" (at 90.2 91.095) (layer "F.SilkS")
     (effects (font (size 0.5 0.5) (thickness 0.125)) (justify left))
   )
@@
     (effects (font (size 0.6 0.6) (thickness 0.15)) (justify right))
   )
+  (gr_text ">~{RST}" (at 83.3 96.9) (layer "F.SilkS")
+    (effects (font (size 0.5 0.5) (thickness 0.125)) (justify left))
+  )
   (gr_text "D+" (at 100.635 86.8 90) (layer "F.SilkS")
     (effects (font (size 0.6 0.6) (thickness 0.15)) (justify right))
@@
     (effects (font (size 0.6 0.6) (thickness 0.125)) (justify right))
   )
-  (gr_text "SCL" (at 90.5 93.635) (layer "F.SilkS")
+  (gr_text "SCL" (at 90.2 93.635) (layer "F.SilkS")
     (effects (font (size 0.5 0.5) (thickness 0.125)) (justify left))
   )
@@
     (effects (font (size 0.6 0.6) (thickness 0.125)))
   )
-  (gr_text "Vsec" (at 114 91.285) (layer "F.SilkS")
+  (gr_text "Vsec" (at 114 91.3) (layer "F.SilkS")
     (effects (font (size 0.6 0.6) (thickness 0.125)))
   )
