File: Hardware/Prototype.kicad_sch (KiCad schematic)
At the start: 8 parts, among them J1 Conn_01x07_Male, J2 Conn_01x04_Male, J3 Conn_01x02_Male, J4 Conn_01x02_Male, J5 Conn_01x02_Male, J6 Conn_01x02_Male, J7 Conn_01x08_Male, J9 QWIIC_Stackable

Commit message: Cleanup & working on J7/J9 rework
Parts:
- added J8: Conn_01x08_Male, Tinker:PinHeader_2x04_P1.27mm_Vertical, symbol Connector:Conn_01x08_Male
- J2: LCSC (none) -> C2938401 + C2881513; now in the parts list
- J3, J4, J5, J6: LCSC (none) -> C2938400 + C2881511; now in the parts list
- J7: now in the parts list
- J9: LCSC (none) -> C145956 + C2938401 + C2881513; now in the parts list
Connections:
- net ALERT: now also J8.7 (Pin_7); no longer J7.7 (Pin_7)
- net ATTACH: now also J8.2 (Pin_2); no longer J7.2 (Pin_2)
- net GPIO: now also J8.8 (Pin_8); no longer J7.8 (Pin_8)
- net POWER_OK2: now also J8.4 (Pin_4); no longer J7.4 (Pin_4)
- net POWER_OK3: now also J8.6 (Pin_6); no longer J7.6 (Pin_6)
- net RESET: now also J7.2 (Pin_2), J8.1 (Pin_1); no longer J7.1 (Pin_1)
- net SCL: now also J8.3 (Pin_3); no longer J7.3 (Pin_3)
- net SDA: now also J8.5 (Pin_5); no longer J7.5 (Pin_5)
- new net MISO: J7.6 (Pin_6)
- new net MOSI: J7.8 (Pin_8)
- new net SCLK: J7.4 (Pin_4)
- new net ~{SCS}0: J7.7 (Pin_7)
- new net ~{SCS}1: J7.5 (Pin_5)
- new net ~{SCS}2: J7.3 (Pin_3)
- new net ~{SCS}3: J7.1 (Pin_1)
Other:
- note added: "I2C"
- note added: "SPI"
- note removed: "QWIIC"
- moved on the sheet: J7, J9

Commit message: Still migrating to 0.2.x
Connections:
- net ~{SCS}3 renamed ~{RESET}
Changed lines of the file:
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@@
     )
   )
-  (global_label "~{SCS}3" (shape bidirectional) (at 63.5 72.39 180) (fields_autoplaced)
+  (global_label "~{RESET}" (shape input) (at 63.5 72.39 180) (fields_autoplaced)
     (effects (font (size 1.27 1.27) (thickness 0.254) bold) (justify right))
-    (property "Intersheet References" "${INTERSHEET_REFS}" (id 0) (at 55.9979 72.263 0)
+    (property "Intersheet References" "${INTERSHEET_REFS}" (id 0) (at 55.1513 72.263 0)
       (effects (font (size 1.27 1.27) (thickness 0.254) bold) (justify right) hide)
     )

Commit message: Whole bunch of cleanup & 3D rework
Parts:
- removed J8: Conn_01x08_Male, Tinker:PinHeader_2x04_P1.27mm_Vertical, symbol Connector:Conn_01x08_Male
- added J8: QWIIC_Vertical, Tinker:QWIIC_Vertical, symbol Connector_Generic_MountingPin:Conn_01x04_MountingPin
- J9: value QWIIC_Stackable -> QWIIC_Stack_II
Connections:
- net GND: now also J8.1 (Pin_1), J8.MP (MountPin)
- net SCL: now also J8.4 (Pin_4)
- net SDA: now also J8.3 (Pin_3)
- net Vcc?: now also J8.2 (Pin_2)
Other:
- note added: "Stackable QWIIC"
- note added: "Vertical QWIIC"
- note removed: "Control"
- moved on the sheet: J1, J2, J3, J4, J5, J6, J7, J9
