File: Hardware/Li-Ion Charger.kicad_pcb (KiCad board)
At the start: 2 copper layers, 34 x 34 mm, 49 parts, among them IC1 BQ25792RQMR, J10 Output, J11 Conn_01x06, J2 Conn_01x04_Male, J3 Conn_01x02_Male, J4 Conn_01x02_Male, J5 Conn_01x02_Male, J6 Conn_01x02_Male, J7 Conn_01x08_Male, J9 QWIIC_Stack_II

Commit message: Now...There's a BMS for the Charger!
Parts:
- J11: value Conn_01x06 -> Conn_01x02; footprint Connector_PinSocket_1.27mm:PinSocket_1x06_P1.27mm_Vertical_SMD_Pin1Right -> Connector_PinSocket_1.27mm:PinSocket_1x02_P1.27mm_Vertical
- moved J11 10.8 mm to (105.7, 104.4), turned to 180 degrees
Routing:
- net VBUS: track 25.6 -> 14.8 mm
- net VDD: track 35.1 -> 31.1 mm
Changed lines of the file:
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@@
     )
   )
-  (footprint "Connector_PinSocket_1.27mm:PinSocket_1x06_P1.27mm_Vertical_SMD_Pin1Right" (layer "B.Cu")
-    (at 100 113.6 90)
-    (descr "surface-mounted straight socket strip, 1x06, 1.27mm pitch, single row, style 2 (pin 1 right) (https://gct.co/pdfjs/web/viewer.html?file=/Files/Drawings/BD075.pdf&t=1511594726925), script generated")
-    (tags "Surface mounted socket strip SMD 1x06 1.27mm single row style2 pin1 right")
+  (footprint "Connector_PinSocket_1.27mm:PinSocket_1x02_P1.27mm_Vertical" (layer "B.Cu")
+    (at 105.7 104.4 180)
+    (descr "Through hole straight socket strip, 1x02, 1.27mm pitch, single row (from Kicad 4.0.7), script generated")
+    (tags "Through hole socket strip THT 1x02 1.27mm single row")
     (property "Sheetfile" "Li-Ion Charger.kicad_sch")
     (property "Sheetname" "")
-    (attr smd)
-    (fp_text reference "J11" (at 0 5.485 180) (layer "B.SilkS")
-      (effects (font (size 0.6 0.6) (thickness 0.15)) (justify mirror))
-    )
-    (fp_text value "Conn_01x06" (at 0 -5.485 90) (layer "B.Fab")
+    (attr through_hole)
+    (fp_text reference "J11" (at 0 2.135) (layer "B.SilkS")
       (effects (font (size 1 1) (thickness 0.15)) (justify mirror))
     )
-    (fp_text user "${REFERENCE}" (at 0 0) (layer "B.Fab")
+    (fp_text value "Conn_01x02" (at 0 -3.405) (layer "B.Fab")
       (effects (font (size 1 1) (thickness 0.15)) (justify mirror))
     )
-    (fp_line (start -0.96 -3.76) (end -0.96 -4.045) (layer "B.SilkS") (width 0.12))
-    (fp_line (start 0.96 4.045) (end 0.96 3.76) (layer "B.SilkS") (width 0.12))
-    (fp_line (start 0.96 2.59) (end 0.96 1.22) (layer "B.SilkS") (width 0.12))
-    (fp_line (start -0.96 1.32) (end -0.96 -0.05) (layer "B.SilkS") (width 0.12))
-    (fp_line (start 0.96 3.76) (end 2.19 3.76) (layer "B.SilkS") (width 0.12))
-    (fp_line (start 0.96 -2.49) (end 0.96 -4.045) (layer "B.SilkS") (width 0.12))
-    (fp_line (start -0.96 -4.045) (end 0.96 -4.045) (layer "B.SilkS") (width 0.12))
-    (fp_line (start -0.96 4.045) (end -0.96 2.49) (layer "B.SilkS") (width 0.12))
-    (fp_line (start -0.96 4.045) (end 0.96 4.045) (layer "B.SilkS") (width 0.12))
-    (fp_line (start -0.96 -1.22) (end -0.96 -2.59) (layer "B.SilkS") (width 0.12))
-    (fp_line (start 0.96 0.05) (end 0.96 -1.32) (layer "B.SilkS") (width 0.12))
-    (fp_line (start -2.75 4.5) (end 2.75 4.5) (layer "B.CrtYd") (width 0.05))
-    (fp_line (start 2.75 -4.5) (end -2.75 -4.5) (layer "B.CrtYd") (width 0.05))
-    (fp_line (start -2.75 -4.5) (end -2.75 4.5) (layer "B.CrtYd") (width 0.05))
-    (fp_line (start 2.75 4.5) (end 2.75 -4.5) (layer "B.CrtYd") (width 0.05))
-    (fp_line (start -0.9 -3.385) (end -1.75 -3.385) (layer "B.Fab") (width 0.1))
-    (fp_line (start 0.9 -1.695) (end 1.75 -1.695) (layer "B.Fab") (width 0.1))
-    (fp_line (start -1.75 1.695) (end -1.75 2.115) (layer "B.Fab") (width 0.1))
-    (fp_line (start 1.75 0.845) (end 1.75 0.425) (layer "B.Fab") (width 0.1))
-    (fp_line (start -1.75 -0.845) (end -1.75 -0.425) (layer "B.Fab") (width 0.1))
-    (fp_line (start -1.75 -0.425) (end -0.9 -0.425) (layer "B.Fab") (width 0.1))
-    (fp_line (start -0.9 1.695) (end -1.75 1.695) (layer "B.Fab") (width 0.1))
-    (fp_line (start 0.45 3.985) (end 0.9 3.535) (layer "B.Fab") (width 0.1))
-    (fp_line (start 1.75 2.965) (end 0.9 2.965) (layer "B.Fab") (width 0.1))
-    (fp_line (start 0.9 0.845) (end 1.75 0.845) (layer "B.Fab") (width 0.1))
-    (fp_line (start 0.9 -3.985) (end -0.9 -3.985) (layer "B.Fab") (width 0.1))
-    (fp_line (start -1.75 -2.965) (end -0.9 -2.965) (layer "B.Fab") (width 0.1))
-    (fp_line (start -0.9 -0.845) (end -1.75 -0.845) (layer "B.Fab") (width 0.1))
-    (fp_line (start 1.75 3.385) (end 1.75 2.965) (layer "B.Fab") (width 0.1))
-    (fp_line (start 1.75 -1.695) (end 1.75 -2.115) (layer "B.Fab") (width 0.1))
-    (fp_line (start -1.75 -3.385) (end -1.75 -2.965) (layer "B.Fab") (width 0.1))
-    (fp_line (start 1.75 0.425) (end 0.9 0.425) (layer "B.Fab") (width 0.1))
-    (fp_line (start -0.9 -3.985) (end -0.9 3.985) (layer "B.Fab") (width 0.1))
-    (fp_line (start 0.9 3.535) (end 0.9 -3.985) (layer "B.Fab") (width 0.1))
-    (fp_line (start 0.9 3.385) (end 1.75 3.385) (layer "B.Fab") (width 0.1))
-    (fp_line (start 1.75 -2.115) (end 0.9 -2.115) (layer "B.Fab") (width 0.1))
-    (fp_line (start -0.9 3.985) (end 0.45 3.985) (layer "B.Fab") (width 0.1))
-    (fp_line (start -1.75 2.115) (end -0.9 2.115) (layer "B.Fab") (width 0.1))
-    (pad "1" smd rect (at 1.35 3.175 90) (size 1.8 0.65) (layers "B.Cu" "B.Paste" "B.Mask")
+    (fp_text user "${REFERENCE}" (at 0 -0.635 90) (layer "B.Fab")
+      (effects (font (size 1 1) (thickness 0.15)) (justify mirror))
+    )
+    (fp_line (start 0.76 -0.635) (end 1.33 -0.635) (layer "B.SilkS") (width 0.12))
+    (fp_line (start 0.30753 -1.965) (end 1.33 -1.965) (layer "B.SilkS") (width 0.12))
+    (fp_line (start 1.33 0.76) (end 1.33 0) (layer "B.SilkS") (width 0.12))
+    (fp_line (start 1.33 -0.635) (end 1.33 -1.965) (layer "B.SilkS") (width 0.12))
+    (fp_line (start -1.33 -0.635) (end -1.33 -1.965) (layer "B.SilkS") (width 0.12))
+    (fp_line (start 0 0.76) (end 1.33 0.76) (layer "B.SilkS") (width 0.12))
+    (fp_line (start -1.33 -0.635) (end -0.76 -0.635) (layer "B.SilkS") (width 0.12))
+    (fp_line (start -1.33 -1.965) (end -0.30753 -1.965) (layer "B.SilkS") (width 0.12))
+    (fp_line (start 1.75 -2.4) (end -1.8 -2.4) (layer "B.CrtYd") (width 0.05))
+    (fp_line (start 1.75 1.15) (end 1.75 -2.4) (layer "B.CrtYd") (width 0.05))
+    (fp_line (start -1.8 -2.4) (end -1.8 1.15) (layer "B.CrtYd") (width 0.05))
+    (fp_line (start -1.8 1.15) (end 1.75 1.15) (layer "B.CrtYd") (width 0.05))
+    (fp_line (start -1.27 -1.905) (end -1.27 0.635) (layer "B.Fab") (width 0.1))
+    (fp_line (start 1.27 -1.905) (end -1.27 -1.905) (layer "B.Fab") (width 0.1))
+    (fp_line (start 0.635 0.635) (end 1.27 0) (layer "B.Fab") (width 0.1))
+    (fp_line (start -1.27 0.635) (end 0.635 0.635) (layer "B.Fab") (width 0.1))
+    (fp_line (start 1.27 0) (end 1.27 -1.905) (layer "B.Fab") (width 0.1))
+    (pad "1" thru_hole rect (at 0 0 180) (size 1 1) (drill 0.7) (layers *.Cu *.Mask)
       (net 27 "VBUS") (pinfunction "Pin_1") (pintype "passive"))
-    (pad "2" smd rect (at -1.35 1.905 90) (size 1.8 0.65) (layers "B.Cu" "B.Paste" "B.Mask")
+    (pad "2" thru_hole oval (at 0 -1.27 180) (size 1 1) (drill 0.7) (layers *.Cu *.Mask)
       (net 27 "VBUS") (pinfunction "Pin_2") (pintype "passive"))
-    (pad "3" smd rect (at 1.35 0.635 90) (size 1.8 0.65) (layers "B.Cu" "B.Paste" "B.Mask")
-      (net 3 "GND") (pinfunction "Pin_3") (pintype "passive"))
-    (pad "4" smd rect (at -1.35 -0.635 90) (size 1.8 0.65) (layers "B.Cu" "B.Paste" "B.Mask")
-      (net 3 "GND") (pinfunction "Pin_4") (pintype "passive"))
-    (pad "5" smd rect (at 1.35 -1.905 90) (size 1.8 0.65) (layers "B.Cu" "B.Paste" "B.Mask")
-      (net 25 "VDD") (pinfunction "Pin_5") (pintype "passive"))
-    (pad "6" smd rect (at -1.35 -3.175 90) (size 1.8 0.65) (layers "B.Cu" "B.Paste" "B.Mask")
-      (net 25 "VDD") (pinfunction "Pin_6") (pintype "passive"))
-    (model "${KICAD6_3DMODEL_DIR}/Connector_PinSocket_1.27mm.3dshapes/PinSocket_1x06_P1.27mm_Vertical_SMD_Pin1Right.wrl"
+    (model "${KICAD6_3DMODEL_DIR}/Connector_PinSocket_1.27mm.3dshapes/PinSocket_1x02_P1.27mm_Vertical.wrl"
       (offset (xyz 0 0 0))
       (scale (xyz 1 1 1))
@@
   (segment (start 98.776505 110.32819) (end 103.960902 105.143793) (width 0.5) (layer "B.Cu") (net 25))
   (segment (start 101.675 97.7) (end 103.960902 99.985902) (width 0.5) (layer "B.Cu") (net 25))
-  (segment (start 98.19533 112.14967) (end 98.095 112.25) (width 0.5) (layer "B.Cu") (net 25))
   (segment (start 98.776505 112.14967) (end 98.776505 110.32819) (width 0.5) (layer "B.Cu") (net 25))
-  (segment (start 96.825 114.95) (end 96.825 113.52) (width 0.5) (layer "B.Cu") (net 25))
   (segment (start 103.960902 99.985902) (end 103.960902 105.143793) (width 0.5) (layer "B.Cu") (net 25))
-  (segment (start 96.825 113.52) (end 98.095 112.25) (width 0.5) (layer "B.Cu") (net 25))
-  (segment (start 98.776505 112.14967) (end 98.19533 112.14967) (width 0.5) (layer "B.Cu") (net 25))
   (segment (start 101.85 100.4) (end 104.4 100.4) (width 0.2) (layer "F.Cu") (net 26))
   (segment (start 104.4 100.4) (end 104.8 100) (width 0.2) (layer "F.Cu") (net 26))
@@
   (segment (start 107.8 101.65) (end 109.3 101.65) (width 0.5) (layer "F.Cu") (net 27))
   (via (at 105.556347 101.659533) (size 0.8) (drill 0.4) (layers "F.Cu" "B.Cu") (net 27))
-  (segment (start 103.175 112.25) (end 103.175 113.68) (width 0.5) (layer "B.Cu") (net 27))
-  (segment (start 103.175 112.25) (end 103.175 108.751486) (width 0.5) (layer "B.Cu") (net 27))
-  (segment (start 103.175 113.68) (end 101.905 114.95) (width 0.5) (layer "B.Cu") (net 27))
-  (segment (start 103.175 108.751486) (end 105.556347 106.370139) (width 0.5) (layer "B.Cu") (net 27))
-  (segment (start 105.556347 101.659533) (end 105.556347 106.370139) (width 0.5) (layer "B.Cu") (net 27))
+  (segment (start 105.7 104.3) (end 105.7 105.57) (width 0.6) (layer "B.Cu") (net 27))
+  (segment (start 105.7 101.803186) (end 105.7 104.3) (width 0.6) (layer "B.Cu") (net 27))
+  (segment (start 105.556347 101.659533) (end 105.7 101.803186) (width 0.6) (layer "B.Cu") (net 27))
   (segment (start 103.012389 102.396356) (end 103.008745 102.4) (width 0.2) (layer "F.Cu") (net 28))
   (segment (start 103.008745 102.4) (end 101.9 102.4) (width 0.2) (layer "F.Cu") (net 28))

Commit message: ...
Parts:
- added JP1: Load on Vsec, Tinker:SolderJumper-2_P_Open_Rounded_skinny, F.Cu at (108.3, 110.7)
- added JP2: Load on Vout, Tinker:SolderJumper-2_P_Open_Rounded_skinny, F.Cu at (108.3, 112.7)
Connections:
- J3 pad 1: unconnected-(J3-Pad1) -> Vout
- J4 pad 1: unconnected-(J4-Pad1) -> Vout
- J5 pad 1: unconnected-(J5-Pad1) -> Vsec
- J6 pad 1: unconnected-(J6-Pad1) -> Vsec
Routing:
- net Vout: track 0.00 -> 37.0 mm, vias 0 -> 1
- net Vsec: track 0.00 -> 21.8 mm, vias 0 -> 1
- net VDD: track 31.1 -> 43.4 mm
