File: Hardware/Li-Ion Charger.kicad_sch (KiCad schematic)
At the start: 44 parts, among them IC1 BQ25792RQMR, J1 Conn_01x07_Male, J10 Output, J11 Conn_01x06, J2 Conn_01x04_Male, J3 Conn_01x02_Male, J4 Conn_01x02_Male, J5 Conn_01x02_Male, J6 Conn_01x02_Male, J7 Conn_01x08_Male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

Commit message: Now...There's a BMS for the Charger!
Parts:
- removed J11: Conn_01x06, Connector_PinSocket_1.27mm:PinSocket_1x06_P1.27mm_Vertical_SMD_Pin1Right, symbol Connector_Generic:Conn_01x06
- added J11: Conn_01x02, Connector_PinSocket_1.27mm:PinSocket_1x02_P1.27mm_Vertical, symbol Connector_Generic:Conn_01x02
Connections:
- net VBUS: now also J11.1 (Pin_1), J11.2 (Pin_2)
Changed lines of the file:
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@@
   (junction (at 114.3 66.04) (diameter 0) (color 0 0 0 0)
   )
-  (junction (at 264.16 132.08) (diameter 0) (color 0 0 0 0)
-  )
   (junction (at 162.56 107.95) (diameter 0) (color 0 0 0 0)
   )
@@
   (junction (at 172.72 48.26) (diameter 0) (color 0 0 0 0)
   )
+  (junction (at 223.52 144.78) (diameter 0) (color 0 0 0 0)
+  )
   (junction (at 242.57 43.18) (diameter 0) (color 0 0 0 0)
   )
@@
   (junction (at 243.84 66.04) (diameter 0) (color 0 0 0 0)
   )
-  (junction (at 264.16 121.92) (diameter 0) (color 0 0 0 0)
-  )
   (junction (at 237.49 66.04) (diameter 0) (color 0 0 0 0)
   )
   (junction (at 193.04 48.26) (diameter 0) (color 0 0 0 0)
-  )
-  (junction (at 267.97 127) (diameter 0) (color 0 0 0 0)
   )
   (junction (at 214.63 66.04) (diameter 0) (color 0 0 0 0)
@@
     (stroke (width 0) (type default) (color 0 0 0 0))
   )
-  (wire (pts (xy 264.16 124.46) (xy 267.97 124.46))
-    (stroke (width 0) (type default) (color 0 0 0 0))
-  )
   (polyline (pts (xy 115.57 144.78) (xy 171.45 144.78))
     (stroke (width 0) (type default) (color 0 0 0 0))
@@
     (stroke (width 0) (type default) (color 0 0 0 0))
   )
-  (wire (pts (xy 264.16 121.92) (xy 264.16 124.46))
-    (stroke (width 0) (type default) (color 0 0 0 0))
-  )
   (polyline (pts (xy 152.4 63.5) (xy 146.05 63.5))
     (stroke (width 0) (type default) (color 0 0 0 0))
@@
   )
   (wire (pts (xy 214.63 55.88) (xy 214.63 66.04))
-    (stroke (width 0) (type default) (color 0 0 0 0))
-  )
-  (wire (pts (xy 264.16 121.92) (xy 267.97 121.92))
     (stroke (width 0) (type default) (color 0 0 0 0))
   )
@@
     (stroke (width 0) (type default) (color 0 0 0 0))
   )
-  (wire (pts (xy 259.08 127) (xy 267.97 127))
-    (stroke (width 0) (type default) (color 0 0 0 0))
-  )
   (wire (pts (xy 191.77 102.87) (xy 186.69 102.87))
     (stroke (width 0) (type default) (color 0 0 0 0))
@@
     (stroke (width 0) (type default) (color 0 0 0 0))
   )
-  (wire (pts (xy 264.16 132.08) (xy 264.16 134.62))
-    (stroke (width 0) (type default) (color 0 0 0 0))
-  )
   (wire (pts (xy 114.3 73.66) (xy 124.46 73.66))
     (stroke (width 0) (type default) (color 0 0 0 0))
@@
     (stroke (width 0) (type default) (color 0 0 0 0))
   )
-  (wire (pts (xy 267.97 127) (xy 267.97 129.54))
-    (stroke (width 0) (type default) (color 0 0 0 0))
-  )
   (wire (pts (xy 250.19 66.04) (xy 243.84 66.04))
     (stroke (width 0) (type default) (color 0 0 0 0))
@@
     (stroke (width 0) (type default) (color 0 0 0 0))
   )
-  (wire (pts (xy 264.16 134.62) (xy 267.97 134.62))
-    (stroke (width 0) (type default) (color 0 0 0 0))
-  )
   (wire (pts (xy 208.28 68.58) (xy 210.82 68.58))
     (stroke (width 0) (type default) (color 0 0 0 0))
@@
     (stroke (width 0) (type default) (color 0 0 0 0))
   )
-  (wire (pts (xy 264.16 132.08) (xy 267.97 132.08))
-    (stroke (width 0) (type default) (color 0 0 0 0))
-  )
   (wire (pts (xy 242.57 35.56) (xy 252.73 35.56))
     (stroke (width 0) (type default) (color 0 0 0 0))
@@
   )
   (wire (pts (xy 184.15 102.87) (xy 186.69 102.87))
+    (stroke (width 0) (type default) (color 0 0 0 0))
+  )
+  (wire (pts (xy 223.52 144.78) (xy 223.52 147.32))
     (stroke (width 0) (type default) (color 0 0 0 0))
   )
@@
     )
   )
+  (symbol (lib_id "Connector_Generic:Conn_01x02") (at 228.6 144.78 0) (unit 1)
+    (in_bom yes) (on_board yes) (fields_autoplaced)
+    (property "Reference" "J11" (id 0) (at 231.14 144.7799 0)
+      (effects (font (size 1.27 1.27)) (justify left))
+    )
+    (property "Value" "Conn_01x02" (id 1) (at 231.14 147.3199 0)
+      (effects (font (size 1.27 1.27)) (justify left))
+    )
+    (property "Footprint" "Connector_PinSocket_1.27mm:PinSocket_1x02_P1.27mm_Vertical" (id 2) (at 228.6 144.78 0)
+      (effects (font (size 1.27 1.27)) hide)
+    )
+    (property "Datasheet" "~" (id 3) (at 228.6 144.78 0)
+      (effects (font (size 1.27 1.27)) hide)
+    )
+    (pin "1")
+    (pin "2")
+  )
   (symbol (lib_id "power:GND") (at 267.97 102.87 0) (unit 1)
     (in_bom yes) (on_board yes)
@@
     (pin "1")
     (pin "2")
-  )
-  (symbol (lib_id "power:VDD") (at 264.16 132.08 0) (unit 1)
-    (in_bom yes) (on_board yes)
-    (property "Reference" "#PWR0126" (id 0) (at 264.16 135.89 0)
-      (effects (font (size 1.27 1.27)) hide)
-    )
-    (property "Value" "VDD" (id 1) (at 264.16 128.27 0))
-    (property "Footprint" "" (id 2) (at 264.16 132.08 0)
-      (effects (font (size 1.27 1.27)) hide)
-    )
-    (property "Datasheet" "" (id 3) (at 264.16 132.08 0)
-      (effects (font (size 1.27 1.27)) hide)
-    )
-    (pin "1")
-  )
-  (symbol (lib_id "Connector_Generic:Conn_01x06") (at 273.05 127 0) (unit 1)
-    (in_bom yes) (on_board yes) (fields_autoplaced)
-    (property "Reference" "J11" (id 0) (at 275.59 126.9999 0)
-      (effects (font (size 1.27 1.27)) (justify left))
-    )
-    (property "Value" "Conn_01x06" (id 1) (at 275.59 129.5399 0)
-      (effects (font (size 1.27 1.27)) (justify left))
-    )
-    (property "Footprint" "Connector_PinSocket_1.27mm:PinSocket_1x06_P1.27mm_Vertical_SMD_Pin1Right" (id 2) (at 273.05 127 0)
-      (effects (font (size 1.27 1.27)) hide)
-    )
-    (property "Datasheet" "~" (id 3) (at 273.05 127 0)
-      (effects (font (size 1.27 1.27)) hide)
-    )
-    (pin "1")
-    (pin "2")
-    (pin "3")
-    (pin "4")
-    (pin "5")
-    (pin "6")
   )
   (symbol (lib_id "Device:C") (at 148.59 88.9 180) (unit 1)
@@
     (pin "2")
   )
+  (symbol (lib_id "power:VBUS") (at 223.52 144.78 0) (unit 1)
+    (in_bom yes) (on_board yes)
+    (property "Reference" "#PWR0127" (id 0) (at 223.52 148.59 0)
+      (effects (font (size 1.27 1.27)) hide)
+    )
+    (property "Value" "VBUS" (id 1) (at 223.52 140.97 0)
+      (effects (font (size 1.27 1.27) bold))
+    )
+    (property "Footprint" "" (id 2) (at 223.52 144.78 0)
+      (effects (font (size 1.27 1.27)) hide)
+    )
+    (property "Datasheet" "" (id 3) (at 223.52 144.78 0)
+      (effects (font (size 1.27 1.27)) hide)
+    )
+    (pin "1")
+  )
   (symbol (lib_id "Device:C") (at 232.41 39.37 180) (unit 1)
     (in_bom yes) (on_board yes)
@@
     )
     (property "Datasheet" "" (id 3) (at 87.63 41.91 0)
+      (effects (font (size 1.27 1.27)) hide)
+    )
+    (pin "1")
+  )
+  (symbol (lib_id "power:GND") (at 217.17 148.59 0) (unit 1)
+    (in_bom yes) (on_board yes)
+    (property "Reference" "#PWR0128" (id 0) (at 217.17 154.94 0)
+      (effects (font (size 1.27 1.27)) hide)
+    )
+    (property "Value" "GND" (id 1) (at 217.17 152.4 0))
+    (property "Footprint" "" (id 2) (at 217.17 148.59 0)
+      (effects (font (size 1.27 1.27)) hide)
+    )
+    (property "Datasheet" "" (id 3) (at 217.17 148.59 0)
       (effects (font (size 1.27 1.27)) hide)
     )
@@
     (pin "1")
   )
-  (symbol (lib_id "power:GND") (at 259.08 127 0) (unit 1)
-    (in_bom yes) (on_board yes)
-    (property "Reference" "#PWR0122" (id 0) (at 259.08 133.35 0)
-      (effects (font (size 1.27 1.27)) hide)
-    )
-    (property "Value" "GND" (id 1) (at 259.08 130.81 0))
-    (property "Footprint" "" (id 2) (at 259.08 127 0)
-      (effects (font (size 1.27 1.27)) hide)
-    )
-    (property "Datasheet" "" (id 3) (at 259.08 127 0)
-      (effects (font (size 1.27 1.27)) hide)
-    )
-    (pin "1")
-  )
   (symbol (lib_id "Device:C") (at 242.57 39.37 180) (unit 1)
     (in_bom yes) (on_board yes)
@@
     (pin "1")
     (pin "2")
-  )
-  (symbol (lib_id "power:VBUS") (at 264.16 121.92 0) (unit 1)
-    (in_bom yes) (on_board yes)
-    (property "Reference" "#PWR0125" (id 0) (at 264.16 125.73 0)
-      (effects (font (size 1.27 1.27)) hide)
-    )
-    (property "Value" "VBUS" (id 1) (at 264.16 118.11 0))
-    (property "Footprint" "" (id 2) (at 264.16 121.92 0)
-      (effects (font (size 1.27 1.27)) hide)
-    )
-    (property "Datasheet" "" (id 3) (at 264.16 121.92 0)
-      (effects (font (size 1.27 1.27)) hide)
-    )
-    (pin "1")
   )
   (symbol (lib_id "Device:C") (at 162.56 87.63 0) (mirror x) (unit 1)
@@
       (reference "#PWR0121") (unit 1) (value "GND") (footprint "")
     )
-    (path "/b1e87284-c686-4416-b8d0-669d3c8a57f0"
-      (reference "#PWR0122") (unit 1) (value "GND") (footprint "")
-    )
     (path "/df37fa07-f19e-4b86-8f6a-f7465dd4c78c"
       (reference "#PWR0123") (unit 1) (value "GND") (footprint "")
@@
       (reference "#PWR0124") (unit 1) (value "GND") (footprint "")
     )
-    (path "/d4f280cd-7045-43b7-a9c0-c3d43be727f9"
-      (reference "#PWR0125") (unit 1) (value "VBUS") (footprint "")
-    )
-    (path "/1a3b6aff-314d-40d1-b9b3-5ee0561229a6"
-      (reference "#PWR0126") (unit 1) (value "VDD") (footprint "")
+    (path "/4c67a7ba-1a64-46e3-bad8-7626fcfb4ac1"
+      (reference "#PWR0127") (unit 1) (value "VBUS") (footprint "")
+    )
+    (path "/55da2797-c273-46ff-8b24-10c778880c9d"
+      (reference "#PWR0128") (unit 1) (value "GND") (footprint "")
     )
     (path "/d19e3ffc-0a66-4816-942e-569b76b7b9f1"
@@
       (reference "J10") (unit 1) (value "Output") (footprint "Connector_JST:JST_GH_SM04B-GHS-TB_1x04-1MP_P1.25mm_Horizontal")
     )
-    (path "/24e9123d-f6b2-4e3b-993d-e5a78f2d2135"
-      (reference "J11") (unit 1) (value "Conn_01x06") (footprint "Connector_PinSocket_1.27mm:PinSocket_1x06_P1.27mm_Vertical_SMD_Pin1Right")
+    (path "/0483484f-6ae7-4fc9-aea3-5eec488a5fef"
+      (reference "J11") (unit 1) (value "Conn_01x02") (footprint "Connector_PinSocket_1.27mm:PinSocket_1x02_P1.27mm_Vertical")
     )
     (path "/0df60046-7947-4fb7-bc8b-fe56c1ffd6b8"

Commit message: ...
Parts:
- added JP1: Load on Vsec, Tinker:SolderJumper-2_P_Open_Rounded_skinny, symbol Jumper:SolderJumper_2_Open
- added JP2: Load on Vout, Tinker:SolderJumper-2_P_Open_Rounded_skinny, symbol Jumper:SolderJumper_2_Open
Connections:
- net VDD: now also JP1.1 (A), JP2.1 (A)
- net Vout: now also J3.1 (Pin_1), J4.1 (Pin_1), JP2.2 (B)
- net Vsec: now also J5.1 (Pin_1), J6.1 (Pin_1), JP1.2 (B)
Other:
- moved on the sheet: J10, J11
