File: Hardware/Li-Ion BMS.kicad_pcb (KiCad board)
At the start: 2 copper layers, 34 x 34 mm, 54 parts, among them IC1 MAX17320, J10 Battery, J11 Conn_01x02, J2 Conn_01x04_Male, J3 Conn_01x02_Male, J4 Conn_01x02_Male, J5 Conn_01x02_Male, J6 Conn_01x02_Male, J7 Conn_01x08_Male, J9 QWIIC_Stack_II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

Commit message: ...
Parts:
- moved Q2 1.00 mm to (92.0, 103.5)
- moved R6 1.00 mm to (92.0, 100.8)
Routing:
- net /pfail: track 20.3 -> 21.5 mm
- net Net-(F1-Pad2): track 2.66 -> 1.66 mm
Changed lines of the file:
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@@
   )
   (footprint "Package_TO_SOT_SMD:SOT-23" (layer "F.Cu")
-    (at 92 102.5 -90)
+    (at 92 103.5 -90)
     (descr "SOT, 3 Pin (https://www.jedec.org/system/files/docs/to-236h.pdf variant AB), generated with kicad-footprint-generator ipc_gullwing_generator.py")
     (tags "SOT TO_SOT_SMD")
@@
   )
   (footprint "Resistor_SMD:R_0603_1608Metric" (layer "F.Cu")
-    (at 92 99.8 180)
+    (at 92 100.8 180)
     (descr "Resistor SMD 0603 (1608 Metric), square (rectangular) end terminal, IPC_7351 nominal, (Body size source: IPC-SM-782 page 72, https://www.pcb-3d.com/wordpress/wp-content/uploads/ipc-sm-782a_amendment_1_and_2.pdf), generated with kicad-footprint-generator")
     (tags "resistor")
@@
       (effects (font (size 1.27 1.27) (thickness 0.254)))
     )
-    (fp_line (start -2 1.5) (end -1.2 1.5) (layer "F.SilkS") (width 0.2))
-    (fp_line (start -1.2 -1.5) (end -2 -1.5) (layer "F.SilkS") (width 0.2))
-    (fp_line (start 2 -1.5) (end 2 1.5) (layer "F.SilkS") (width 0.2))
-    (fp_line (start 0.25 2.6) (end 0.25 2.6) (layer "F.SilkS") (width 0.1))
-    (fp_line (start 1.8 -1.5) (end 2 -1.5) (layer "F.SilkS") (width 0.2))
+    (fp_line (start -2 -1.5) (end -2 -1.2) (layer "F.SilkS") (width 0.2))
     (fp_line (start 2 1.5) (end 1.8 1.5) (layer "F.SilkS") (width 0.2))
+    (fp_line (start 2 -1.5) (end 2 1.5) (layer "F.SilkS") (width 0.2))
     (fp_line (start 0.25 2.5) (end 0.25 2.5) (layer "F.SilkS") (width 0.1))
-    (fp_line (start -2 -1.5) (end -2 -1.2) (layer "F.SilkS") (width 0.2))
+    (fp_line (start 0.25 2.6) (end 0.25 2.6) (layer "F.SilkS") (width 0.1))
     (fp_line (start -2 1.2) (end -2 1.5) (layer "F.SilkS") (width 0.2))
-    (fp_arc (start 0.25 2.5) (mid 0.3 2.55) (end 0.25 2.6) (layer "F.SilkS") (width 0.1))
+    (fp_line (start 1.8 -1.5) (end 2 -1.5) (layer "F.SilkS") (width 0.2))
+    (fp_line (start -2 1.5) (end -1.2 1.5) (layer "F.SilkS") (width 0.2))
+    (fp_line (start -1.2 -1.5) (end -2 -1.5) (layer "F.SilkS") (width 0.2))
     (fp_arc (start 0.25 2.6) (mid 0.2 2.55) (end 0.25 2.5) (layer "F.SilkS") (width 0.1))
-    (fp_line (start -3.5 3) (end -3.5 -3) (layer "F.CrtYd") (width 0.1))
-    (fp_line (start 3 -3) (end 3 3) (layer "F.CrtYd") (width 0.1))
-    (fp_line (start 3 3) (end -3.5 3) (layer "F.CrtYd") (width 0.1))
-    (fp_line (start -3.5 -3) (end 3 -3) (layer "F.CrtYd") (width 0.1))
-    (fp_line (start -2 -1.5) (end -2 1.5) (layer "F.Fab") (width 0.1))
+    (fp_arc (start 0.25 2.5) (mid 0.3 2.55) (end 0.25 2.6) (layer "F.SilkS") (width 0.1))
+    (fp_line (start -2.5 2) (end -2.5 -2) (layer "F.CrtYd") (width 0.05))
+    (fp_line (start -2.5 -2) (end 2.5 -2) (layer "F.CrtYd") (width 0.05))
+    (fp_line (start 2.5 -2) (end 2.5 2) (layer "F.CrtYd") (width 0.05))
+    (fp_line (start 2.5 2) (end -2.5 2) (layer "F.CrtYd") (width 0.05))
     (fp_line (start 2 -1.5) (end -2 -1.5) (layer "F.Fab") (width 0.1))
     (fp_line (start -2 1.5) (end 2 1.5) (layer "F.Fab") (width 0.1))
+    (fp_line (start -2 -1.5) (end -2 1.5) (layer "F.Fab") (width 0.1))
     (fp_line (start 2 1.5) (end 2 -1.5) (layer "F.Fab") (width 0.1))
     (pad "1" smd rect (at 0.25 1.225) (size 1.55 2.4) (layers "F.Cu" "F.Paste" "F.Mask")
@@
   (segment (start 101.058564 91.083564) (end 100.175 90.2) (width 0.2) (layer "F.Cu") (net 40))
   (segment (start 100.797361 93.440256) (end 100.797361 92.884118) (width 0.2) (layer "F.Cu") (net 40))
-  (segment (start 92 106.1) (end 92 103.4375) (width 0.2) (layer "F.Cu") (net 41))
+  (segment (start 92 106.1) (end 92 104.4375) (width 0.2) (layer "F.Cu") (net 41))
   (segment (start 100.109861 96.627756) (end 100.109861 97.815139) (width 0.2) (layer "F.Cu") (net 42))
   (segment (start 98.754672 99.2) (end 100.180183 100.625511) (width 0.2) (layer "F.Cu") (net 42))
@@
   (segment (start 102.297361 98.294431) (end 102.604264 98.601334) (width 0.2) (layer "F.Cu") (net 52))
   (segment (start 102.797361 98.061689) (end 102.797361 97.315256) (width 0.2) (layer "F.Cu") (net 53))
-  (segment (start 92.95 99.14818) (end 92.95 101.3625) (width 0.2) (layer "F.Cu") (net 53))
+  (segment (start 92.95 99.14818) (end 92.95 102.5625) (width 0.2) (layer "F.Cu") (net 53))
   (segment (start 92.991277 99.306903) (end 92.95 99.34818) (width 0.2) (layer "F.Cu") (net 53))
   (via (at 92.991277 99.106903) (size 0.5) (drill 0.3) (layers "F.Cu" "B.Cu") (net 53))

Commit message: ...
Parts:
- removed J10: Battery, Connector_JST:JST_GH_SM04B-GHS-TB_1x04-1MP_P1.25mm_Horizontal
- added J12: Conn_01x05_MountingPin, Connector_JST:JST_GH_SM05B-GHS-TB_1x05-1MP_P1.25mm_Horizontal, F.Cu at (100.0, 114.0)
- moved B1 1.00 mm to (109.0, 114.0)
- moved B2 1.00 mm to (91.0, 114.0)
- moved R3 1.00 mm to (106.5, 114.0)
- moved R9 1.00 mm to (93.5, 114.0)
Connections:
- net /batts renamed batts
- net /cell1 renamed cell3
- R15 pad 2: /cell -> cell
Routing:
- net cell: track 0.00 -> 28.7 mm, vias 0 -> 2
- net /cell: track 27.3 -> 0.00 mm, vias 2 -> 0
- net VBUS: track 31.4 -> 32.8 mm
- net +BATT: track 27.5 -> 26.9 mm
