File: Hardware/Li-Ion BMS.kicad_sch (KiCad schematic)
At the start: 49 parts, among them IC1 MAX17320, J1 Conn_01x07_Male, J10 Battery, J11 Conn_01x02, J2 Conn_01x04_Male, J3 Conn_01x02_Male, J4 Conn_01x02_Male, J5 Conn_01x02_Male, J6 Conn_01x02_Male, J7 Conn_01x08_Male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

Commit message: ...
Parts:
- added J12: Conn_01x05_MountingPin, Connector_JST:JST_GH_SM05B-GHS-TB_1x05-1MP_P1.25mm_Horizontal, symbol Connector_Generic_MountingPin:Conn_01x05_MountingPin
- J10: now left out of the parts list
Connections:
- net +BATT: now also J12.1 (Pin_1); no longer J10.1 (Pin_1)
- net GND: now also J12.MP (MountPin)
- net GNDREF: now also J12.5 (Pin_5)
- net cell: now also J12.2 (Pin_2), J12.3 (Pin_3), J12.4 (Pin_4); no longer J10.2 (Pin_2), J10.3 (Pin_3)
- new net: J10.2 (Pin_2), J10.3 (Pin_3)
Other:
- moved on the sheet: J11
