File: Hardware/USB Hub.kicad_sch (KiCad schematic)
At the start: 24 parts, among them J1 Conn_01x07_Male, J10 Conn_01x04_Male, J11 USB_C_Receptacle, J12 USB_C_Receptacle, J2 Conn_01x04_Male, J3 Conn_01x02_Male, J4 Conn_01x02_Male, J5 Conn_01x02_Male, J6 Conn_01x02_Male, J7 Conn_01x08_Male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

Commit message: workin' on the USB Hub
Parts:
- added C10, C5, C6, C7, C8, C9: 22pf, Capacitor_SMD:C_0603_1608Metric, symbol Device:C
- added R10, R11, R12, R13, R14, R15: 1K5, Resistor_SMD:R_0603_1608Metric, symbol Device:R
- added R4, R5, R6, R7, R8, R9: 30, Resistor_SMD:R_0603_1608Metric, symbol Device:R
Connections:
- net GND: now also C10.2, C5.2, C6.2, C7.2, C8.2, C9.2, R10.2, R11.2, R12.2, R13.2, R14.2, R15.2
- net UD1+: now also R10.1, R4.2; no longer U1.12 (DP1)
- net UD1-: now also R13.1, R5.2; no longer U1.11 (DM1)
- net UD2+: now also R11.1, R6.2; no longer U1.16 (DP2)
- net UD2-: now also R14.1, R7.2; no longer U1.15 (DM2)
- net UD3+: now also R12.1, R8.2; no longer U1.20 (DP3)
- net UD3-: now also R15.1, R9.2; no longer U1.19 (DM3)
- net USB0+: now reaches C3.1, R1.2, R3.1, U1.1 (DP0)
- net USB0-: now reaches C4.1, R2.2, U1.2 (DM0)
- new net USB1+: C5.1, R4.1, U1.12 (DP1)
- new net USB1-: C8.1, R5.1, U1.11 (DM1)
- new net USB2+: C6.1, R6.1, U1.16 (DP2)
- new net USB2-: C9.1, R7.1, U1.15 (DM2)
- new net USB3+: C7.1, R8.1, U1.20 (DP3)
- new net USB3-: C10.1, R9.1, U1.19 (DM3)
Other:
- moved on the sheet: D1, D2, D3, D4, J10, J11, J12

Commit message: Some updates to the hub
Parts:
- added C11: .1uf, Capacitor_SMD:C_0603_1608Metric, symbol Device:C
- added R16: 15, Resistor_SMD:R_0603_1608Metric, symbol Device:R
Connections:
- net +3V3: now also U1.26 (~{EXTMEM}), R16.1
- net GND: now also C11.2; no longer U1.26 (~{EXTMEM})
- net ~{reset}: now reaches U1.4 (~{RESET})
- net ~{reset}: now also C11.1, R16.2
- no-connect marks 4 -> 7

Commit message: Possibly completed USB Hub board
Parts:
- added C12, C13: 1uF, Capacitor_SMD:C_0603_1608Metric, symbol Device:C
- added C2: 0.1uf, Capacitor_SMD:C_0603_1608Metric, symbol Device:C
- added U2: AP2112K-3.3, Package_TO_SOT_SMD:SOT-23-5, symbol Regulator_Linear:AP2112K-3.3
- added X1: ASE-xxxMHz, Oscillator:Oscillator_SMD_Abracon_ASE-4Pin_3.2x2.5mm, symbol Oscillator:ASE-xxxMHz
- renumbered C2 to C14
Connections:
- net Vout is gone; now on net Vbus: J2.1 (Pin_1)
- net +3V3: now also U1.31 (MODE), C13.1, C2.1, U2.5 (VOUT), X1.1 (EN), X1.4 (Vdd)
- net GND: now also C12.2, C13.2, C2.2, U2.2 (GND), X1.2 (GND); no longer U1.31 (MODE)
- net Vbus: now also C12.1, U2.1 (VIN), U2.3 (EN)
- net XTAL1: now reaches U1.30 (XTAL1/CLK48)
- net XTAL1: now also X1.3 (OUT)
- net CC21: no longer names the net of J11.A5 (CC1)
- net CC22: no longer names the net of J11.B5 (CC2)
- net CC31: no longer names the net of J12.A5 (CC1)
- net CC32: no longer names the net of J12.B5 (CC2)
- no-connect marks 7 -> 12
Other:
- note added: "This is because it's a BUS POWERED hub..."
- note added: "Vusb Power"
- note removed: "Vout Power"
- moved on the sheet: C1, C10, C11, C14, C3, C4, C5, C6, C7, C8, C9, J10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
