File: Hardware/USB Hub.kicad_pcb (KiCad board)
At the start: 2 copper layers, 34 x 34 mm, 42 parts, among them J10 Conn_01x04_Male, J11 USB_C_Receptacle, J12 USB_C_Receptacle, J2 Conn_01x04_Male, J3 Conn_01x02_Male, J4 Conn_01x02_Male, J5 Conn_01x02_Male, J6 Conn_01x02_Male, J7 Conn_01x08_Male, J9 QWIIC_Stack_II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

Commit message: Some updates to the hub
Parts:
- added C11: .1uf, Capacitor_SMD:C_0603_1608Metric, F.Cu at (93.8, 96.0)
- added R16: 15, Resistor_SMD:R_0603_1608Metric, F.Cu at (93.8, 93.0)
- moved C1 2.18 mm to (95.3, 93.0), turned to 90 degrees
Connections:
- U1 pad 26: GND -> +3V3
- U1 pad 4: unconnected-(U1-Pad4) -> /~{reset}
Routing:
- net /~{reset}: track 0.00 -> 5.57 mm
- net +3V3: track 13.6 -> 17.7 mm

Commit message: Possibly completed USB Hub board
Parts:
- added C12: 1uF, Capacitor_SMD:C_0603_1608Metric, B.Cu at (106.8, 93.8)
- added C13: 1uF, Capacitor_SMD:C_0603_1608Metric, B.Cu at (106.8, 100.1)
- added C2: 0.1uf, Capacitor_SMD:C_0603_1608Metric, F.Cu at (110.3, 95.0)
- added U2: AP2112K-3.3, Package_TO_SOT_SMD:SOT-23-5, B.Cu at (107.0, 96.7)
- added X1: ASE-xxxMHz, Oscillator:Oscillator_SMD_Abracon_ASE-4Pin_3.2x2.5mm, F.Cu at (107.8, 95.0)
- moved C11 4.08 mm to (93.0, 100.0)
- moved R16 3.57 mm to (94.9, 96.4), turned to -135 degrees
- moved C7 3.18 mm to (101.7, 105.0), turned to 180 degrees
- moved C9 3.18 mm to (98.3, 105.0), turned to 0 degrees
- moved C14 2.45 mm to (107.0, 100.0), turned to -90 degrees
- moved C1 2.14 mm to (97.0, 94.3), turned to 45 degrees
- moved R3 1.20 mm to (103.5, 94.8), turned to -45 degrees
- moved C10 0.84 mm to (101.7, 106.5), turned to 180 degrees
- moved C6 0.83 mm to (98.3, 106.5), turned to 0 degrees
- moved C5 0.67 mm to (105.3, 90.0)
- moved C8 0.67 mm to (105.3, 91.5)
- moved R4 0.56 mm to (102.3, 90.0)
- moved R5 0.56 mm to (102.3, 91.5)
- moved R10 0.50 mm to (99.4, 90.0)
- moved R13 0.50 mm to (99.4, 91.5)
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- renumbered C2 to C14
Connections:
- J11 pad A5: CC21 -> unconnected-(J11-PadA5)
- J11 pad B5: CC22 -> unconnected-(J11-PadB5)
- J12 pad A5: CC31 -> unconnected-(J12-PadA5)
- J12 pad B5: CC32 -> unconnected-(J12-PadB5)
- J2 pad 1: Vout -> Vusb
- U1 pad 30: unconnected-(U1-Pad30) -> /XTAL1
- U1 pad 31: GND -> +3V3
Routing:
- net Vusb: track 0.00 -> 16.1 mm
- net +3V3: track 17.7 -> 28.8 mm, vias 0 -> 1
- net /XTAL1: track 0.00 -> 5.79 mm
- net Vbus: track 47.6 -> 45.3 mm
- net GND: track 0.00 -> 1.95 mm, vias 0 -> 1
- net /USB0-: track 6.15 -> 7.61 mm
- net Net-(R3-Pad2): track 4.55 -> 3.16 mm
- net /USB2+: track 5.63 -> 4.28 mm
- net /USB0+: track 7.94 -> 6.61 mm
- net /USB2-: track 4.60 -> 3.32 mm
- net /~{reset}: track 5.57 -> 6.61 mm
- net /USB3-: track 5.28 -> 4.55 mm
- net /USB3+: track 2.70 -> 3.38 mm
- net UD1-: track 5.68 -> 6.25 mm

Commit message: ...
Connections:
- C12 pad 1: Vusb -> Vbus
- J2 pad 1: Vusb -> Vbus
- U2 pad 1: Vusb -> Vbus
- U2 pad 3: Vusb -> Vbus
Routing:
- net Vbus: track 45.3 -> 65.7 mm
- net Vusb: track 16.1 -> 0.00 mm
Changed lines of the file:
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@@
   (net 51 "unconnected-(U2-Pad4)")
   (net 52 "unconnected-(U1-Pad29)")
-  (net 53 "Vusb")
-  (net 54 "unconnected-(J11-PadA5)")
-  (net 55 "unconnected-(J11-PadB5)")
-  (net 56 "unconnected-(J12-PadA5)")
-  (net 57 "unconnected-(J12-PadB5)")
+  (net 53 "unconnected-(J11-PadA5)")
+  (net 54 "unconnected-(J11-PadB5)")
+  (net 55 "unconnected-(J12-PadA5)")
+  (net 56 "unconnected-(J12-PadB5)")
   (footprint "Tinker:Mount" (layer "F.Cu")
     (at 114 114 45)
@@
       (net 29 "Vbus") (pinfunction "VBUS") (pintype "passive"))
     (pad "A5" smd rect (at -1.25 -4.045) (size 0.3 1.45) (layers "F.Cu" "F.Paste" "F.Mask")
-      (net 56 "unconnected-(J12-PadA5)") (pinfunction "CC1") (pintype "bidirectional+no_connect"))
+      (net 55 "unconnected-(J12-PadA5)") (pinfunction "CC1") (pintype "bidirectional+no_connect"))
     (pad "A6" smd rect (at -0.25 -4.045) (size 0.3 1.45) (layers "F.Cu" "F.Paste" "F.Mask")
       (net 34 "UD3+") (pinfunction "D+") (pintype "bidirectional"))
@@
       (net 29 "Vbus") (pinfunction "VBUS") (pintype "passive"))
     (pad "B5" smd rect (at 1.75 -4.045) (size 0.3 1.45) (layers "F.Cu" "F.Paste" "F.Mask")
-      (net 57 "unconnected-(J12-PadB5)") (pinfunction "CC2") (pintype "bidirectional+no_connect"))
+      (net 56 "unconnected-(J12-PadB5)") (pinfunction "CC2") (pintype "bidirectional+no_connect"))
     (pad "B6" smd rect (at 0.75 -4.045) (size 0.3 1.45) (layers "F.Cu" "F.Paste" "F.Mask")
       (net 34 "UD3+") (pinfunction "D+") (pintype "bidirectional"))
@@
       (net 29 "Vbus") (pinfunction "VBUS") (pintype "passive"))
     (pad "A5" smd rect (at -1.25 -4.045) (size 0.3 1.45) (layers "F.Cu" "F.Paste" "F.Mask")
-      (net 54 "unconnected-(J11-PadA5)") (pinfunction "CC1") (pintype "bidirectional+no_connect"))
+      (net 53 "unconnected-(J11-PadA5)") (pinfunction "CC1") (pintype "bidirectional+no_connect"))
     (pad "A6" smd rect (at -0.25 -4.045) (size 0.3 1.45) (layers "F.Cu" "F.Paste" "F.Mask")
       (net 30 "UD2+") (pinfunction "D+") (pintype "bidirectional"))
@@
       (net 29 "Vbus") (pinfunction "VBUS") (pintype "passive"))
     (pad "B5" smd rect (at 1.75 -4.045) (size 0.3 1.45) (layers "F.Cu" "F.Paste" "F.Mask")
-      (net 55 "unconnected-(J11-PadB5)") (pinfunction "CC2") (pintype "bidirectional+no_connect"))
+      (net 54 "unconnected-(J11-PadB5)") (pinfunction "CC2") (pintype "bidirectional+no_connect"))
     (pad "B6" smd rect (at 0.75 -4.045) (size 0.3 1.45) (layers "F.Cu" "F.Paste" "F.Mask")
       (net 30 "UD2+") (pinfunction "D+") (pintype "bidirectional"))
@@
     (fp_line (start -0.8 1.05) (end -0.4 1.45) (layer "B.Fab") (width 0.1))
     (pad "1" smd roundrect (at -1.1375 0.95 270) (size 1.325 0.6) (layers "B.Cu" "B.Paste" "B.Mask") (roundrect_rratio 0.25)
-      (net 53 "Vusb") (pinfunction "VIN") (pintype "power_in"))
+      (net 29 "Vbus") (pinfunction "VIN") (pintype "power_in"))
     (pad "2" smd roundrect (at -1.1375 0 270) (size 1.325 0.6) (layers "B.Cu" "B.Paste" "B.Mask") (roundrect_rratio 0.25)
       (net 3 "GND") (pinfunction "GND") (pintype "power_in"))
     (pad "3" smd roundrect (at -1.1375 -0.95 270) (size 1.325 0.6) (layers "B.Cu" "B.Paste" "B.Mask") (roundrect_rratio 0.25)
-      (net 53 "Vusb") (pinfunction "EN") (pintype "input"))
+      (net 29 "Vbus") (pinfunction "EN") (pintype "input"))
     (pad "4" smd roundrect (at 1.1375 -0.95 270) (size 1.325 0.6) (layers "B.Cu" "B.Paste" "B.Mask") (roundrect_rratio 0.25)
       (net 51 "unconnected-(U2-Pad4)") (pinfunction "NC") (pintype "no_connect"))
@@
     (fp_line (start -0.8 0.4) (end 0.8 0.4) (layer "B.Fab") (width 0.1))
     (pad "1" smd roundrect (at -0.775 0) (size 0.9 0.95) (layers "B.Cu" "B.Paste" "B.Mask") (roundrect_rratio 0.25)
-      (net 53 "Vusb") (pintype "passive"))
+      (net 29 "Vbus") (pintype "passive"))
     (pad "2" smd roundrect (at 0.775 0) (size 0.9 0.95) (layers "B.Cu" "B.Paste" "B.Mask") (roundrect_rratio 0.25)
       (net 3 "GND") (pintype "passive"))
@@
     (fp_line (start 0.9 2.715) (end 0.9 -2.715) (layer "B.Fab") (width 0.1))
     (pad "1" smd rect (at -1.35 1.905 90) (size 1.8 1) (layers "B.Cu" "B.Paste" "B.Mask")
-      (net 53 "Vusb") (pinfunction "Pin_1") (pintype "passive"))
+      (net 29 "Vbus") (pinfunction "Pin_1") (pintype "passive"))
     (pad "2" smd rect (at 1.35 0.635 90) (size 1.8 1) (layers "B.Cu" "B.Paste" "B.Mask")
       (net 1 "UD+") (pinfunction "Pin_2") (pintype "passive"))
@@
   (segment (start 106.989551 94.01464) (end 104.290772 94.01464) (width 0.25) (layer "F.Cu") (net 27))
   (segment (start 108.45 108.955) (end 108.45 107.8) (width 0.5) (layer "F.Cu") (net 29))
-  (segment (start 102.982789 87.489881) (end 102.97267 87.5) (width 0.5) (layer "F.Cu") (net 29))
   (segment (start 96.45 108.955) (end 96.45 107.8) (width 0.5) (layer "F.Cu") (net 29))
   (segment (start 91.55 108.955) (end 91.55 107.8) (width 0.5) (layer "F.Cu") (net 29))
-  (segment (start 102.97267 87.5) (end 101.905 87.5) (width 0.5) (layer "F.Cu") (net 29))
+  (segment (start 104.34809 87.404737) (end 104.252827 87.5) (width 0.5) (layer "F.Cu") (net 29))
+  (segment (start 104.252827 87.5) (end 101.905 87.5) (width 0.5) (layer "F.Cu") (net 29))
   (segment (start 103.55 108.955) (end 103.55 107.8) (width 0.5) (layer "F.Cu") (net 29))
   (via (at 103.55 107.8) (size 0.8) (drill 0.4) (layers "F.Cu" "B.Cu") (net 29))
   (via (at 91.55 107.8) (size 0.8) (drill 0.4) (layers "F.Cu" "B.Cu") (net 29))
-  (via (at 102.982789 87.489881) (size 0.8) (drill 0.4) (layers "F.Cu" "B.Cu") (net 29))
+  (via (at 104.34809 87.404737) (size 0.8) (drill 0.4) (layers "F.Cu" "B.Cu") (net 29))
   (via (at 108.45 107.8) (size 0.8) (drill 0.4) (layers "F.Cu" "B.Cu") (net 29))
   (via (at 96.45 107.8) (size 0.8) (drill 0.4) (layers "F.Cu" "B.Cu") (net 29))
   (segment (start 96.45 107.8) (end 100.01347 107.8) (width 0.5) (layer "B.Cu") (net 29))
-  (segment (start 102.982789 87.489881) (end 104.369826 88.876918) (width 0.5) (layer "B.Cu") (net 29))
-  (segment (start 100.01347 100.12795) (end 100.01347 107.8) (width 0.5) (layer "B.Cu") (net 29))
+  (segment (start 102.205591 86.141594) (end 104.89476 86.141594) (width 0.5) (layer "B.Cu") (net 29))
+  (segment (start 106.632331 96.486833) (end 107.459372 96.486833) (width 0.25) (layer "B.Cu") (net 29))
+  (segment (start 104.34809 87.404737) (end 101.959737 87.404737) (width 0.5) (layer "B.Cu") (net 29))
+  (segment (start 104.34809 87.404737) (end 104.369826 87.426473) (width 0.5) (layer "B.Cu") (net 29))
+  (segment (start 106 93.83599) (end 106 95.540961) (width 0.5) (layer "B.Cu") (net 29))
+  (segment (start 101.905 87.35) (end 101.905 86.442185) (width 0.5) (layer "B.Cu") (net 29))
+  (segment (start 107.459372 96.486833) (end 107.9 96.046205) (width 0.25) (layer "B.Cu") (net 29))
+  (segment (start 104.369826 95.771594) (end 100.01347 100.12795) (width 0.5) (layer "B.Cu") (net 29))
+  (segment (start 104.369826 87.426473) (end 104.369826 95.771594) (width 0.5) (layer "B.Cu") (net 29))
+  (segment (start 107.9 96.046205) (end 107.9 95.540961) (width 0.25) (layer "B.Cu") (net 29))
   (segment (start 96.45 107.8) (end 91.55 107.8) (width 0.5) (layer "B.Cu") (net 29))
   (segment (start 103.55 107.8) (end 108.45 107.8) (width 0.5) (layer "B.Cu") (net 29))
+  (segment (start 101.905 86.442185) (end 102.205591 86.141594) (width 0.5) (layer "B.Cu") (net 29))
+  (segment (start 106 95.854502) (end 106.632331 96.486833) (width 0.25) (layer "B.Cu") (net 29))
   (segment (start 100.01347 107.8) (end 103.55 107.8) (width 0.5) (layer "B.Cu") (net 29))
-  (segment (start 104.369826 95.771594) (end 100.01347 100.12795) (width 0.5) (layer "B.Cu") (net 29))
-  (segment (start 104.369826 88.876918) (end 104.369826 95.771594) (width 0.5) (layer "B.Cu") (net 29))
+  (segment (start 106 95.540961) (end 106 95.854502) (width 0.25) (layer "B.Cu") (net 29))
+  (segment (start 104.89476 86.141594) (end 106 87.246834) (width 0.5) (layer "B.Cu") (net 29))
+  (segment (start 100.01347 100.12795) (end 100.01347 107.8) (width 0.5) (layer "B.Cu") (net 29))
+  (segment (start 101.959737 87.404737) (end 101.905 87.35) (width 0.5) (layer "B.Cu") (net 29))
+  (segment (start 106 87.246834) (end 106 93.83599) (width 0.5) (layer "B.Cu") (net 29))
   (segment (start 94.581806 110.007341) (end 94.75 109.839147) (width 0.2) (layer "F.Cu") (net 30))
   (segment (start 94.75 108.955) (end 94.75 107.45) (width 0.2) (layer "F.Cu") (net 30))
@@
   (segment (start 96.245747 96.400342) (end 94.995499 97.650591) (width 0.25) (layer "F.Cu") (net 50))
   (segment (start 94.316637 96.983363) (end 94.983865 97.650591) (width 0.25) (layer "F.Cu") (net 50))
-  (segment (start 103.299744 86.141594) (end 102.205591 86.141594) (width 0.5) (layer "B.Cu") (net 53))
-  (segment (start 106.632331 96.486833) (end 107.459372 96.486833) (width 0.25) (layer "B.Cu") (net 53))
-  (segment (start 106 93.83599) (end 106 88.841851) (width 0.5) (layer "B.Cu") (net 53))
-  (segment (start 106 93.83599) (end 106 95.540961) (width 0.5) (layer "B.Cu") (net 53))
-  (segment (start 107.459372 96.486833) (end 107.9 96.046205) (width 0.25) (layer "B.Cu") (net 53))
-  (segment (start 101.905 86.442185) (end 101.905 87.35) (width 0.5) (layer "B.Cu") (net 53))
-  (segment (start 107.9 96.046205) (end 107.9 95.540961) (width 0.25) (layer "B.Cu") (net 53))
-  (segment (start 106 95.854502) (end 106.632331 96.486833) (width 0.25) (layer "B.Cu") (net 53))
-  (segment (start 106 88.841851) (end 103.299744 86.141594) (width 0.5) (layer "B.Cu") (net 53))
-  (segment (start 102.205591 86.141594) (end 101.905 86.442185) (width 0.5) (layer "B.Cu") (net 53))
-  (segment (start 106 95.540961) (end 106 95.854502) (width 0.25) (layer "B.Cu") (net 53))
   (zone (net 3) (net_name "GND") (layer "F.Cu") (hatch edge 0.508)
     (connect_pads (clearance 0.254))

Commit message: USB Hub2... Now with Overcurrent Protection
Parts:
- added R23: 0, Resistor_SMD:R_0603_1608Metric, B.Cu at (108.6, 91.5)
- moved C8 11.2 mm to (94.3, 90.0), turned to 180 degrees
- moved C5 11.2 mm to (94.3, 91.5), turned to 180 degrees
- moved C2 8.23 mm to (105.0, 88.7), turned to 180 degrees
- moved R5 5.28 mm to (97.3, 90.0), turned to 0 degrees
- moved R4 5.28 mm to (97.3, 91.5), turned to 0 degrees
- moved X1 4.90 mm to (104.7, 91.2), turned to 180 degrees
- moved C11 4.77 mm to (93.8, 95.3), turned to 45 degrees
- moved R13 1.75 mm to (100.3, 90.0), turned to 0 degrees
- moved R10 1.75 mm to (100.3, 91.5), turned to 0 degrees
- moved R3 0.57 mm to (103.1, 94.4)
Connections:
- C12 pad 1: Vbus -> Vusb
- J2 pad 1: Vbus -> Vusb
- U1 pad 10: unconnected-(U1-Pad10) -> OVERCUR1
- U1 pad 9: unconnected-(U1-Pad9) -> PWRON1
- U2 pad 1: Vbus -> Vusb
- U2 pad 3: Vbus -> Vusb
Routing:
- net Vusb: track 0.00 -> 16.6 mm
- net Vbus: track 65.7 -> 61.1 mm
- net +3V3: track 28.8 -> 32.1 mm
- net /USB1+: track 18.0 -> 15.2 mm
- net UD1-: track 6.25 -> 4.12 mm
- net UD1+: track 6.77 -> 8.78 mm
- net /~{reset}: track 6.61 -> 5.16 mm
- net /USB0+: track 6.61 -> 5.60 mm
- net /XTAL1: track 5.79 -> 4.78 mm
- net Net-(R3-Pad2): track 3.16 -> 3.73 mm
