File: Hardware/USB Hub2.kicad_pcb (KiCad board)
At the start: 2 copper layers, 34 x 34 mm, 61 parts, among them J10 Conn_01x04_Male, J11 USB_C_Receptacle, J12 USB_C_Receptacle, J2 Conn_01x04_Male, J3 Conn_01x02_Male, J4 Conn_01x02_Male, J5 Conn_01x02_Male, J6 Conn_01x02_Male, J7 Conn_01x08_Male, J9 QWIIC_Stack_II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

Commit message: More about the Hub...
Parts:
- moved R3 0.57 mm to (103.5, 94.8)
- moved X1 0.33 mm to (104.9, 91.5)
- moved C2 0.29 mm to (104.9, 89.0)
Routing:
- net /USB0+: track 5.60 -> 6.61 mm
- net +3V3: track 34.0 -> 34.7 mm
- net Net-(R3-Pad2): track 3.73 -> 3.16 mm
Changed lines of the file:
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@@
   )
   (footprint "Resistor_SMD:R_0603_1608Metric" (layer "F.Cu")
-    (at 103.1 94.4 -45)
+    (at 103.5 94.8 -45)
     (descr "Resistor SMD 0603 (1608 Metric), square (rectangular) end terminal, IPC_7351 nominal, (Body size source: IPC-SM-782 page 72, https://www.pcb-3d.com/wordpress/wp-content/uploads/ipc-sm-782a_amendment_1_and_2.pdf), generated with kicad-footprint-generator")
     (tags "resistor")
@@
   )
   (footprint "Capacitor_SMD:C_0603_1608Metric" (layer "F.Cu")
-    (at 105 88.7 180)
+    (at 104.932471 88.979515 180)
     (descr "Capacitor SMD 0603 (1608 Metric), square (rectangular) end terminal, IPC_7351 nominal, (Body size source: IPC-SM-782 page 76, https://www.pcb-3d.com/wordpress/wp-content/uploads/ipc-sm-782a_amendment_1_and_2.pdf), generated with kicad-footprint-generator")
     (tags "capacitor")
@@
   )
   (footprint "Oscillator:Oscillator_SMD_Abracon_ASE-4Pin_3.2x2.5mm" (layer "F.Cu")
-    (at 104.7 91.2 180)
+    (at 104.902965 91.457995 180)
     (descr "Miniature Crystal Clock Oscillator Abracon ASE series, http://www.abracon.com/Oscillators/ASEseries.pdf, 3.2x2.5mm^2 package")
     (tags "SMD SMT crystal oscillator")
@@
   (segment (start 102.325 105.153427) (end 101.537957 104.366384) (width 0.25) (layer "F.Cu") (net 24))
   (via (at 105.668067 103.348469) (size 0.5) (drill 0.3) (layers "F.Cu" "B.Cu") (net 24))
-  (segment (start 102.684667 95.601598) (end 102.693007 95.609938) (width 0.25) (layer "F.Cu") (net 25))
-  (segment (start 102.684667 94.764206) (end 102.684667 95.601598) (width 0.25) (layer "F.Cu") (net 25))
-  (segment (start 103.55 92.025) (end 103.55 93.898873) (width 0.25) (layer "F.Cu") (net 25))
-  (segment (start 103.55 93.898873) (end 102.684667 94.764206) (width 0.25) (layer "F.Cu") (net 25))
-  (segment (start 102.103643 96.199301) (end 102.693007 95.609938) (width 0.25) (layer "F.Cu") (net 25))
+  (segment (start 103.976898 93.534989) (end 103.852965 93.411056) (width 0.25) (layer "F.Cu") (net 25))
+  (segment (start 103.976898 94.326046) (end 103.976898 93.534989) (width 0.25) (layer "F.Cu") (net 25))
+  (segment (start 103.852965 93.411056) (end 103.852965 92.282995) (width 0.25) (layer "F.Cu") (net 25))
+  (segment (start 102.103643 96.199301) (end 103.976898 94.326046) (width 0.25) (layer "F.Cu") (net 25))
   (segment (start 94.581806 110.007341) (end 94.75 109.839147) (width 0.2) (layer "F.Cu") (net 27))
   (segment (start 94.75 108.955) (end 94.75 107.45) (width 0.2) (layer "F.Cu") (net 27))
@@
   (segment (start 105.950535 99.066496) (end 106.841496 99.066496) (width 0.5) (layer "F.Cu") (net 33))
   (segment (start 101.537957 95.633616) (end 100.073174 97.098399) (width 0.5) (layer "F.Cu") (net 33))
+  (segment (start 105.039019 93.196941) (end 105.952965 92.282995) (width 0.5) (layer "F.Cu") (net 33))
   (segment (start 105.911767 99.027728) (end 104.93207 99.027728) (width 0.5) (layer "F.Cu") (net 33))
   (segment (start 97.896357 96.199301) (end 96.651992 94.954936) (width 0.5) (layer "F.Cu") (net 33))
   (segment (start 105.739752 92.063172) (end 105.739752 90.413172) (width 0.5) (layer "F.Cu") (net 33))
   (segment (start 105.950535 99.066496) (end 105.911767 99.027728) (width 0.5) (layer "F.Cu") (net 33))
+  (segment (start 105.039019 94.583962) (end 105.039019 93.196941) (width 0.5) (layer "F.Cu") (net 33))
   (segment (start 102.988069 99.868492) (end 101.565548 99.868492) (width 0.5) (layer "F.Cu") (net 33))
   (segment (start 100.181318 96.990255) (end 101.537957 95.633616) (width 0.5) (layer "F.Cu") (net 33))
   (segment (start 104.366384 98.462043) (end 104.93207 99.027728) (width 0.5) (layer "F.Cu") (net 33))
   (segment (start 101.565548 99.868492) (end 100.073174 98.376118) (width 0.5) (layer "F.Cu") (net 33))
-  (segment (start 105.75 92.025) (end 105.75 92.432466) (width 0.5) (layer "F.Cu") (net 33))
-  (segment (start 105.75 92.432466) (end 104.594975 93.587491) (width 0.5) (layer "F.Cu") (net 33))
   (segment (start 106.841496 99.066496) (end 107 99.225) (width 0.5) (layer "F.Cu") (net 33))
   (segment (start 103.221988 99.606439) (end 103.221988 99.634573) (width 0.5) (layer "F.Cu") (net 33))
@@
   (segment (start 105.739752 90.413172) (end 105.739752 89.013172) (width 0.5) (layer "F.Cu") (net 33))
   (via (at 106 98.530675) (size 0.8) (drill 0.4) (layers "F.Cu" "B.Cu") (net 33))
-  (via (at 104.594975 93.587491) (size 0.8) (drill 0.4) (layers "F.Cu" "B.Cu") (net 33))
+  (via (at 105.039019 94.583962) (size 0.8) (drill 0.4) (layers "F.Cu" "B.Cu") (net 33))
   (via (at 100.073174 98.376118) (size 0.8) (drill 0.4) (layers "F.Cu" "B.Cu") (net 33))
+  (segment (start 105.039019 94.583962) (end 103.598504 94.583962) (width 0.5) (layer "B.Cu") (net 33))
   (segment (start 104.665867 97.815961) (end 104.462589 98.019239) (width 0.5) (layer "B.Cu") (net 33))
   (segment (start 106 98.530675) (end 106 97.815961) (width 0.5) (layer "B.Cu") (net 33))
-  (segment (start 100.073174 98.376118) (end 100.073174 98.109292) (width 0.5) (layer "B.Cu") (net 33))
+  (segment (start 100.073174 98.109292) (end 100.073174 98.376118) (width 0.5) (layer "B.Cu") (net 33))
   (segment (start 106 97.815961) (end 104.665867 97.815961) (width 0.5) (layer "B.Cu") (net 33))
-  (segment (start 100.073174 98.109292) (end 104.594975 93.587491) (width 0.5) (layer "B.Cu") (net 33))
-  (segment (start 104.726805 96.026805) (end 103.683363 94.983363) (width 0.25) (layer "F.Cu") (net 38))
+  (segment (start 103.598504 94.583962) (end 100.073174 98.109292) (width 0.5) (layer "B.Cu") (net 33))
+  (segment (start 103.800699 97.896357) (end 104.726805 96.970251) (width 0.25) (layer "F.Cu") (net 38))
   (segment (start 104.726805 96.970251) (end 104.726805 96.026805) (width 0.25) (layer "F.Cu") (net 38))
-  (segment (start 103.800699 97.896357) (end 104.726805 96.970251) (width 0.25) (layer "F.Cu") (net 38))
+  (segment (start 104.726805 96.026805) (end 104.083363 95.383363) (width 0.25) (layer "F.Cu") (net 38))
   (segment (start 95.190422 103.373128) (end 96.061186 103.373128) (width 0.2) (layer "F.Cu") (net 39))
   (segment (start 96.061186 103.373128) (end 96.764986 102.669328) (width 0.2) (layer "F.Cu") (net 39))
@@
   (segment (start 100.75 93.5) (end 102.2 93.5) (width 0.2) (layer "F.Cu") (net 41))
   (segment (start 100.75 93.5) (end 99.18207 95.06793) (width 0.2) (layer "F.Cu") (net 41))
+  (segment (start 102.2 93.5) (end 102.916637 94.216637) (width 0.2) (layer "F.Cu") (net 41))
   (via (at 100.75 93.5) (size 0.5) (drill 0.3) (layers "F.Cu" "B.Cu") (net 41))
   (segment (start 100.75 92) (end 100.75 91.125) (width 0.25) (layer "B.Cu") (net 41))

Commit message: USB Hub2 is pretty much complete!
Parts:
- added D3: PGB1010603NR, Tinker:PGB1010603NRHF, B.Cu at (97.8, 90.5)
- added D4: PGB1010603NR, Tinker:PGB1010603NRHF, B.Cu at (102.2, 90.5)
- added D5: PGB1010603NR, Tinker:PGB1010603NRHF, B.Cu at (92.1, 109.0)
- added D6: PGB1010603NR, Tinker:PGB1010603NRHF, B.Cu at (95.9, 109.0)
- added D7: PGB1010603NR, Tinker:PGB1010603NRHF, B.Cu at (104.1, 109.0)
- added D8: PGB1010603NR, Tinker:PGB1010603NRHF, B.Cu at (107.9, 109.0)
- added JP1: Jumper_3_Bridged12, Jumper:SolderJumper-3_P1.3mm_Bridged2Bar12_RoundedPad1.0x1.5mm, B.Cu at (106.0, 87.3)
- added JP2: Jumper_3_Bridged12, Jumper:SolderJumper-3_P1.3mm_Bridged12_RoundedPad1.0x1.5mm, B.Cu at (94.0, 87.3)
- X1: value ASE-xxxMHz -> ASE-48.000MHz
- moved C13 1.68 mm to (104.5, 95.6)
- moved U2 1.48 mm to (107.0, 95.2)
- moved C12 1.47 mm to (106.8, 92.4)
- moved C1 0.28 mm to (97.2, 94.1)
- moved C11 0.28 mm to (94.0, 95.1)
- moved R16 0.28 mm to (95.1, 96.2)
- moved R1 0.10 mm to (100.8, 90.4)
- moved R2 0.10 mm to (99.2, 90.4)
- moved C3 0.10 mm to (101.5, 93.0)
- moved C4 0.10 mm to (98.5, 93.0)
Connections:
- net /XTAL1 renamed /CLK48
- C12 pad 1: Vusb -> Vusb_PWR
- C15 pad 1: Vusb -> Vusb_PWR
- C16 pad 1: Vusb -> Vusb_PWR
- C17 pad 1: Vusb -> Vusb_PWR
- J5 pad 1: unconnected-(J5-Pad1) -> Vsec
- J6 pad 1: unconnected-(J6-Pad1) -> Vsec
- R17 pad 1: Vusb -> Vusb_PWR
- R18 pad 1: Vusb -> Vusb_PWR
- R19 pad 1: Vusb -> Vusb_PWR
- U1 pad 6: unconnected-(U1-Pad6) -> +3V3
- U1 pad 8: GND -> ~{BUSPWR}
- U2 pad 1: Vusb -> Vusb_PWR
- U2 pad 3: Vusb -> Vusb_PWR
- U3 pad 1: Vusb -> Vusb_PWR
- U4 pad 1: Vusb -> Vusb_PWR
- U5 pad 1: Vusb -> Vusb_PWR
Routing:
- net Vusb: track 38.3 -> 2.82 mm, vias 2 -> 0
- net Vusb_PWR: track 0.00 -> 34.9 mm, vias 0 -> 2
- net Vsec: track 0.00 -> 17.4 mm
- net +3V3: track 34.7 -> 48.0 mm
- net ~{BUSPWR}: track 0.00 -> 12.7 mm, vias 0 -> 1
- net /USB1+: track 19.7 -> 14.2 mm
- net /USB1-: track 20.1 -> 15.0 mm
- net UD2+: track 7.11 -> 10.4 mm, vias 1 -> 2
- net UD2-: track 8.14 -> 11.4 mm, vias 1 -> 2
- net UD3-: track 7.13 -> 10.2 mm, vias 1 -> 2
- net UD3+: track 7.53 -> 10.6 mm, vias 1 -> 2
- net UD1+: track 8.78 -> 11.0 mm, vias 0 -> 1
- net UD1-: track 4.12 -> 5.96 mm, vias 0 -> 1
- net PWRON1: track 21.1 -> 19.8 mm
- net OVERCUR1: track 21.9 -> 21.0 mm
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
Commit message: Yay fer Hub2!
Parts:
- added D1: PGB1010603NR, Tinker:PGB1010603NRHF, B.Cu at (96.7, 90.9)
- added D2: PGB1010603NR, Tinker:PGB1010603NRHF, B.Cu at (103.3, 90.9)
- moved D3 0.43 mm to (97.9, 90.9)
- moved D4 0.43 mm to (102.1, 90.9)
- moved C3 0.40 mm to (101.5, 93.4)
- moved C4 0.40 mm to (98.5, 93.4)
- moved R1 0.40 mm to (100.8, 90.8)
- moved R2 0.40 mm to (99.2, 90.8)
Routing:
- net UD+: track 4.87 -> 8.88 mm
- net UD-: track 2.17 -> 6.17 mm
- net /USB0-: track 7.61 -> 5.35 mm
- net GND: track 5.50 -> 3.56 mm, vias 7 -> 8
- net UD1+: track 11.0 -> 12.8 mm
- net UD1-: track 5.96 -> 6.65 mm
Other:
- board text removed: "WIP!"

Commit message: s'more work on the hub
Routing:
- net Vusb_PWR: track 34.9 -> 35.4 mm
- net GND: vias 8 -> 7
Other:
- board text added: "self|bus"
