File: Hardware/___/zzzzzz.kicad_pcb (KiCad board)
At the start: 2 copper layers, 66.7 x 40.1 mm, 0 parts

Commit message: ...
Other:
- board text removed: "Vusb"
Changed lines of the file:
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@@
     (effects (font (size 1 1) (thickness 0.15)))
   )
-  (gr_text "Vusb" (at 116.2 107 90) (layer "F.SilkS")
+  (gr_text "Vout" (at 116.2 107 90) (layer "F.SilkS")
     (effects (font (size 1 1) (thickness 0.15)))
   )
@@
     (effects (font (size 0.5 0.5) (thickness 0.125)) (justify left))
   )
-  (gr_text "Vusb" (at 83.8 107 -90) (layer "F.SilkS")
+  (gr_text "Vout" (at 83.8 107 -90) (layer "F.SilkS")
     (effects (font (size 1 1) (thickness 0.15)))
   )
