File: Hardware/Controller-RP2040/Controller-RP2040.kicad_sch (KiCad schematic)
At the start: 45 parts, among them J1 Conn_01x07_Male, J2 Conn_01x04_Male, J3 Conn_01x02_Male, J4 Conn_01x02_Male, J5 Conn_01x02_Male, J6 Conn_01x02_Male, J7 Conn_01x08_Male, J8 QWIIC_Vertical, J9 QWIIC_Stack_II, Q1 DMG1012T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

Commit message: Re-arranging the hardware files for better clarity.
Parts:
- U1: LCSC (none) -> C2040
Changed lines of the file:
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@@
+      (effects (font (size 1.27 1.27)) hide)
+    )
+    (property "LCSC" "C2040" (id 4) (at 185.42 88.9 0)
       (effects (font (size 1.27 1.27)) hide)
     )
