File: Hardware/USB Hub/USB Hub2.kicad_sch (KiCad schematic)
At the start: 67 parts, among them J1 Conn_01x07_Male, J10 Conn_01x04_Male, J11 USB_C_Receptacle, J12 USB_C_Receptacle, J2 Conn_01x04_Male, J3 Conn_01x02_Male, J4 Conn_01x02_Male, J5 Conn_01x02_Male, J6 Conn_01x02_Male, J7 Conn_01x08_Male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

Commit message: Re-arranging the hardware files for better clarity.
Parts:
- U2: LCSC (none) -> C51118
- X1: LCSC (none) -> C2650694
Changed lines of the file:
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@@
+      (effects (font (size 1.27 1.27)) hide)
+    )
+    (property "LCSC" "C51118" (id 4) (at 125.73 41.91 0)
       (effects (font (size 1.27 1.27)) hide)
     )
@@
       (effects (font (size 1.27 1.27)) hide)
     )
+    (property "LCSC" "C2650694" (id 4) (at 120.65 140.97 0)
+      (effects (font (size 1.27 1.27)) hide)
+    )
